File: 6522 VIA/6522 VIA.sch (KiCad schematic (older format))
At the start: 11 parts

Commit message: Fixed bugs...
Connections:
- net IRQ: now reaches J?.IRQ2
- net IRQ: now also U?.21 (~IRQ)
- net NMI: no longer names the net of J?.NMI
- net NMI: no longer U?.21 (~IRQ)
Changed lines of the file:
@@
 D7
 Text GLabel 4450 4050 2    50   Output ~ 0
-NMI
+IRQ
 Text GLabel 3150 2250 0    50   Output ~ 0
 GPIO0
@@
 NoConn ~ 4250 6850
 NoConn ~ 4350 6850
-NoConn ~ 4450 6850
 NoConn ~ 4950 6850
 NoConn ~ 5050 6850
@@
 	-1   0    0    1
 $EndComp
-Text GLabel 4750 6850 3    50   Input ~ 0
-NMI
 Text GLabel 4850 6850 3    50   Output ~ 0
 PHI2
@@
 Text GLabel 8800 3900 2    50   Input ~ 0
 A9
+NoConn ~ 4750 6850
+Text GLabel 4450 6850 3    50   Input ~ 0
+IRQ
 $EndSCHEMATC
