File: Baseboard and PSU/Baseboard and PSU.sch (KiCad schematic (older format))
At the start: 16 parts, among them J1 Barrel_Jack, P1 Conn_WallPlug, U1 LM7805_TO220

Commit message: Finished Baseboard schematic...
Parts:
- added J3, J4, J5, J6, J7, J8, J9: BaseboardConnector, PC:BreadboardConnector_Female, symbol PC:BaseboardConnector
- J2: renamed from J?; footprint (none) -> PC:BreadboardConnector_Female
Connections:
- net +5V: now also J3.VCC, J4.VCC, J5.VCC, J6.VCC, J7.VCC, J8.VCC, J9.VCC
- net A0: now also J3.A0, J4.A0, J5.A0, J6.A0, J7.A0, J8.A0, J9.A0
- net A1: now also J3.A1, J4.A1, J5.A1, J6.A1, J7.A1, J8.A1, J9.A1
- net A2: now also J3.A2, J4.A2, J5.A2, J6.A2, J7.A2, J8.A2, J9.A2
- net A3: now also J3.A3, J4.A3, J5.A3, J6.A3, J7.A3, J8.A3, J9.A3
- net A4: now also J3.A4, J4.A4, J5.A4, J6.A4, J7.A4, J8.A4, J9.A4
- net A5: now also J3.A5, J4.A5, J5.A5, J6.A5, J7.A5, J8.A5, J9.A5
- net GND: now also J3.GND, J4.GND, J5.GND, J6.GND, J7.GND, J8.GND, J9.GND
- net 46: now reaches J2.46 (Pin_46)
- net 46: now also J3.46 (Pin_46), J4.46 (Pin_46), J5.46 (Pin_46), J6.46 (Pin_46), J7.46 (Pin_46), J8.46 (Pin_46), J9.46 (Pin_46)
- net 47: now reaches J2.47 (Pin_47)
- net 47: now also J3.47 (Pin_47), J4.47 (Pin_47), J5.47 (Pin_47), J6.47 (Pin_47), J7.47 (Pin_47), J8.47 (Pin_47), J9.47 (Pin_47)
- net 48: now reaches J2.48 (Pin_48)
- net 48: now also J3.48 (Pin_48), J4.48 (Pin_48), J5.48 (Pin_48), J6.48 (Pin_48), J7.48 (Pin_48), J8.48 (Pin_48), J9.48 (Pin_48)
- net 49: now reaches J2.49 (Pin_49)
- net 49: now also J3.49 (Pin_49), J4.49 (Pin_49), J5.49 (Pin_49), J6.49 (Pin_49), J7.49 (Pin_49), J8.49 (Pin_49), J9.49 (Pin_49)
- net 50: now reaches J2.50 (Pin_50)
- net 50: now also J3.50 (Pin_50), J4.50 (Pin_50), J5.50 (Pin_50), J6.50 (Pin_50), J7.50 (Pin_50), J8.50 (Pin_50), J9.50 (Pin_50)
- net 51: now reaches J2.51 (Pin_51)
- net 51: now also J3.51 (Pin_51), J4.51 (Pin_51), J5.51 (Pin_51), J6.51 (Pin_51), J7.51 (Pin_51), J8.51 (Pin_51), J9.51 (Pin_51)
- net 52: now reaches J2.52 (Pin_52)
- net 52: now also J3.52 (Pin_52), J4.52 (Pin_52), J5.52 (Pin_52), J6.52 (Pin_52), J7.52 (Pin_52), J8.52 (Pin_52), J9.52 (Pin_52)
- net 53: now reaches J2.53 (Pin_53)
- net 53: now also J3.53 (Pin_53), J4.53 (Pin_53), J5.53 (Pin_53), J6.53 (Pin_53), J7.53 (Pin_53), J8.53 (Pin_53), J9.53 (Pin_53)
- net 54: now reaches J2.54 (Pin_54)
- net 54: now also J3.54 (Pin_54), J4.54 (Pin_54), J5.54 (Pin_54), J6.54 (Pin_54), J7.54 (Pin_54), J8.54 (Pin_54), J9.54 (Pin_54)
- net 55: now reaches J2.55 (Pin_55)
- net 55: now also J3.55 (Pin_55), J4.55 (Pin_55), J5.55 (Pin_55), J6.55 (Pin_55), J7.55 (Pin_55), J8.55 (Pin_55), J9.55 (Pin_55)
- net 56: now reaches J2.56 (Pin_56)
- net 56: now also J3.56 (Pin_56), J4.56 (Pin_56), J5.56 (Pin_56), J6.56 (Pin_56), J7.56 (Pin_56), J8.56 (Pin_56), J9.56 (Pin_56)
- net 57: now reaches J2.57 (Pin_57)
- net 57: now also J3.57 (Pin_57), J4.57 (Pin_57), J5.57 (Pin_57), J6.57 (Pin_57), J7.57 (Pin_57), J8.57 (Pin_57), J9.57 (Pin_57)
- net 58: now reaches J2.58 (Pin_58)
- net 58: now also J3.58 (Pin_58), J4.58 (Pin_58), J5.58 (Pin_58), J6.58 (Pin_58), J7.58 (Pin_58), J8.58 (Pin_58), J9.58 (Pin_58)
- net 59: now reaches J2.59 (Pin_59)
- net 59: now also J3.59 (Pin_59), J4.59 (Pin_59), J5.59 (Pin_59), J6.59 (Pin_59), J7.59 (Pin_59), J8.59 (Pin_59), J9.59 (Pin_59)
- net 60: now reaches J2.60 (Pin_60)
- net 60: now also J3.60 (Pin_60), J4.60 (Pin_60), J5.60 (Pin_60), J6.60 (Pin_60), J7.60 (Pin_60), J8.60 (Pin_60), J9.60 (Pin_60)
- net A10: now reaches J2.A10
- net A10: now also J3.A10, J4.A10, J5.A10, J6.A10, J7.A10, J8.A10, J9.A10
- net A11: now reaches J2.A11
- net A11: now also J3.A11, J4.A11, J5.A11, J6.A11, J7.A11, J8.A11, J9.A11
- net A12: now reaches J2.A12
- net A12: now also J3.A12, J4.A12, J5.A12, J6.A12, J7.A12, J8.A12, J9.A12
- net A13: now reaches J2.A13
- net A13: now also J3.A13, J4.A13, J5.A13, J6.A13, J7.A13, J8.A13, J9.A13
- net A14: now reaches J2.A14
- net A14: now also J3.A14, J4.A14, J5.A14, J6.A14, J7.A14, J8.A14, J9.A14
- net A15: now reaches J2.A15
- net A15: now also J3.A15, J4.A15, J5.A15, J6.A15, J7.A15, J8.A15, J9.A15
- net A6: now reaches J2.A6
- net A6: now also J3.A6, J4.A6, J5.A6, J6.A6, J7.A6, J8.A6, J9.A6
- net A7: now reaches J2.A7
- net A7: now also J3.A7, J4.A7, J5.A7, J6.A7, J7.A7, J8.A7, J9.A7
- net A8: now reaches J2.A8
- net A8: now also J3.A8, J4.A8, J5.A8, J6.A8, J7.A8, J8.A8, J9.A8
- net A9: now reaches J2.A9
- net A9: now also J3.A9, J4.A9, J5.A9, J6.A9, J7.A9, J8.A9, J9.A9
- net D0: now reaches J2.D0
- net D0: now also J3.D0, J4.D0, J5.D0, J6.D0, J7.D0, J8.D0, J9.D0
- net D1: now reaches J2.D1
- net D1: now also J3.D1, J4.D1, J5.D1, J6.D1, J7.D1, J8.D1, J9.D1
- net D2: now reaches J2.D2
- net D2: now also J3.D2, J4.D2, J5.D2, J6.D2, J7.D2, J8.D2, J9.D2
- net D3: now reaches J2.D3
- net D3: now also J3.D3, J4.D3, J5.D3, J6.D3, J7.D3, J8.D3, J9.D3
- net D4: now reaches J2.D4
- net D4: now also J3.D4, J4.D4, J5.D4, J6.D4, J7.D4, J8.D4, J9.D4
- net D5: now reaches J2.D5
- net D5: now also J3.D5, J4.D5, J5.D5, J6.D5, J7.D5, J8.D5, J9.D5
- net D6: now reaches J2.D6
- net D6: now also J3.D6, J4.D6, J5.D6, J6.D6, J7.D6, J8.D6, J9.D6
- net D7: now reaches J2.D7
- net D7: now also J3.D7, J4.D7, J5.D7, J6.D7, J7.D7, J8.D7, J9.D7
- net IRQ0: now reaches J2.IRQ0
- net IRQ0: now also J3.IRQ0, J4.IRQ0, J5.IRQ0, J6.IRQ0, J7.IRQ0, J8.IRQ0, J9.IRQ0
- net IRQ1: now reaches J2.IRQ1
- net IRQ1: now also J3.IRQ1, J4.IRQ1, J5.IRQ1, J6.IRQ1, J7.IRQ1, J8.IRQ1, J9.IRQ1
- net IRQ2: now reaches J2.IRQ2
- net IRQ2: now also J3.IRQ2, J4.IRQ2, J5.IRQ2, J6.IRQ2, J7.IRQ2, J8.IRQ2, J9.IRQ2
- net IRQ3: now reaches J2.IRQ3
- net IRQ3: now also J3.IRQ3, J4.IRQ3, J5.IRQ3, J6.IRQ3, J7.IRQ3, J8.IRQ3, J9.IRQ3
- net IRQ4: now reaches J2.IRQ4
- net IRQ4: now also J3.IRQ4, J4.IRQ4, J5.IRQ4, J6.IRQ4, J7.IRQ4, J8.IRQ4, J9.IRQ4
- net IRQ5: now reaches J2.IRQ5
- net IRQ5: now also J3.IRQ5, J4.IRQ5, J5.IRQ5, J6.IRQ5, J7.IRQ5, J8.IRQ5, J9.IRQ5
- net IRQ6: now reaches J2.IRQ6
- net IRQ6: now also J3.IRQ6, J4.IRQ6, J5.IRQ6, J6.IRQ6, J7.IRQ6, J8.IRQ6, J9.IRQ6
- net IRQ7: now reaches J2.IRQ7
- net IRQ7: now also J3.IRQ7, J4.IRQ7, J5.IRQ7, J6.IRQ7, J7.IRQ7, J8.IRQ7, J9.IRQ7
- net NMI: now reaches J2.NMI
- net NMI: now also J3.NMI, J4.NMI, J5.NMI, J6.NMI, J7.NMI, J8.NMI, J9.NMI
- net PHI0: now reaches J2.PHI0
- net PHI0: now also J3.PHI0, J4.PHI0, J5.PHI0, J6.PHI0, J7.PHI0, J8.PHI0, J9.PHI0
- net PHI1: now reaches J2.PHI1
- net PHI1: now also J3.PHI1, J4.PHI1, J5.PHI1, J6.PHI1, J7.PHI1, J8.PHI1, J9.PHI1
- net PHI2: now reaches J2.PHI2
- net PHI2: now also J3.PHI2, J4.PHI2, J5.PHI2, J6.PHI2, J7.PHI2, J8.PHI2, J9.PHI2
- net Page_En: now reaches J2.Page_En
- net Page_En: now also J3.Page_En, J4.Page_En, J5.Page_En, J6.Page_En, J7.Page_En, J8.Page_En, J9.Page_En
- net RDY: now reaches J2.RDY
- net RDY: now also J3.RDY, J4.RDY, J5.RDY, J6.RDY, J7.RDY, J8.RDY, J9.RDY
- net RW: now reaches J2.RW
- net RW: now also J3.RW, J4.RW, J5.RW, J6.RW, J7.RW, J8.RW, J9.RW
- net Reset: now reaches J2.Reset
- net Reset: now also J3.Reset, J4.Reset, J5.Reset, J6.Reset, J7.Reset, J8.Reset, J9.Reset
- net Rx: now reaches J2.Rx
- net Rx: now also J3.Rx, J4.Rx, J5.Rx, J6.Rx, J7.Rx, J8.Rx, J9.Rx
- net Sync: now reaches J2.Sync
- net Sync: now also J3.Sync, J4.Sync, J5.Sync, J6.Sync, J7.Sync, J8.Sync, J9.Sync
- net Tx: now reaches J2.Tx
- net Tx: now also J3.Tx, J4.Tx, J5.Tx, J6.Tx, J7.Tx, J8.Tx, J9.Tx
