File: SBC/SBC.sch (KiCad schematic (older format))
At the start: 0 parts

Commit message: Updated SBC...
Parts:
- added C1, C4, C5, C? (x8): C, symbol Device:C
- added C2, C3: CP, symbol Device:CP
- added D1, D2, D3, D4: 1N4148, Diode_THT:D_DO-35_SOD27_P7.62mm_Horizontal, symbol Diode:1N4148
- added D5: LED, symbol Device:LED
- added J1: Jack-DC, symbol Connector:Jack-DC
- added JP1, JP2, JP3, JP6, JP7, JP8: Jumper_2_Bridged, symbol Jumper:Jumper_2_Bridged
- added JP4: Jumper_3_Open, symbol Jumper:Jumper_3_Open
- added JP5: Jumper_2_Open, symbol Jumper:Jumper_2_Open
- added P1: Conn_WallPlug, symbol Connector:Conn_WallPlug
- added R1, R2, R3: 3.3k, symbol Device:R
- added R10, R11, R12, R13, R14, R4, R5, R6, R7, R8, R9: R, symbol Device:R
- added SW1: SW_Push, symbol Switch:SW_Push
- added T1: Transformer_1P_1S, symbol Device:Transformer_1P_1S
- added U1: NE555P, Package_DIP:DIP-8_W7.62mm, symbol Timer:NE555P
- added U2: WD65C02, symbol 65xx:WD65C02
- added U4: 74HC74, symbol 74xx:74HC74
- added U5: 74LS138, symbol 74xx:74LS138
- added U6: L7809, symbol Regulator_Linear:L7809
- added U7, U? (x2): 74HC04, symbol 74xx:74HC04
- added U8: 4071, symbol 4xxx:4071
- added U?: 74LS148, symbol 74xx:74LS148
- added U? (x2): 74HCT574, symbol 74xx:74HCT574
- added U?: 74LS85, symbol 74xx:74LS85
- added X1: ACO-xxxMHz, Oscillator:Oscillator_DIP-14, symbol Oscillator:ACO-xxxMHz
Connections:
- new net: P1.1 (AC_P), T1.1 (AA)
- new net: P1.2 (AC_N), T1.2 (AB)
- new net: D3.2 (A), D4.1 (K), T1.3 (SA)
- new net: D1.1 (K), D2.2 (A), T1.4 (SB)
- new net: C3.1, D2.1 (K), D4.2 (A), JP4.3 (B)
- new net: J1.1, JP4.1 (A)
- new net: C4.1, JP4.2 (C), JP5.1 (A), U6.1 (IN)
- new net: JP3.2 (B), U2.1 (~VP)
- new net: D5.2 (A), R6.2
- new net: JP2.2 (B), R2.1, U2.4 (~IRQ)
- new net: JP1.2 (B), R3.1, U2.6 (~NMI)
- new net: U5.10 (O5), U8.1, U8.5
- new net: U7.2, U8.6
- new net: C1.1, SW1.1, U1.2 (TR)
- new net: U1.3 (Q), U?.3
- new net: C2.1, R4.2, U1.6 (THR), U1.7 (DIS)
- new net: U4.11 (C), U4.2 (D), U4.6 (~Q)
- new net: U4.12 (D), U4.8 (~Q)
- new net: U?.14 (GS), U?.15 (A3), U?.6 (D4)
- new net: U?.13 (A2), U?.5 (D3), U?.6 (S2)
- new net: U?.12 (A1), U?.4 (D2), U?.7 (S1)
- new net: U?.10 (A0), U?.3 (D1), U?.9 (S0)
- new net: U?.1 (B3), U?.16 (Q3)
- new net: U?.14 (B2), U?.17 (Q2)
- new net: U?.11 (B1), U?.18 (Q1)
- new net: U?.19 (Q0), U?.9 (B0)
- new net: U?.5, U?.7 (Oa<b)
- new net A0: U2.9 (A0)
- new net A1: U2.10 (A1)
- new net A10: U2.19 (A10)
- new net A11: U2.20 (A11)
- new net A12: U2.22 (A12), U5.1 (A0)
- new net A13: U2.23 (A13), U5.2 (A1)
- new net A14: U2.24 (A14), U5.3 (A2)
- new net A15: U2.25 (A15), U5.6 (E3)
- new net A2: U2.11 (A2)
- new net A3: U2.12 (A3)
- new net A4: U2.13 (A4)
- new net A5: U2.14 (A5)
- new net A6: U2.15 (A6)
- new net A7: U2.16 (A7)
- new net A8: U2.17 (A8)
- new net A9: U2.18 (A9)
- new net CLK: JP6.2 (B), JP7.2 (B), JP8.2 (B), U2.37 (PHI2)
- new net CLK1: JP6.1 (A), U4.3 (C), X1.8 (OUT)
- new net CLK2: JP7.1 (A), U4.5 (Q)
- new net CLK3: JP8.1 (A)
- new net CLK4: U4.9 (Q)
- new net CS_RD: U8.4, U?.1 (OE)
- new net CS_WR: U8.3, U?.11 (Cp)
- new net D0: U2.33 (D0), U?.19 (Q0), U?.2 (D0)
- new net D1: U2.32 (D1), U?.18 (Q1), U?.3 (D1)
- new net D2: U2.31 (D2), U?.17 (Q2), U?.4 (D2)
- new net D3: U2.30 (D3), U?.16 (Q3), U?.5 (D3)
- new net D4: U2.29 (D4), U?.15 (Q4), U?.6 (D4)
- new net D5: U2.28 (D5), U?.14 (Q5), U?.7 (D5)
- new net D6: U2.27 (D6), U?.13 (Q6), U?.8 (D6)
- new net D7: U2.26 (D7), U?.12 (Q7), U?.9 (D7)
- new net GND: C1.2, C2.2, C3.2, C4.2, C5.2, C?.1, C?.1, C?.1, C?.1, C?.2, C?.2, C?.2, C?.2, D1.2 (A), D3.1 (K), D5.1 (K), J1.2, JP3.1 (A), SW1.2, U1.1 (GND), U2.21 (GND), U4.7 (GND), U5.4 (E1), U5.5 (E2), U5.8 (GND), U6.2 (GND), U?.1 (OE), U?.10 (GND), U?.10 (GND), U?.2 (D0), U?.5 (EI), U?.7 (D5), U?.8 (D6), U?.8 (GND), U?.9 (D7), X1.7 (GND)
- new net IRQ: JP2.1 (A), U?.6
- new net IRQ0: R14.2, U?.10 (IO)
- new net IRQ1: R13.2, U?.11 (I1)
- new net IRQ2: R12.2, U?.12 (I2)
- new net IRQ3: R11.2, U?.13 (I3)
- new net IRQ4: R10.2, U?.1 (I4)
- new net IRQ5: R9.2, U?.2 (I5)
- new net IRQ6: R8.2, U?.3 (I6)
- new net IRQ7: R7.2, U?.4 (I7)
- new net NMI: JP1.1 (A)
- new net PHI1: U2.3 (PHI1out)
- new net PHI2: U?.11 (Cp)
- new net RDY: R1.1, U2.2 (RDY)
- new net RESET: R5.1, U?.4
- new net RW: U2.34 (R/~W), U7.1, U8.2
- new net SYNC: U2.7 (SYNC)
- new net VCC: C5.1, C?.1, C?.1, C?.1, C?.1, C?.2, C?.2, C?.2, C?.2, JP5.2 (B), R1.2, R10.1, R11.1, R12.1, R13.1, R14.1, R2.2, R3.2, R4.1, R5.2, R6.1, R7.1, R8.1, R9.1, U1.4 (R), U1.8 (VCC), U2.38 (~SO), U2.8 (VCC), U4.1 (~R), U4.10 (~S), U4.13 (~R), U4.14 (VCC), U4.4 (~S), U6.3 (OUT), U?.15 (EO), U?.16 (VCC), U?.16 (VCC), U?.20 (VCC), U?.20 (VCC), X1.14 (Vcc)
- no-connect marks 0 -> 20
Other:
- note added: "6502 CPU"
- note added: "Chip Select - Read/Write"
- note added: "Clock and clock divider"
- note added: "IRQ Priority and handling registers"
- note added: "Power Supply"
- note added: "Reset and Power-On-Reset"

Commit message: Updated SBC...
Parts:
- removed U6: L7809, symbol Regulator_Linear:L7809
- removed U7, U? (x2): 74HC04, symbol 74xx:74HC04
- added J2: GPIO_Connector, Connector_PinHeader_2.54mm:PinHeader_2x03_P2.54mm_Vertical, symbol PC:GPIO_Connector
- added J3, J4: DB9_Male, Connector_Dsub:DSUB-9_Female_Horizontal_P2.77x2.54mm_EdgePinOffset9.40mm, symbol Connector:DB9_Male
- added JP10: Jumper_2_Bridged, Connector_PinHeader_2.54mm:PinHeader_1x02_P2.54mm_Vertical, symbol Jumper:Jumper_2_Bridged
- added JP11: Jumper_2_Open, Connector_PinHeader_2.54mm:PinHeader_1x02_P2.54mm_Vertical, symbol Jumper:Jumper_2_Open
- added JP9: Jumper_3_Bridged12, Connector_PinHeader_2.54mm:PinHeader_1x03_P2.54mm_Vertical, symbol Jumper:Jumper_3_Bridged12
- added R15, R16: R, Resistor_THT:R_Axial_DIN0204_L3.6mm_D1.6mm_P5.08mm_Horizontal, symbol Device:R
- added U1: WD65C22, symbol 65xx:WD65C22
- added U10, U21: 74LS08, symbol 74xx:74LS08
- added U12, U22: W65C51N, symbol 65xx:W65C51N
- added U13, U23, U5: 74LS138, symbol 74xx:74LS138
- added U16, U25, U8: 74LS21, symbol 74xx:74LS21
- added U17, U20, U27, U4: 74HCT04, symbol 74xx:74HCT04
- added U24: 28C256, symbol Memory_EEPROM:28C256
- added U26: 74HCT00, symbol 74xx:74HCT00
- added U9: L7805, symbol Regulator_Linear:L7805
- C1: footprint (none) -> Capacitor_THT:C_Disc_D3.4mm_W2.1mm_P2.50mm
- C10, C11, C12, C13, C2, C5, C6, C9: renamed from C?; footprint (none) -> Capacitor_THT:C_Disc_D3.4mm_W2.1mm_P2.50mm
- C3: renamed from C2; footprint (none) -> Capacitor_THT:CP_Radial_D5.0mm_P2.50mm
- C4: renamed from C3; footprint (none) -> Capacitor_THT:CP_Radial_D5.0mm_P2.50mm
- C7: renamed from C4; footprint (none) -> Capacitor_THT:C_Disc_D3.4mm_W2.1mm_P2.50mm
- C8: renamed from C5; footprint (none) -> Capacitor_THT:C_Disc_D3.4mm_W2.1mm_P2.50mm
- JP1, JP2, JP3, JP5, JP6, JP7, JP8: footprint (none) -> Connector_PinHeader_2.54mm:PinHeader_1x02_P2.54mm_Vertical
- JP4: footprint (none) -> Connector_PinHeader_2.54mm:PinHeader_1x03_P2.54mm_Vertical
- R1, R10, R11, R12, R13, R14, R2, R3, R4, R5, R6, R7, R8, R9: footprint (none) -> Resistor_THT:R_Axial_DIN0204_L3.6mm_D1.6mm_P5.08mm_Horizontal
- SW1: footprint (none) -> Button_Switch_THT:SW_PUSH_6mm
- gave numbers to parts that had none: 4
- renumbered U8 to U11, U1 to U2, U2 to U3, U4 to U6, U5 to U7
Connections:
- net A0: now also U1.38 (RS0), U12.13 (RS0), U22.13 (RS0), U24.10 (A0)
- net A1: now also U1.37 (RS1), U12.14 (RS1), U22.14 (RS1), U24.9 (A1)
- net A10: now also U24.21 (A10)
- net A11: now also U24.23 (A11)
- net A12: now also U13.1 (A0), U23.1 (A0), U24.2 (A12), U5.1 (A0)
- net A13: now also U13.2 (A1), U23.2 (A1), U24.26 (A13), U26.4, U5.2 (A1)
- net A14: now also U13.3 (A2), U23.3 (A2), U24.1 (A14), U26.10, U5.3 (A2)
- net A15: now also U13.6 (E3), U23.6 (E3), U26.9, U5.6 (E3)
- net A2: now also U1.36 (RS2), U16.9, U24.8 (A2), U8.9
- net A3: now also U1.35 (RS3), U17.1, U24.7 (A3), U27.1
- net A4: now also U10.4, U24.6 (A4), U27.3, U8.12
- net A5: now also U10.5, U16.13, U17.3, U24.5 (A5)
- net A6: now also U17.5, U24.4 (A6), U27.5, U4.1
- net A7: now also U17.9, U24.3 (A7), U27.9, U4.3
- net A8: now also U17.11, U20.11, U24.25 (A8), U4.5
- net A9: now also U17.13, U20.13, U24.24 (A9), U4.9
- net D0: now also U1.33 (D0), U12.18 (D0), U22.18 (D0), U24.11 (D0)
- net D1: now also U1.32 (D1), U12.19 (D1), U22.19 (D1), U24.12 (D1)
- net D2: now also U1.31 (D2), U12.20 (D2), U22.20 (D2), U24.13 (D2)
- net D3: now also U1.30 (D3), U12.21 (D3), U22.21 (D3), U24.15 (D3)
- net D4: now also U1.29 (D4), U12.22 (D4), U22.22 (D4), U24.16 (D4)
- net D5: now also U1.28 (D5), U12.23 (D5), U22.23 (D5), U24.17 (D5)
- net D6: now also U1.27 (D6), U12.24 (D6), U22.24 (D6), U24.18 (D6)
- net D7: now also U1.26 (D7), U12.25 (D7), U22.25 (D7), U24.19 (D7)
- net GND: now also U18.8 (GND), J3.5, J3.9, J4.5, J4.9, R16.1, U1.1 (GND), U12.1 (GND), U13.4 (E1), U13.5 (E2), U13.8 (GND), U22.1 (GND), U23.4 (E1), U23.5 (E2), U23.8 (GND), U24.14 (GND), U26.7 (GND), U4.7 (GND), U5.4 (E1), U5.5 (E2), U5.8 (GND), U9.2 (GND)
- net IRQ: now also U20.8
- net IRQ0: now also U12.26 (~IRQ)
- net IRQ1: now also U22.26 (~IRQ)
- net NMI: now also U1.21 (~IRQ)
- net PHI2: now also U3.39 (PHI2out), U1.25 (PHI2), U12.27 (PHI2), U22.27 (PHI2)
- net RESET: now also U3.40 (~RESET), U1.34 (~RESET), U12.4 (~RESET), U22.4 (~RESET), U4.12
- net RW: now also U1.22 (R/~W), U12.28 (R/~W), U22.28 (R/~W), U4.11
- net VCC: now also R15.2, U1.20 (VCC), U12.15 (VCC), U13.16 (VCC), U22.15 (VCC), U23.16 (VCC), U24.28 (VCC), U26.14 (VCC), U4.14 (VCC), U5.16 (VCC), U9.3 (OUT)
- net at C7.1, JP4.2 (C), JP5.1 (A): now also U9.1 (IN)
- net at U11.6: now also U4.10
- net at U2.3 (Q): now also U4.13
- net at U18.7 (Oa<b): now also U20.9
- new net: R15.1, U24.27 (~WE)
- new net: U20.2, U26.1
- new net: U20.4, U26.2
- new net: JP9.1 (A), U26.3
- new net: U20.6, U26.5
- new net: JP9.3 (B), U20.1, U26.6
- new net: U20.5, U26.8
- new net: JP10.2 (B), R16.2
- new net: U1.23 (~CS2), U5.10 (O5)
- new net: U4.2, U8.1
- new net: U4.4, U8.2
- new net: U4.6, U8.4
- new net: U4.8, U8.5
- new net: U10.1, U8.6
- new net: U10.2, U10.6
- new net: J3.3, U12.10 (Tx_Data)
- new net: J3.4, U12.11 (~DTR)
- new net: J3.2, U12.12 (Rx_Data)
- new net: J3.1, U12.16 (~DCD)
- new net: J3.6, U12.17 (~DSR)
- new net: U12.3 (~CS1), U13.10 (O5)
- new net: J3.7, U12.8 (~RTS)
- new net: J3.8, U12.9 (~CTS)
- new net: U10.10, U16.6
- new net: U10.9, U8.8
- new net: U16.1, U17.6
- new net: U16.2, U17.8
- new net: U16.4, U17.10
- new net: U16.5, U17.12
- new net: U17.2, U8.10
- new net: U17.4, U8.13
- new net: J4.3, U22.10 (Tx_Data)
- new net: J4.4, U22.11 (~DTR)
- new net: J4.2, U22.12 (Rx_Data)
- new net: J4.1, U22.16 (~DCD)
- new net: J4.6, U22.17 (~DSR)
- new net: U22.3 (~CS1), U23.10 (O5)
- new net: J4.7, U22.8 (~RTS)
- new net: J4.8, U22.9 (~CTS)
- new net: U21.10, U25.6
- new net: U16.8, U21.9
- new net: U25.1, U27.6
- new net: U25.2, U27.8
- new net: U20.10, U25.4
- new net: U20.12, U25.5
- new net: U16.10, U27.2
- new net: U16.12, U27.4
- new net CA1: J2.17 (Pin_17), U1.40 (CA1)
- new net CA2: J2.18 (Pin_18), U1.39 (CA2)
- new net CB1: J2.19 (Pin_19), U1.18 (CB1)
- new net CB2: J2.20 (Pin_20), U1.19 (CB2)
- new net CS: JP9.2 (C), U24.20 (~CS), U24.22 (~OE)
- new net CS_COM1: U10.8, U12.2 (CS0)
- new net CS_COM2: U21.8, U22.2 (CS0)
- new net CS_GPIO: U1.24 (CS1), U10.3
- new net GPIO0: J2.1 (Pin_1), U1.2 (PA0)
- new net GPIO1: J2.2 (Pin_2), U1.3 (PA1)
- new net GPIO10: J2.11 (Pin_11), U1.12 (PB2)
- new net GPIO11: J2.12 (Pin_12), U1.13 (PB3)
- new net GPIO12: J2.13 (Pin_13), U1.14 (PB4)
- new net GPIO13: J2.14 (Pin_14), U1.15 (PB5)
- new net GPIO14: J2.15 (Pin_15), U1.16 (PB6)
- new net GPIO15: J2.16 (Pin_16), U1.17 (PB7)
- new net GPIO2: J2.3 (Pin_3), U1.4 (PA2)
- new net GPIO3: J2.4 (Pin_4), U1.5 (PA3)
- new net GPIO4: J2.5 (Pin_5), U1.6 (PA4)
- new net GPIO5: J2.6 (Pin_6), U1.7 (PA5)
- new net GPIO6: J2.7 (Pin_7), U1.8 (PA6)
- new net GPIO7: J2.8 (Pin_8), U1.9 (PA7)
- new net GPIO8: J2.9 (Pin_9), U1.10 (PB0)
- new net GPIO9: J2.10 (Pin_10), U1.11 (PB1)
- new net PAGE_EN: JP11.2 (B)
- new net PG: JP10.1 (A), JP11.1 (A), U20.3
- no-connect marks 20 -> 43
Other:
- note added: "6522 GPIO Connector"
- note added: "COM (Serial) Ports and handling circuitry"
- note added: "Read-Only Memory"
- moved on the sheet: C1, C10, C11, C12, C13, C2, C3, C4, C5, C6, C7, C8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
