File: Motherboard/Motherboard.sch (KiCad schematic (older format))
At the start: 110 parts, among them J1 Jack-DC_15v, J2 GPIO_Connector, J3 DB9_Male, J4 Expansion_Connector, J5 Expansion_Connector, J6 Expansion_Connector, J7 65SIB_Connector, J8 Expansion_Connector, J9 Expansion_Connector, P1 Conn_WallPlug, Q1 TIC106, Q2 2N3055, SW1 RESET, SW2 SW_Push, SW3 SW_DPDT_x2, T1 Transformer_1P_1S_240v-16v, U1 WD65C22, U10 74LS138, U11 74LS21, U12 LM7912_TO220, U13 LM7812_TO220, U14 74LS08, U16 74LS21, U17 W65C51N, U18 74LS138, U19 74LS148, U2 NE555P, U20 74HCT574, U21 74HCT04, U22 74LS85, U23 74HCT574, U24 74HCT04, U25 MAX235, U26 28C256, U27 74HCT00, U28 74LS138, U29 74HCT04, U3 74HCT04, U30 HM62256BLP, U31 74LS138, U32 74LS08, U33 74HCT00, U34 74LS08, U35 WD65C22, U36 74LS138, U37 74HCT541, U38 28C256, U39 74LS138, U4 WD65C02, U5 74LS138, U6 74LS08, U7 LM386, U8 74HC74, U9 LM7805_TO220, X1 ACO-2MHz, X2 ACO-1.8432MHz

Commit message: Updated schematic...
Parts:
- R10: value R -> 150
- R11: value R -> 560
Changed lines of the file:
@@
-$EndComp
-$Comp
-L Generic_Device:R R11
-U 1 1 62934453
-P 7800 2450
-F 0 "R11" H 7870 2496 50  0000 L CNN
-F 1 "R" H 7870 2405 50  0000 L CNN
-F 2 "" V 7730 2450 50  0001 C CNN
-F 3 "~" H 7800 2450 50  0001 C CNN
-	1    7800 2450
-	1    0    0    -1
 $EndComp
 $Comp
@@
 P 7050 2450
 F 0 "R10" H 7120 2496 50  0000 L CNN
-F 1 "R" H 7120 2405 50  0000 L CNN
+F 1 "150" H 7120 2405 50  0000 L CNN
 F 2 "" V 6980 2450 50  0001 C CNN
 F 3 "~" H 7050 2450 50  0001 C CNN
@@
 Text GLabel 15450 4500 0    50   Input ~ 0
 ROM_EN
+$Comp
+L Generic_Device:R R11
+U 1 1 62934453
+P 7800 2450
+F 0 "R11" H 7870 2496 50  0000 L CNN
+F 1 "560" H 7870 2405 50  0000 L CNN
+F 2 "" V 7730 2450 50  0001 C CNN
+F 3 "~" H 7800 2450 50  0001 C CNN
+	1    7800 2450
+	1    0    0    -1
+$EndComp
 $EndSCHEMATC

Commit message: Completed 65SIB address decoding and added annotations for parts...
Parts:
- removed U39: 74LS138, symbol 74xx:74LS138
- added unit 3 of U14
- added unit 2 of U19
- added unit 5 of U23
- added unit 6 of U23
- added unit 2 of U27
- added unit 3 of U27
- added unit 1 of U27
- added U30: 74HCT04, symbol 74xx:74HCT04
- added U31: 74LS21, symbol 74xx:74LS21
- JP1, JP2, JP3, JP5, JP6, JP7: footprint (none) -> Connector_PinHeader_2.54mm:PinHeader_1x02_P2.54mm_Vertical
- JP10: renamed from JP12; footprint (none) -> Connector_PinHeader_2.54mm:PinHeader_1x03_P2.54mm_Vertical
- JP11: renamed from JP13; footprint (none) -> Connector_PinHeader_2.54mm:PinHeader_1x03_P2.54mm_Vertical
- JP12: renamed from JP14; footprint (none) -> Connector_PinHeader_2.54mm:PinHeader_1x03_P2.54mm_Vertical
- JP13: renamed from JP15; footprint (none) -> Connector_PinHeader_2.54mm:PinHeader_1x03_P2.54mm_Vertical
- JP14: renamed from JP16; footprint (none) -> Connector_PinHeader_2.54mm:PinHeader_1x03_P2.54mm_Vertical
- JP15: renamed from JP17; footprint (none) -> Connector_PinHeader_2.54mm:PinHeader_1x03_P2.54mm_Vertical
- JP16: renamed from JP18; footprint (none) -> Connector_PinHeader_2.54mm:PinHeader_1x03_P2.54mm_Vertical
- JP4, JP8: footprint (none) -> Connector_PinHeader_2.54mm:PinHeader_1x03_P2.54mm_Vertical
- JP9: renamed from JP11; footprint (none) -> Connector_PinHeader_2.54mm:PinHeader_1x03_P2.54mm_Vertical
- Q1, U12, U13: footprint (none) -> Package_TO_SOT_THT:TO-220-3_Horizontal_TabDown
- Q2: footprint (none) -> Package_TO_SOT_THT:TO-3
- R1, R10, R11, R12, R13, R14, R15, R16, R17, R18, R19, R2, R20, R21, R3, R4, R5, R6, R7, R8, R9: footprint (none) -> Resistor_THT:R_Axial_DIN0207_L6.3mm_D2.5mm_P7.62mm_Horizontal
- SW1, SW2: footprint (none) -> Button_Switch_THT:SW_PUSH_6mm_H4.3mm
- SW3: value SW_DPDT_x2 -> SW_SPDT; footprint (none) -> Button_Switch_THT:SW_Slide_1P2T_CK_OS102011MS2Q; symbol Switch:SW_DPDT_x2 -> Switch:SW_SPDT
- U1: footprint (none) -> Package_DIP:DIP-40_W15.24mm_LongPads
- U2: footprint (none) -> Package_DIP:DIP-8_W7.62mm_LongPads
- U25: renamed from U26; footprint (none) -> Package_DIP:DIP-28_W15.24mm_Socket_LongPads
- U28: footprint (none) -> Package_DIP:DIP-16_W7.62mm_Socket_LongPads
- U29: renamed from U30; footprint Package_DIP:DIP-28_W7.62mm_Socket_LongPads -> Package_DIP:DIP-28_W15.24mm_LongPads
- U3: renamed from U4; footprint (none) -> Package_DIP:DIP-40_W15.24mm_LongPads
- U36: renamed from U35; footprint (none) -> Package_DIP:DIP-28_W15.24mm_Socket_LongPads
- U37: renamed from U36; footprint (none) -> Package_DIP:DIP-16_W7.62mm_Socket_LongPads
- U40: renamed from U38; footprint (none) -> Package_DIP:DIP-28_W15.24mm_Socket_LongPads
- U6: renamed from U7; footprint (none) -> Package_DIP:DIP-8_W7.62mm_LongPads
- U7: renamed from U9; footprint (none) -> Package_TO_SOT_THT:TO-220-3_Horizontal_TabDown
- X1, X2: footprint (none) -> Oscillator:Oscillator_DIP-14_LargePads
- renumbered C4 to C2, C10 to C3, C12 to C4, C13 to C5, C14 to C6, C15 to C7, C16 to C8, J8 to J7, J7 to J8, U11 to U10, U6 to U11, U17 to U15, U18 to U16, U19 to U17, U20 to U18, U16 to U19, U21 to U20, U22 to U21, U23 to U22, U24 to U23, U25 to U24, U27 to U26, U24 to U27, U29 to U27, U31 to U32, U32 to U33, U14 to U33, U33 to U34, U34 to U35, U32 to U35, U29 to U38, U37 to U39, U3 to U4, U10 to U9
Connections:
- wire segments 481 -> 503
- no-connect marks 53 -> 64
Other:
- note added: "65SIB ports"
- note added: "Address space: 0xD040 - 0xD04F"
- note added: "IRQ2"
- note added: "IRQ3-7"
- note removed: "IRQ2-7"
- note removed: "TODO: Finish address decoding for 6522"
- note removed: "TODO: Write code for EEPROM and Software-side."
- moved on the sheet: J8

Commit message: Finished routing and placement...
Parts:
- removed T1: Transformer_1P_1S_240v-16v, symbol Device:Transformer_1P_1S
- removed unit 1 of U10
- removed unit 1 of U11
- removed unit 2 of U11
- removed unit 1 of U4
- removed unit 2 of U4
- removed unit 3 of U4
- removed unit 4 of U4
- added R22: 3.3k Ω, Resistor_THT:R_Axial_DIN0207_L6.3mm_D2.5mm_P7.62mm_Horizontal, symbol Device:R
- added TR1: Transformer, Transformer_THT:Transformer_CHK_EI48-8VA_2xSec, symbol PC:Transformer
- added unit 5 of U14
- added unit 7 of U15
- added unit 6 of U15
- added unit 5 of U18
- added unit 3 of U18
- added unit 2 of U23
- added unit 3 of U23
- added unit 5 of U23
- added unit 7 of U23
- added unit 3 of U24
- added unit 5 of U3
- added unit 7 of U31
- added U32: 74HCT04, Package_DIP:DIP-14_W7.62mm_Socket_LongPads, symbol 74xx:74HCT04
- added unit 3 of U35
- added unit 1 of U36
- added unit 4 of U36
- added unit 7 of U36
- added U37: 74LS21, Package_DIP:DIP-14_W7.62mm_Socket_LongPads, symbol 74xx:74LS21
- added unit 7 of U38
- added unit 5 of U40
- added unit 5 of U6
- added unit 7 of U7
- added unit 5 of U8
- C1: renamed from C5; value C -> 0.33 uF; footprint (none) -> Capacitor_THT:C_Disc_D3.0mm_W1.6mm_P2.50mm
- C2: renamed from C7; value C -> 0.1 uF; footprint (none) -> Capacitor_THT:C_Disc_D3.0mm_W1.6mm_P2.50mm
- C3: renamed from C4; value C -> 0.33 uF; footprint (none) -> Capacitor_THT:C_Disc_D3.0mm_W1.6mm_P2.50mm
- C4: renamed from C3; value C -> 0.33 uF; footprint (none) -> Capacitor_THT:C_Disc_D3.0mm_W1.6mm_P2.50mm
- C5: renamed from C6; value C -> 25 uF; footprint (none) -> Capacitor_THT:CP_Radial_D5.0mm_P2.50mm; symbol Generic_Device:C -> Generic_Device:CP
- C6: renamed from C8; value C -> 25 uF; footprint (none) -> Capacitor_THT:CP_Radial_D5.0mm_P2.50mm; symbol Generic_Device:C -> Generic_Device:CP
- C7: renamed from C1; footprint (none) -> Capacitor_THT:C_Disc_D3.0mm_W1.6mm_P2.50mm
- C8: renamed from C2; footprint (none) -> Capacitor_THT:C_Disc_D3.0mm_W1.6mm_P2.50mm
- CP1: renamed from CP2; footprint (none) -> Capacitor_THT:CP_Radial_D5.0mm_P2.50mm
- CP2: renamed from CP1; footprint (none) -> Capacitor_THT:CP_Radial_D5.0mm_P2.50mm
- D1: renamed from D2; footprint (none) -> Diode_THT:D_DO-41_SOD81_P7.62mm_Horizontal
- D2: renamed from D1; footprint (none) -> Diode_THT:D_DO-41_SOD81_P7.62mm_Horizontal
- D3: renamed from D4; footprint (none) -> Diode_THT:D_DO-41_SOD81_P7.62mm_Horizontal
- D4: renamed from D3; footprint (none) -> Diode_THT:D_DO-41_SOD81_P7.62mm_Horizontal
- D5: value LED_5v -> 5v INDICATOR
- D6: value LED_12v -> 12v INDICATOR
- D7: value LED_-12v -> -12v INDICATOR
- J1: value Jack-DC_15v -> Jack-DC_18v
- J3: value DB9_Male -> DB9_Header; footprint Connector_PinHeader_2.54mm:PinHeader_2x05_P2.54mm_Vertical -> PC:DB9_Header
- J4: renamed from J2; footprint Connector_PinSocket_2.54mm:PinSocket_2x10_P2.54mm_Vertical -> Connector_PinSocket_2.54mm:PinSocket_2x11_P2.54mm_Vertical
- JP1: renamed from JP8; value Jumper_3_Bridged12 -> PAGE_EN
- JP12: renamed from JP13; value Jumper_3_Bridged12 -> CS1
- JP13: renamed from JP5; value Jumper_2_Bridged -> CLK/1
- JP14: renamed from JP6; value Jumper_2_Bridged -> CLK/2
- JP15: renamed from JP7; value Jumper_2_Bridged -> CLK/4
- JP16: renamed from JP4; value Jumper_3_Bridged12 -> NMI/IRQ1
- JP2: renamed from JP10; value Jumper_3_Bridged12 -> CS6
- JP3: renamed from JP14; value Jumper_3_Bridged12 -> CS7
- JP4: renamed from JP11; value Jumper_3_Bridged12 -> CS4
- JP5: renamed from JP15; value Jumper_3_Bridged12 -> CS5
- JP6: renamed from JP12; value Jumper_3_Bridged12 -> CS2
- JP7: renamed from JP16; value Jumper_3_Bridged12 -> CS3
- JP8: renamed from JP9; value Jumper_3_Bridged12 -> CS0
- P1: value Conn_WallPlug -> POWER TERMINAL
- R1: renamed from R13; value R -> 4.7k Ω
- R10: renamed from R11; value 560 -> 560 Ω
- R11: renamed from R12; value Ω -> 560 Ω
- R16: renamed from R21; value R -> 3.3k Ω
- R2: renamed from R14; value R -> 4.7k Ω
- R3: renamed from R15; value R -> 4.7k Ω
- R4: renamed from R16; value R -> 4.7k Ω
- R5: renamed from R17; value R -> 4.7k Ω
- R6: renamed from R18; value R -> 4.7k Ω
- R7: renamed from R19; value R -> 4.7k Ω
- R8: renamed from R20; value R -> 4.7k Ω
- R9: renamed from R10; value 150 -> 150 Ω
- SW1: renamed from SW3; value SW_SPDT -> POWER SELECT
- SW2: value SW_Push -> FUSE RESET
- SW3: renamed from SW1; value RESET -> PROCESSOR RESET
- U10: renamed from U39; footprint (none) -> Package_DIP:DIP-20_W7.62mm_Socket_LongPads
- U11: renamed from U25; footprint Package_DIP:DIP-28_W15.24mm_Socket_LongPads -> Socket:DIP_Socket-28_W11.9_W12.7_W15.24_W17.78_W18.5_3M_228-1277-00-0602J
- U14, U6: renamed from U26; footprint (none) -> Package_DIP:DIP-14_W7.62mm_Socket_LongPads
- U14, U6: renamed from U34; footprint (none) -> Package_DIP:DIP-14_W7.62mm_Socket_LongPads
- U15, U23: renamed from U4; footprint (none) -> Package_DIP:DIP-14_W7.62mm_Socket_LongPads
- U15, U23, U36, U43, U7: renamed from U20; footprint (none) -> Package_DIP:DIP-14_W7.62mm_Socket_LongPads
- U15, U36, U38, U7: renamed from U27; footprint (none) -> Package_DIP:DIP-14_W7.62mm_Socket_LongPads
- U15: renamed from U38; footprint (none) -> Package_DIP:DIP-14_W7.62mm_Socket_LongPads
- U16: renamed from U18; footprint (none) -> Package_DIP:DIP-20_W7.62mm_Socket_LongPads
- U17: renamed from U22; footprint (none) -> Package_DIP:DIP-20_W7.62mm_Socket_LongPads
- U18, U40: renamed from U14; footprint (none) -> Package_DIP:DIP-14_W7.62mm_Socket_LongPads
- U19: renamed from U40; footprint Package_DIP:DIP-28_W15.24mm_Socket_LongPads -> Socket:DIP_Socket-28_W11.9_W12.7_W15.24_W17.78_W18.5_3M_228-1277-00-0602J
- U20: renamed from U9; footprint (none) -> Package_DIP:DIP-16_W7.62mm_Socket_LongPads
- U22: renamed from U32; footprint (none) -> Package_DIP:DIP-16_W7.62mm_Socket_LongPads
- U23: footprint (none) -> Package_DIP:DIP-14_W7.62mm_Socket_LongPads
- U24: renamed from U8; footprint (none) -> Package_DIP:DIP-14_W7.62mm_Socket_LongPads
- U25: renamed from U15; footprint (none) -> Package_DIP:DIP-28_W15.24mm_Socket_LongPads
- U29: renamed from U24; footprint (none) -> Package_DIP:DIP-24_W15.24mm_Socket_LongPads
- U3, U8: renamed from U33; footprint (none) -> Package_DIP:DIP-14_W7.62mm_Socket_LongPads
- U3, U42: renamed from U11; footprint (none) -> Package_DIP:DIP-14_W7.62mm_Socket_LongPads
- U3, U8: renamed from U35; footprint (none) -> Package_DIP:DIP-14_W7.62mm_Socket_LongPads
- U31, U38: renamed from U30; footprint (none) -> Package_DIP:DIP-14_W7.62mm_Socket_LongPads
- U34: renamed from U16; footprint (none) -> Package_DIP:DIP-16_W7.62mm_Socket_LongPads
- U35, U39: renamed from U19; footprint (none) -> Package_DIP:DIP-14_W7.62mm_Socket_LongPads
- U35: renamed from U31; footprint (none) -> Package_DIP:DIP-14_W7.62mm_Socket_LongPads
- U36, U7: renamed from U23; footprint (none) -> Package_DIP:DIP-14_W7.62mm_Socket_LongPads
- U39: renamed from U10; footprint (none) -> Package_DIP:DIP-14_W7.62mm_Socket_LongPads
- U4: renamed from U17; footprint (none) -> Package_DIP:DIP-16_W7.62mm_Socket_LongPads
- U41: renamed from U5; footprint (none) -> Package_DIP:DIP-16_W7.62mm_Socket_LongPads
- U5: renamed from U21; footprint (none) -> Package_DIP:DIP-16_W7.62mm_Socket_LongPads
- X1: value ACO-2MHz -> ACO-8MHz
- renumbered J8 to J2, J4 to J5, J5 to J6, J6 to J7, J7 to J8, JP2 to JP10, JP3 to JP11, JP1 to JP9, Q2 to Q1, Q1 to Q2, R6 to R12, R9 to R13, R8 to R14, R5 to R15, R2 to R17, R3 to R18, R4 to R19, R1 to R20, R7 to R21, U13 to U1, U6 to U12, U12 to U13, U7 to U2, U3 to U21, U2 to U26, U36 to U27, U37 to U30, U1 to U33, U29 to U9
Connections:
- net +12v: now also C4.1, U2.1 (VI)
- net -12v: now also C6.2; no longer C6.1
- net A10: now also U23.11
- net A11: now also U15.13
- net A4: now also U37.9
- net A5: now also U37.10
- net A6: now also U36.1
- net A7: now also U23.3
- net A8: now also U23.5
- net A9: now also U36.9
- net CS_GPIO: now also U18.8
- net GND: now also C5.1, C6.1, J4.1 (Pin_1), J4.22 (Pin_22), U20.16 (VCC), U29.12 (VCC), R22.2, U14.14 (VCC), U14.7 (GND), U15.14 (VCC), U15.7 (GND), U18.14 (VCC), U18.7 (GND), U23.14 (VCC), U23.7 (GND), U24.14 (VCC), U24.7 (GND), U3.14 (VCC), U3.7 (GND), U31.14 (VCC), U31.7 (GND), U35.14 (VCC), U35.7 (GND), U36.14 (VCC), U36.7 (GND), U37.14 (VCC), U37.7 (GND), U38.14 (VCC), U38.7 (GND), U40.14 (VCC), U40.7 (GND), U6.14 (VCC), U6.7 (GND), U7.14 (VCC), U7.7 (GND), U8.14 (VCC), U8.7 (GND); no longer C5.2, C6.2, U19.27 (~WE)
- net RESET\: now also U23.2; no longer U23.12
- net RW: now also U15.3; no longer U15.11
- net at P1.1 (AC_P): now also TR1.6
- net at P1.2 (AC_N): now also TR1.1
- net at D3.2 (A), D4.1 (K): now also TR1.8
- net at D1.2 (A), D2.1 (K): now also TR1.7
- net at U26.3 (Q): now also U23.1; no longer U23.13
- net at U18.5: now also U15.4; no longer U15.10
- net CS1_COM\: now reaches U25.3 (~CS1), U34.10 (O5)
- net at U29.20 (En\): now also U32.4
- net at R13.2, U12.5, U13.2 (VI): now also C5.2; no longer C5.1
- net 15v_UNREG renamed FUSE_OUT
- net FUSE_OUT: no longer C4.1, U2.1 (VI)
- net 65SIB_E2\ renamed 65SIB_CS2\
- net 65SIB_E3 renamed 65SIB_CS3
- net CS_COM renamed CS0_COM
- net CS0_COM: now also U32.3
- new net: R22.1, U19.27 (~WE)
- new net: U18.10, U37.6
- new net: U18.9, U37.8
- new net: U23.6, U37.1
- new net: U36.8, U37.2
- new net: U23.10, U37.4
- new net: U15.12, U37.5
- new net: U36.2, U37.12
- new net: U23.4, U37.13
- no-connect marks 64 -> 68
Other:
- note added: "65SIB port"
- note removed: "65SIB ports"
- moved on the sheet: C4, D1, J4, R15, SW2, U23F, U31A, U35A, U35B, U36C, U36E, U38A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

Commit message: Extra routing and placement completed...
Changed lines of the file:
@@
 F 0 "#LOGO1" H 31750 21500 50  0001 C CNN
 F 1 "Logo_Open_Hardware_Large" H 31750 20600 50  0001 C CNN
-F 2 "" H 31750 21000 50  0001 C CNN
+F 2 "Symbol:OSHW-Logo2_14.6x12mm_SilkScreen" H 31750 21000 50  0001 C CNN
 F 3 "~" H 31750 21000 50  0001 C CNN
 	1    31750 21000
@@
 Wire Notes Line
 	8700 4450 1800 4450
-Text Notes 18100 7700 2    50   ~ 0
+Text Notes 18750 7550 2    50   ~ 0
 RS-232 (Serial/COM) ports
 $Comp
@@
 Wire Wire Line
 	26800 8500 26800 8750
-Text Notes 18100 7800 2    50   ~ 0
+Text Notes 18750 7650 2    50   ~ 0
 IRQ0
 Text Notes 8550 9850 2    50   ~ 0
@@
 	1    0    0    -1
 $EndComp
-Text Notes 18100 7900 2    50   ~ 0
+Text Notes 18750 7750 2    50   ~ 0
 Address space: 0xD014 - 0xD017
 Text GLabel 11750 12550 2    50   Input ~ 0

Commit message: Completed version 2 schematic...
Parts:
- added unit 3 of U39
- added unit 5 of U42
- added unit 7 of U43
- U27: footprint Package_DIP:DIP-28_W15.24mm_Socket_LongPads -> Package_DIP:DIP-40_W15.24mm_Socket_LongPads
Connections:
- net GND: now also U39.14 (VCC), U39.7 (GND), U42.14 (VCC), U42.7 (GND), U43.14 (VCC), U43.7 (GND)
Other:
- moved on the sheet: C3
Changed lines of the file:
@@
 L Device:C C3
 U 1 1 61918BA3
-P 6700 2650
-F 0 "C3" H 6815 2696 50  0000 L CNN
-F 1 "0.33 uF" H 6815 2605 50  0000 L CNN
-F 2 "Capacitor_THT:C_Disc_D3.0mm_W1.6mm_P2.50mm" H 6738 2500 50  0001 C CNN
-F 3 "~" H 6700 2650 50  0001 C CNN
-	1    6700 2650
+P 6700 2700
+F 0 "C3" H 6815 2746 50  0000 L CNN
+F 1 "0.33 uF" H 6815 2655 50  0000 L CNN
+F 2 "Capacitor_THT:C_Disc_D3.0mm_W1.6mm_P2.50mm" H 6738 2550 50  0001 C CNN
+F 3 "~" H 6700 2700 50  0001 C CNN
+	1    6700 2700
 	1    0    0    -1
 $EndComp
 Wire Wire Line
-	6700 2800 6700 3100
-Wire Wire Line
-	6700 2500 6700 2200
-Wire Wire Line
 	2350 3100 3750 3100
 $Comp
@@
 Wire Wire Line
 	7050 2900 7050 3100
-Connection ~ 6700 3100
-Wire Wire Line
-	6700 2200 7050 2200
 Wire Wire Line
 	7050 2200 7050 2300
@@
 $EndComp
 Wire Wire Line
-	6550 2200 6700 2200
-Connection ~ 6700 2200
-Wire Wire Line
 	6250 2500 6250 3100
 $Comp
@@
 	7800 1700 8250 1700
 Connection ~ 6550 3100
-Wire Wire Line
-	6550 3100 6700 3100
 Connection ~ 6550 2200
 Wire Wire Line
@@
 $EndComp
 Wire Wire Line
-	6700 3100 6850 3100
-Wire Wire Line
 	7450 3100 7650 3100
 Wire Wire Line
@@
 F 0 "U27" H 24350 7413 60  0000 C CNN
 F 1 "WD65C22" H 24350 7519 60  0000 C CNN
-F 2 "Package_DIP:DIP-28_W15.24mm_Socket_LongPads" H 23850 8850 60  0001 C CNN
+F 2 "Package_DIP:DIP-40_W15.24mm_Socket_LongPads" H 23850 8850 60  0001 C CNN
 F 3 "" H 23850 8850 60  0000 C CNN
 	1    24350 8650
@@
 GND
 NoConn ~ 16200 10450
+$Comp
+L 74xx:74LS21 U39
+U 3 1 626DCCF3
+P 13700 11750
+F 0 "U39" H 13930 11796 50  0000 L CNN
+F 1 "74LS21" H 13930 11705 50  0000 L CNN
+F 2 "Package_DIP:DIP-14_W7.62mm_Socket_LongPads" H 13700 11750 50  0001 C CNN
+F 3 "http://www.ti.com/lit/gpn/sn74LS21" H 13700 11750 50  0001 C CNN
+	3    13700 11750
+	1    0    0    -1
+$EndComp
+Text GLabel 13700 11250 1    50   Input ~ 0
+VCC
+Text GLabel 13700 12250 3    50   Output ~ 0
+GND
+$Comp
+L 74xx:74LS08 U42
+U 5 1 626EAF96
+P 14450 11750
+F 0 "U42" H 14680 11796 50  0000 L CNN
+F 1 "74LS08" H 14680 11705 50  0000 L CNN
+F 2 "Package_DIP:DIP-14_W7.62mm_Socket_LongPads" H 14450 11750 50  0001 C CNN
+F 3 "http://www.ti.com/lit/gpn/sn74LS08" H 14450 11750 50  0001 C CNN
+	5    14450 11750
+	1    0    0    -1
+$EndComp
+Text GLabel 14450 11250 1    50   Input ~ 0
+VCC
+Text GLabel 14450 12250 3    50   Output ~ 0
+GND
+$Comp
+L 74xx:74HCT04 U43
+U 7 1 626F5FEB
+P 15200 11750
+F 0 "U43" H 15430 11796 50  0000 L CNN
+F 1 "74HCT04" H 15430 11705 50  0000 L CNN
+F 2 "Package_DIP:DIP-14_W7.62mm_Socket_LongPads" H 15200 11750 50  0001 C CNN
+F 3 "https://assets.nexperia.com/documents/data-sheet/74HC_HCT04.pdf" H 15200 11750 50  0001 C CNN
+	7    15200 11750
+	1    0    0    -1
+$EndComp
+Text GLabel 15200 11250 1    50   Input ~ 0
+VCC
+Text GLabel 15200 12250 3    50   Output ~ 0
+GND
+Wire Wire Line
+	6550 2200 6700 2200
+Wire Wire Line
+	6550 3100 6700 3100
+Wire Wire Line
+	6700 2850 6700 3100
+Connection ~ 6700 3100
+Wire Wire Line
+	6700 3100 6850 3100
+Wire Wire Line
+	6700 2550 6700 2200
+Connection ~ 6700 2200
+Wire Wire Line
+	6700 2200 7050 2200
 $EndSCHEMATC
