File: Motherboard/Motherboard.sch (KiCad schematic (older format))
At the start: 136 parts, among them J1 Jack-DC_18v, J2 65SIB_Connector, J3 DB9_Header, J4 GPIO_Connector, J5 Expansion_Connector, J6 Expansion_Connector, J7 Expansion_Connector, J8 Expansion_Connector, J9 Expansion_Connector, P1 POWER TERMINAL, Q1 2N3055, Q2 TIC106, SW1 SW_DPDT, SW2 FUSE RESET, SW3 PROCESSOR RESET, U1 LM7812_TO220, U13 LM386, U14 LM7912_TO220, U4 LM7805_TO220, X1 ACO-8MHz

Commit message: Well on the road to 2.3...
Other:
- note added: "VCC, GND and capacitors."
- moved on the sheet: H1, H2, H3, H4, H5, H6
Changed lines of the file:
@@
 L Graphic:Logo_Open_Hardware_Large #LOGO1
 U 1 1 61C12325
-P 14850 20600
-F 0 "#LOGO1" H 14850 21100 50  0001 C CNN
-F 1 "Logo_Open_Hardware_Large" H 14850 20200 50  0001 C CNN
-F 2 "Symbol:OSHW-Logo2_14.6x12mm_SilkScreen" H 14850 20600 50  0001 C CNN
-F 3 "~" H 14850 20600 50  0001 C CNN
-	1    14850 20600
+P 14700 21100
+F 0 "#LOGO1" H 14700 21600 50  0001 C CNN
+F 1 "Logo_Open_Hardware_Large" H 14700 20700 50  0001 C CNN
+F 2 "Symbol:OSHW-Logo2_14.6x12mm_SilkScreen" H 14700 21100 50  0001 C CNN
+F 3 "~" H 14700 21100 50  0001 C CNN
+	1    14700 21100
 	1    0    0    -1
 $EndComp
@@
 	25050 1150 25050 7150
 Wire Notes Line
-	30850 1150 30850 13750
-Wire Notes Line
 	1800 1150 30850 1150
 Text GLabel 28850 4150 2    50   Input ~ 0
@@
 L Graphic:SYM_ESD_Large #SYM2
 U 1 1 62084D56
-P 13650 20700
-F 0 "#SYM2" H 13650 20900 50  0001 C CNN
-F 1 "SYM_ESD_Large" H 13650 20450 50  0001 C CNN
-F 2 "Symbol:ESD-Logo_13.2x12mm_SilkScreen" H 13645 20670 50  0001 C CNN
-F 3 "~" H 13645 20670 50  0001 C CNN
-	1    13650 20700
+P 13500 21200
+F 0 "#SYM2" H 13500 21400 50  0001 C CNN
+F 1 "SYM_ESD_Large" H 13500 20950 50  0001 C CNN
+F 2 "Symbol:ESD-Logo_13.2x12mm_SilkScreen" H 13495 21170 50  0001 C CNN
+F 3 "~" H 13495 21170 50  0001 C CNN
+	1    13500 21200
 	1    0    0    -1
 $EndComp
@@
 L Graphic:SYM_Flash_XLarge #SYM4
 U 1 1 620873CC
-P 13200 20750
-F 0 "#SYM4" V 13050 20750 50  0001 C CNN
-F 1 "SYM_Flash_XLarge" V 13350 20750 50  0001 C CNN
-F 2 "Symbol:Symbol_HighVoltage_Type2_CopperTop_Big" H 13200 20725 50  0001 C CNN
-F 3 "~" H 13600 20650 50  0001 C CNN
-	1    13200 20750
+P 13050 21250
+F 0 "#SYM4" V 12900 21250 50  0001 C CNN
+F 1 "SYM_Flash_XLarge" V 13200 21250 50  0001 C CNN
+F 2 "Symbol:Symbol_HighVoltage_Type2_CopperTop_Big" H 13050 21225 50  0001 C CNN
+F 3 "~" H 13450 21150 50  0001 C CNN
+	1    13050 21250
 	1    0    0    -1
 $EndComp
@@
 L Graphic:SYM_Hot_Large #SYM3
 U 1 1 620C2A36
-P 14150 20700
-F 0 "#SYM3" H 14150 20900 50  0001 C CNN
-F 1 "SYM_Hot_Large" H 14150 20450 50  0001 C CNN
-F 2 "" H 14150 20500 50  0001 C CNN
-F 3 "~" H 14180 20500 50  0001 C CNN
-	1    14150 20700
+P 14000 21200
+F 0 "#SYM3" H 14000 21400 50  0001 C CNN
+F 1 "SYM_Hot_Large" H 14000 20950 50  0001 C CNN
+F 2 "" H 14000 21000 50  0001 C CNN
+F 3 "~" H 14030 21000 50  0001 C CNN
+	1    14000 21200
 	1    0    0    -1
 $EndComp
@@
 Wire Wire Line
 	5450 2600 5700 2600
-Text Notes 2700 20150 2    50   ~ 0
+Text Notes 13200 20250 2    50   ~ 0
 Miscellaneous parts
 $Comp
@@
 	8750 1150 8750 19950
 Wire Notes Line
-	12100 13750 12100 19950
-Wire Notes Line
 	22950 16850 1800 16850
 $Comp
@@
 A13
 Wire Notes Line
-	1800 1150 1800 22800
-Wire Notes Line
-	1800 22800 15550 22800
-Wire Notes Line
 	15550 13750 15550 22800
 $Comp
 L Mechanical:MountingHole H2
 U 1 1 6483DDE7
-P 14650 21150
-F 0 "H2" H 14750 21196 50  0000 L CNN
-F 1 "MountingHole" H 14750 21105 50  0000 L CNN
-F 2 "MountingHole:MountingHole_3.2mm_M3" H 14650 21150 50  0001 C CNN
-F 3 "~" H 14650 21150 50  0001 C CNN
-	1    14650 21150
+P 14500 21650
+F 0 "H2" H 14600 21696 50  0000 L CNN
+F 1 "MountingHole" H 14600 21605 50  0000 L CNN
+F 2 "MountingHole:MountingHole_3.2mm_M3" H 14500 21650 50  0001 C CNN
+F 3 "~" H 14500 21650 50  0001 C CNN
+	1    14500 21650
 	1    0    0    -1
 $EndComp
@@
 L Mechanical:MountingHole H1
 U 1 1 6483E48F
-P 13900 21150
-F 0 "H1" H 14000 21196 50  0000 L CNN
-F 1 "MountingHole" H 14000 21105 50  0000 L CNN
-F 2 "MountingHole:MountingHole_3.2mm_M3" H 13900 21150 50  0001 C CNN
-F 3 "~" H 13900 21150 50  0001 C CNN
-	1    13900 21150
+P 13750 21650
+F 0 "H1" H 13850 21696 50  0000 L CNN
+F 1 "MountingHole" H 13850 21605 50  0000 L CNN
+F 2 "MountingHole:MountingHole_3.2mm_M3" H 13750 21650 50  0001 C CNN
+F 3 "~" H 13750 21650 50  0001 C CNN
+	1    13750 21650
 	1    0    0    -1
 $EndComp
@@
 L Mechanical:MountingHole H4
 U 1 1 6483EC45
-P 14650 21400
-F 0 "H4" H 14750 21446 50  0000 L CNN
-F 1 "MountingHole" H 14750 21355 50  0000 L CNN
-F 2 "MountingHole:MountingHole_3.2mm_M3" H 14650 21400 50  0001 C CNN
-F 3 "~" H 14650 21400 50  0001 C CNN
-	1    14650 21400
+P 14500 21900
+F 0 "H4" H 14600 21946 50  0000 L CNN
+F 1 "MountingHole" H 14600 21855 50  0000 L CNN
+F 2 "MountingHole:MountingHole_3.2mm_M3" H 14500 21900 50  0001 C CNN
+F 3 "~" H 14500 21900 50  0001 C CNN
+	1    14500 21900
 	1    0    0    -1
 $EndComp
@@
 L Mechanical:MountingHole H3
 U 1 1 6483EC4B
-P 13900 21400
-F 0 "H3" H 14000 21446 50  0000 L CNN
-F 1 "MountingHole" H 14000 21355 50  0000 L CNN
-F 2 "MountingHole:MountingHole_3.2mm_M3" H 13900 21400 50  0001 C CNN
-F 3 "~" H 13900 21400 50  0001 C CNN
-	1    13900 21400
+P 13750 21900
+F 0 "H3" H 13850 21946 50  0000 L CNN
+F 1 "MountingHole" H 13850 21855 50  0000 L CNN
+F 2 "MountingHole:MountingHole_3.2mm_M3" H 13750 21900 50  0001 C CNN
+F 3 "~" H 13750 21900 50  0001 C CNN
+	1    13750 21900
 	1    0    0    -1
 $EndComp
@@
 L Mechanical:MountingHole H6
 U 1 1 6489366B
-P 14650 21650
-F 0 "H6" H 14750 21696 50  0000 L CNN
-F 1 "MountingHole" H 14750 21605 50  0000 L CNN
-F 2 "MountingHole:MountingHole_3.2mm_M3" H 14650 21650 50  0001 C CNN
-F 3 "~" H 14650 21650 50  0001 C CNN
-	1    14650 21650
+P 14500 22150
+F 0 "H6" H 14600 22196 50  0000 L CNN
+F 1 "MountingHole" H 14600 22105 50  0000 L CNN
+F 2 "MountingHole:MountingHole_3.2mm_M3" H 14500 22150 50  0001 C CNN
+F 3 "~" H 14500 22150 50  0001 C CNN
+	1    14500 22150
 	1    0    0    -1
 $EndComp
@@
 L Mechanical:MountingHole H5
 U 1 1 64893671
-P 13900 21650
-F 0 "H5" H 14000 21696 50  0000 L CNN
-F 1 "MountingHole" H 14000 21605 50  0000 L CNN
-F 2 "MountingHole:MountingHole_3.2mm_M3" H 13900 21650 50  0001 C CNN
-F 3 "~" H 13900 21650 50  0001 C CNN
-	1    13900 21650
+P 13750 22150
+F 0 "H5" H 13850 22196 50  0000 L CNN
+F 1 "MountingHole" H 13850 22105 50  0000 L CNN
+F 2 "MountingHole:MountingHole_3.2mm_M3" H 13750 22150 50  0001 C CNN
+F 3 "~" H 13750 22150 50  0001 C CNN
+	1    13750 22150
 	1    0    0    -1
 $EndComp
+Wire Notes Line
+	30850 21550 15550 21550
+Wire Notes Line
+	30850 1150 30850 21550
+Text Notes 23200 14200 0    50   ~ 0
+VCC, GND and capacitors.
+Wire Notes Line
+	1800 1150 1800 19950
+Wire Notes Line
+	12100 22800 15550 22800
+Wire Notes Line
+	12100 13750 12100 22800
 $EndSCHEMATC

Commit message: 500 odd traces left...
Connections:
- net 8MHz: now also J5.26 (Pin_26), J6.26 (Pin_26), J7.26 (Pin_26), J8.26 (Pin_26), J9.26 (Pin_26)
- no-connect marks 53 -> 48
Other:
- note added: "Expansion ports\nIRQ3 - IRQ7"
- note removed: "Expansion sockets and ports\nIRQ3 - IRQ7"
- moved on the sheet: J4, JP7
Changed lines of the file:
@@
 Date "2022-04-29"
 Rev "2.3"
-Comp "WolfNet"
+Comp "WolfNet Computing"
 Comment1 "Motherboard for the WolfNet 65C02 based (NMOS Compatible) WorkBench Computer."
 Comment2 "CODENAME: Wolfe-1"
@@
 	1    0    0    -1
 $EndComp
-Text GLabel 4300 10000 0    50   BiDi ~ 0
+Text GLabel 4550 10000 0    50   BiDi ~ 0
 GPIO0
-Text GLabel 4300 10100 0    50   BiDi ~ 0
+Text GLabel 4550 10100 0    50   BiDi ~ 0
 GPIO1
-Text GLabel 4300 10200 0    50   BiDi ~ 0
+Text GLabel 4550 10200 0    50   BiDi ~ 0
 GPIO2
-Text GLabel 4300 10300 0    50   BiDi ~ 0
+Text GLabel 4550 10300 0    50   BiDi ~ 0
 GPIO3
-Text GLabel 4300 10400 0    50   BiDi ~ 0
+Text GLabel 4550 10400 0    50   BiDi ~ 0
 GPIO4
 $Comp
 L PC:GPIO_Connector J4
 U 1 1 61A7B6BE
-P 4500 10400
-F 0 "J4" H 4550 11100 50  0000 C CNN
-F 1 "GPIO_Connector" H 4550 11000 50  0000 C CNN
-F 2 "Connector_PinSocket_2.54mm:PinSocket_2x11_P2.54mm_Vertical" H 4500 10400 50  0001 C CNN
-F 3 "~" H 4500 10400 50  0001 C CNN
-	1    4500 10400
+P 4750 10400
+F 0 "J4" H 4800 11100 50  0000 C CNN
+F 1 "GPIO_Connector" H 4800 11000 50  0000 C CNN
+F 2 "Connector_PinSocket_2.54mm:PinSocket_2x11_P2.54mm_Vertical" H 4750 10400 50  0001 C CNN
+F 3 "~" H 4750 10400 50  0001 C CNN
+	1    4750 10400
 	1    0    0    -1
 $EndComp
-Text GLabel 4300 10600 0    50   BiDi ~ 0
+Text GLabel 4550 10600 0    50   BiDi ~ 0
 GPIO6
-Text GLabel 4300 10500 0    50   BiDi ~ 0
+Text GLabel 4550 10500 0    50   BiDi ~ 0
 GPIO5
-Text GLabel 4300 10700 0    50   BiDi ~ 0
+Text GLabel 4550 10700 0    50   BiDi ~ 0
 GPIO7
-Text GLabel 4300 10800 0    50   BiDi ~ 0
+Text GLabel 4550 10800 0    50   BiDi ~ 0
 GPIO8
-Text GLabel 4300 10900 0    50   BiDi ~ 0
+Text GLabel 4550 10900 0    50   BiDi ~ 0
 GPIO9
-Text GLabel 4800 10400 2    50   BiDi ~ 0
+Text GLabel 5050 10400 2    50   BiDi ~ 0
 GPIO15
-Text GLabel 4800 10500 2    50   BiDi ~ 0
+Text GLabel 5050 10500 2    50   BiDi ~ 0
 GPIO14
-Text GLabel 4800 10600 2    50   BiDi ~ 0
+Text GLabel 5050 10600 2    50   BiDi ~ 0
 GPIO13
-Text GLabel 4800 10700 2    50   BiDi ~ 0
+Text GLabel 5050 10700 2    50   BiDi ~ 0
 GPIO12
-Text GLabel 4800 10800 2    50   BiDi ~ 0
+Text GLabel 5050 10800 2    50   BiDi ~ 0
 GPIO11
-Text GLabel 4800 10900 2    50   BiDi ~ 0
+Text GLabel 5050 10900 2    50   BiDi ~ 0
 GPIO10
-Text GLabel 4800 10300 2    50   BiDi ~ 0
+Text GLabel 5050 10300 2    50   BiDi ~ 0
 CA1
-Text GLabel 4800 10200 2    50   BiDi ~ 0
+Text GLabel 5050 10200 2    50   BiDi ~ 0
 CA2
-Text GLabel 4800 10100 2    50   BiDi ~ 0
+Text GLabel 5050 10100 2    50   BiDi ~ 0
 CB1
-Text GLabel 4800 10000 2    50   BiDi ~ 0
+Text GLabel 5050 10000 2    50   BiDi ~ 0
 CB2
 Text GLabel 3650 10050 2    50   Input ~ 0
@@
 L PC_Jumpers:Jumper_3_Bridged12 JP7
 U 1 1 61A75D9B
-P 5850 10150
-F 0 "JP7" V 5804 10217 50  0000 L CNN
-F 1 "NMI/IRQ1" V 5895 10217 50  0000 L CNN
-F 2 "Connector_PinHeader_2.54mm:PinHeader_1x03_P2.54mm_Vertical" H 5850 10150 50  0001 C CNN
-F 3 "~" H 5850 10150 50  0001 C CNN
-	1    5850 10150
+P 5350 11750
+F 0 "JP7" V 5304 11817 50  0000 L CNN
+F 1 "NMI/IRQ1" V 5395 11817 50  0000 L CNN
+F 2 "Connector_PinHeader_2.54mm:PinHeader_1x03_P2.54mm_Vertical" H 5350 11750 50  0001 C CNN
+F 3 "~" H 5350 11750 50  0001 C CNN
+	1    5350 11750
 	0    1    1    0
 $EndComp
-Text GLabel 5700 10150 0    50   Input ~ 0
+Text GLabel 5200 11750 0    50   Input ~ 0
 ~IRQ_DECIDE
-Text GLabel 5850 9900 1    50   Output ~ 0
+Text GLabel 5350 11500 1    50   Output ~ 0
 ~IRQ1
-Text GLabel 5850 10400 3    50   Output ~ 0
+Text GLabel 5350 12000 3    50   Output ~ 0
 ~NMI
 Text GLabel 15100 8900 1    50   Output ~ 0
@@
 	27650 4550 27650 4350
 Text Notes 23200 10900 0    50   ~ 0
-Expansion sockets and ports\nIRQ3 - IRQ7
+Expansion ports\nIRQ3 - IRQ7
 Wire Wire Line
 	7050 3100 7200 3100
@@
 Wire Wire Line
 	16500 9200 16500 9450
-Text GLabel 4300 9900 0    50   Input ~ 0
+Text GLabel 4550 9900 0    50   Input ~ 0
 VCC
-Text GLabel 4800 9900 2    50   Output ~ 0
+Text GLabel 5050 9900 2    50   Output ~ 0
 GND
 NoConn ~ 10150 8350
@@
 Text GLabel 30150 12100 2    50   Input ~ 0
 ~RESET
-NoConn ~ 30150 12500
-NoConn ~ 28600 12500
-NoConn ~ 27000 12500
-NoConn ~ 25400 12500
 Wire Wire Line
 	11800 3100 13100 3100
@@
 Text GLabel 23900 12600 2    50   Input ~ 0
 ~CS_DEV
-NoConn ~ 23900 12500
 Wire Notes Line
 	19100 1150 19100 16850
@@
 Wire Notes Line
 	12100 13750 12100 22800
+Text GLabel 30150 12500 2    50   Input ~ 0
+8MHz
+Text GLabel 28600 12500 2    50   Input ~ 0
+8MHz
+Text GLabel 27000 12500 2    50   Input ~ 0
+8MHz
+Text GLabel 25400 12500 2    50   Input ~ 0
+8MHz
+Text GLabel 23900 12500 2    50   Input ~ 0
+8MHz
 $EndSCHEMATC

Commit message: Caps, Power for gates and traces added...
Parts:
- added C10, C11, C12, C13, C14, C15, C16, C17, C18, C19, C20, C21, C22, C23, C24, C25, C26, C27, C28, C29, C30, C31, C32, C34, C35, C36, C37, C38, C39, C40, C42, C43, C44, C45, C46, C47, C48, C49, C50, C51, C52, C53, C54, C55, C56, C57, C58, C7, C8, C9: 100 nF, Capacitor_THT:C_Disc_D3.0mm_W1.6mm_P2.50mm, symbol Device:C
- added unit 5 of CS_65SIB_AND1
- added unit 3 of CS_65SIB_AND4
- added unit 7 of CS_65SIB_NOR1
- added unit 5 of CS_GPIO_AND1
- added unit 3 of CS_GPIO_AND4
- added unit 7 of CS_GPIO_NOR1
- added unit 5 of CS_UART_AND1
- added unit 3 of CS_UART_AND4
- added unit 7 of CS_UART_NOR1
- added unit 5 of CS_VID_NAND1
- added unit 7 of CS_VID_NOR1
- added unit 7 of IRQ_NOR1
- added unit 5 of IRQ_RW_AND1
- added unit 5 of RAM_NAND1
- added unit 5 of RAM_NAND2
- added unit 7 of RAM_NOR1
- added unit 7 of RESET_NOR1
- added unit 3 of ROM1_NAND4
- added unit 3 of ROM2_NAND4
- added unit 3 of ROM3_NAND4
- added unit 3 of ROM4_NAND4
- added unit 7 of ROM_NOR1
- added unit 3 of SHARED_ROM2
- added unit 7 of ~MAX235_EN1
- renumbered 65SIB1 to 65SIB/MM1
Connections:
- net GND: now also C10.2, C11.2, C12.2, C13.2, C14.2, C15.2, C16.2, C17.2, C18.2, C19.2, C20.2, C21.2, C22.2, C23.2, C24.2, C25.2, C26.2, C27.2, C28.2, C29.2, C30.2, C31.2, C32.2, C34.2, C35.2, C36.2, C37.2, C38.2, C39.2, C40.2, C42.2, C43.2, C44.2, C45.2, C46.2, C47.2, C48.2, C49.2, C50.2, C51.2, C52.2, C53.2, C54.2, C55.2, C56.2, C57.2, C58.2, C7.2, C8.2, C9.2, CS_65SIB_AND1.7 (GND), CS_65SIB_AND4.7 (GND), CS_65SIB_NOR1.7 (GND), CS_GPIO_AND1.7 (GND), CS_GPIO_AND4.7 (GND), CS_GPIO_NOR1.7 (GND), CS_UART_AND1.7 (GND), CS_UART_AND4.7 (GND), CS_UART_NOR1.7 (GND), CS_VID_NAND1.7 (GND), CS_VID_NOR1.7 (GND), IRQ_NOR1.7 (GND), IRQ_RW_AND1.7 (GND), RAM_NAND1.7 (GND), RAM_NAND2.7 (GND), RAM_NOR1.7 (GND), RESET_NOR1.7 (GND), ROM1_NAND4.7 (GND), ROM2_NAND4.7 (GND), ROM3_NAND4.7 (GND), ROM4_NAND4.7 (GND), ROM_NOR1.7 (GND), SHARED_ROM2.7 (GND), ~MAX235_EN1.7 (GND)
- net VCC: now also C10.1, C11.1, C12.1, C13.1, C14.1, C15.1, C16.1, C17.1, C18.1, C19.1, C20.1, C21.1, C22.1, C23.1, C24.1, C25.1, C26.1, C27.1, C28.1, C29.1, C30.1, C31.1, C32.1, C34.1, C35.1, C36.1, C37.1, C38.1, C39.1, C40.1, C42.1, C43.1, C44.1, C45.1, C46.1, C47.1, C48.1, C49.1, C50.1, C51.1, C52.1, C53.1, C54.1, C55.1, C56.1, C57.1, C58.1, C7.1, C8.1, C9.1, CS_65SIB_AND1.14 (VCC), CS_65SIB_AND4.14 (VCC), CS_65SIB_NOR1.14 (VCC), CS_GPIO_AND1.14 (VCC), CS_GPIO_AND4.14 (VCC), CS_GPIO_NOR1.14 (VCC), CS_UART_AND1.14 (VCC), CS_UART_AND4.14 (VCC), CS_UART_NOR1.14 (VCC), CS_VID_NAND1.14 (VCC), CS_VID_NOR1.14 (VCC), IRQ_NOR1.14 (VCC), IRQ_RW_AND1.14 (VCC), RAM_NAND1.14 (VCC), RAM_NAND2.14 (VCC), RAM_NOR1.14 (VCC), RESET_NOR1.14 (VCC), ROM1_NAND4.14 (VCC), ROM2_NAND4.14 (VCC), ROM3_NAND4.14 (VCC), ROM4_NAND4.14 (VCC), ROM_NOR1.14 (VCC), SHARED_ROM2.14 (VCC), ~MAX235_EN1.14 (VCC)
Other:
- note added: "VCC, GND and 52 capacitors."
- note removed: "VCC, GND and capacitors."

Commit message: 539 traces to go...
Parts:
- added C33, C41: 100 nF, Capacitor_THT:C_Disc_D3.0mm_W1.6mm_P2.50mm, symbol Device:C
Connections:
- net GND: now also C33.2, C41.2
- net VCC: now also C33.1, C41.1
Changed lines of the file:
@@
 Text GLabel 23850 18650 3    50   Output ~ 0
 GND
+$Comp
+L Device:C C33
+U 1 1 62755F17
+P 26350 16250
+F 0 "C33" H 26465 16296 50  0000 L CNN
+F 1 "100 nF" H 26465 16205 50  0000 L CNN
+F 2 "Capacitor_THT:C_Disc_D3.0mm_W1.6mm_P2.50mm" H 26388 16100 50  0001 C CNN
+F 3 "~" H 26350 16250 50  0001 C CNN
+	1    26350 16250
+	1    0    0    -1
+$EndComp
+Text GLabel 26350 16100 1    50   Input ~ 0
+VCC
+Text GLabel 26350 16400 3    50   Output ~ 0
+GND
+$Comp
+L Device:C C41
+U 1 1 627AAA94
+P 25350 17000
+F 0 "C41" H 25465 17046 50  0000 L CNN
+F 1 "100 nF" H 25465 16955 50  0000 L CNN
+F 2 "Capacitor_THT:C_Disc_D3.0mm_W1.6mm_P2.50mm" H 25388 16850 50  0001 C CNN
+F 3 "~" H 25350 17000 50  0001 C CNN
+	1    25350 17000
+	1    0    0    -1
+$EndComp
+Text GLabel 25350 16850 1    50   Input ~ 0
+VCC
+Text GLabel 25350 17150 3    50   Output ~ 0
+GND
 $EndSCHEMATC
