File: Motherboard/_autosave-Motherboard.sch (KiCad schematic (older format))
At the start: 155 parts

Commit message: 2.3 ON THE WAY...
Parts:
- removed U?: 74HCT04, Package_DIP:DIP-14_W7.62mm_Socket_LongPads, symbol 74xx:74HCT04
Connections:
- net A6: now also U?.12
- net CS_COM: now also U?.1; no longer U?.3
- net IRQ\: now also U?.4; no longer U?.8
- net RW: now also U?.1; no longer U?.3
- net at U?.7 (Oa<b): now also U?.3; no longer U?.9
- net at U?.5: now also U?.2; no longer U?.4
- net at U?.20 (En\): now also U?.2; no longer U?.4
Other:
- note added: "Address space: 0xD0C0 - 0xD0CF"
- note removed: "Address space: 0xD040 - 0xD04F"
- note removed: "Interrupt Priority Chip Select - Read/Write"
- moved on the sheet: U?A, U?B, U?C, U?E, U?G
