File: Motherboard/_autosave-Motherboard.sch (KiCad schematic (older format))
At the start: 163 parts, among them J1 Jack-DC_18v, J2 65SIB_Connector, J3 DB9_Header, J4 GPIO_Connector, J5 Expansion_Connector, J6 Expansion_Connector, J7 Expansion_Connector, J8 Expansion_Connector, P1 POWER TERMINAL, Q1 2N3055, Q2 TIC106, SW1 SW_DPDT, SW2 FUSE RESET, SW3 PROCESSOR RESET, U1 LM7812_TO220, U13 LM386, U14 LM7912_TO220, U4 LM7805_TO220, X1 ACO-8MHz

Commit message: Part way to bank switched memory...
Connections:
- net A14: no longer ROM1_NAND1.10
- net A15: no longer ROM1_NAND1.9
- net ROM2_EN: now also ROM_NOR?.1; no longer ROM_NOR?.9
- net ROM3_EN: now also ROM_NOR?.9; no longer ROM_NOR?.1
- net ROM4_EN: now also ROM_NOR?.1; no longer ROM_NOR?.9
- net at ROM2_NAND?.5: now also ROM_NOR?.6; no longer ROM_NOR?.12
- net at ROM2_NAND?.6: now also ROM_NOR?.3; no longer ROM_NOR?.11
- net at ROM2_NAND?.8: now also ROM_NOR?.5; no longer ROM_NOR?.13
- net at ROM2_NAND?.1: now also ROM_NOR?.4; no longer ROM_NOR?.10
- net at ROM2_NAND?.2: now also ROM_NOR?.2; no longer ROM_NOR?.8
- net at ROM3_NAND?.5: now also ROM_NOR?.12; no longer ROM_NOR?.6
- net at ROM3_NAND?.6: now also ROM_NOR?.11; no longer ROM_NOR?.3
- net at ROM3_NAND?.8: now also ROM_NOR?.13; no longer ROM_NOR?.5
- net at ROM3_NAND?.1: now also ROM_NOR?.10; no longer ROM_NOR?.4
- net at ROM3_NAND?.2: now also ROM_NOR?.8; no longer ROM_NOR?.2
- net at ROM4_NAND?.5: now also ROM_NOR?.6; no longer ROM_NOR?.12
- net at ROM4_NAND?.6: now also ROM_NOR?.3; no longer ROM_NOR?.11
- net at ROM4_NAND?.8: now also ROM_NOR?.5; no longer ROM_NOR?.13
- net at ROM4_NAND?.1: now also ROM_NOR?.4; no longer ROM_NOR?.10
- net at ROM4_NAND?.2: now also ROM_NOR?.2; no longer ROM_NOR?.8
Other:
- note added: "Read-Only Memory\nBank 1 high"
- note added: "Read-Only Memory\nBank 2 high"
- note added: "Read-Only Memory\nBank 2 low"
- note added: "Read-Only Memory\nBank 3 low"
- note added: "Read-Only Memory\nBank 4 high"
- note added: "Read-Only Memory\nbank 4 low"
- note removed: "Read-Only Memory\nROM Bank 2"
- note removed: "Read-Only Memory\nROM bank 4 high"
- moved on the sheet: ROM1_NAND1A, ROM1_NAND1B, ROM1_NAND1C, ROM_NOR1A, ROM_NOR1B, ROM_NOR1C
Changed lines of the file:
@@
 L 74xx:74HCT00 ROM1_NAND1
 U 2 1 653EA77F
-P 7000 6300
-F 0 "ROM1_NAND1" H 7000 5983 50  0000 C CNN
-F 1 "74HCT00" H 7000 6074 50  0000 C CNN
-F 2 "Package_DIP:DIP-14_W7.62mm_Socket_LongPads" H 7000 6300 50  0001 C CNN
-F 3 "http://www.ti.com/lit/gpn/sn74hct00" H 7000 6300 50  0001 C CNN
-	2    7000 6300
+P 7000 6700
+F 0 "ROM1_NAND1" H 7000 6383 50  0000 C CNN
+F 1 "74HCT00" H 7000 6474 50  0000 C CNN
+F 2 "Package_DIP:DIP-14_W7.62mm_Socket_LongPads" H 7000 6700 50  0001 C CNN
+F 3 "http://www.ti.com/lit/gpn/sn74hct00" H 7000 6700 50  0001 C CNN
+	2    7000 6700
 	0    1    1    0
 $EndComp
@@
 L 74xx:74HCT00 ROM1_NAND1
 U 3 1 653EA785
-P 6900 5000
-F 0 "ROM1_NAND1" H 6900 4683 50  0000 C CNN
-F 1 "74HCT00" H 6900 4774 50  0000 C CNN
-F 2 "Package_DIP:DIP-14_W7.62mm_Socket_LongPads" H 6900 5000 50  0001 C CNN
-F 3 "http://www.ti.com/lit/gpn/sn74hct00" H 6900 5000 50  0001 C CNN
-	3    6900 5000
+P 6900 5400
+F 0 "ROM1_NAND1" H 6900 5083 50  0000 C CNN
+F 1 "74HCT00" H 6900 5174 50  0000 C CNN
+F 2 "Package_DIP:DIP-14_W7.62mm_Socket_LongPads" H 6900 5400 50  0001 C CNN
+F 3 "http://www.ti.com/lit/gpn/sn74hct00" H 6900 5400 50  0001 C CNN
+	3    6900 5400
 	0    1    1    0
 $EndComp
@@
 L 74xx:74HCT04 ROM_NOR1
 U 3 1 653EA78C
-P 6900 5650
-F 0 "ROM_NOR1" H 6900 5333 50  0000 C CNN
-F 1 "74HCT04" H 6900 5424 50  0000 C CNN
-F 2 "Package_DIP:DIP-14_W7.62mm_Socket_LongPads" H 6900 5650 50  0001 C CNN
-F 3 "https://assets.nexperia.com/documents/data-sheet/74HC_HCT04.pdf" H 6900 5650 50  0001 C CNN
-	3    6900 5650
-	0    1    1    0
-$EndComp
-Wire Wire Line
-	6900 5950 6900 6000
-Wire Wire Line
-	6900 5350 6900 5300
+P 6900 6050
+F 0 "ROM_NOR1" H 6900 5733 50  0000 C CNN
+F 1 "74HCT04" H 6900 5824 50  0000 C CNN
+F 2 "Package_DIP:DIP-14_W7.62mm_Socket_LongPads" H 6900 6050 50  0001 C CNN
+F 3 "https://assets.nexperia.com/documents/data-sheet/74HC_HCT04.pdf" H 6900 6050 50  0001 C CNN
+	3    6900 6050
+	0    1    1    0
+$EndComp
+Wire Wire Line
+	6900 6350 6900 6400
+Wire Wire Line
+	6900 5750 6900 5700
 Text GLabel 6800 4700 1    50   Input ~ 0
 A14
-Text GLabel 7100 6000 1    50   Input ~ 0
+Text GLabel 7100 6400 1    50   Input ~ 0
 A13
 Text GLabel 7000 4700 1    50   Input ~ 0
 A15
-Wire Wire Line
-	6600 5350 6600 6650
-Wire Wire Line
-	7000 6600 7000 6650
-Wire Wire Line
-	6600 6650 7000 6650
 $Comp
 L 74xx:74HCT00 ROM1_NAND1
 U 1 1 653EA7A4
-P 6150 6300
-F 0 "ROM1_NAND1" H 6150 5983 50  0000 C CNN
-F 1 "74HCT00" H 6150 6074 50  0000 C CNN
-F 2 "Package_DIP:DIP-14_W7.62mm_Socket_LongPads" H 6150 6300 50  0001 C CNN
-F 3 "http://www.ti.com/lit/gpn/sn74hct00" H 6150 6300 50  0001 C CNN
-	1    6150 6300
+P 6150 6700
+F 0 "ROM1_NAND1" H 6150 6383 50  0000 C CNN
+F 1 "74HCT00" H 6150 6474 50  0000 C CNN
+F 2 "Package_DIP:DIP-14_W7.62mm_Socket_LongPads" H 6150 6700 50  0001 C CNN
+F 3 "http://www.ti.com/lit/gpn/sn74hct00" H 6150 6700 50  0001 C CNN
+	1    6150 6700
 	0    1    1    0
 $EndComp
@@
 L 74xx:74HCT04 ROM_NOR1
 U 2 1 653EA7AA
-P 6400 5650
-F 0 "ROM_NOR1" H 6400 5333 50  0000 C CNN
-F 1 "74HCT04" H 6400 5424 50  0000 C CNN
-F 2 "Package_DIP:DIP-14_W7.62mm_Socket_LongPads" H 6400 5650 50  0001 C CNN
-F 3 "https://assets.nexperia.com/documents/data-sheet/74HC_HCT04.pdf" H 6400 5650 50  0001 C CNN
-	2    6400 5650
+P 6400 6050
+F 0 "ROM_NOR1" H 6400 5733 50  0000 C CNN
+F 1 "74HCT04" H 6400 5824 50  0000 C CNN
+F 2 "Package_DIP:DIP-14_W7.62mm_Socket_LongPads" H 6400 6050 50  0001 C CNN
+F 3 "https://assets.nexperia.com/documents/data-sheet/74HC_HCT04.pdf" H 6400 6050 50  0001 C CNN
+	2    6400 6050
 	0    1    1    0
 $EndComp
@@
 L 74xx:74HCT04 ROM_NOR1
 U 1 1 653EA7B0
-P 5950 5650
-F 0 "ROM_NOR1" H 5950 5333 50  0000 C CNN
-F 1 "74HCT04" H 5950 5424 50  0000 C CNN
-F 2 "Package_DIP:DIP-14_W7.62mm_Socket_LongPads" H 5950 5650 50  0001 C CNN
-F 3 "https://assets.nexperia.com/documents/data-sheet/74HC_HCT04.pdf" H 5950 5650 50  0001 C CNN
-	1    5950 5650
-	0    1    1    0
-$EndComp
-Wire Wire Line
-	6250 6000 6400 6000
-Wire Wire Line
-	6400 6000 6400 5950
-Wire Wire Line
-	6400 5350 6600 5350
-Text GLabel 5950 5350 1    50   Input ~ 0
+P 5950 6050
+F 0 "ROM_NOR1" H 5950 5733 50  0000 C CNN
+F 1 "74HCT04" H 5950 5824 50  0000 C CNN
+F 2 "Package_DIP:DIP-14_W7.62mm_Socket_LongPads" H 5950 6050 50  0001 C CNN
+F 3 "https://assets.nexperia.com/documents/data-sheet/74HC_HCT04.pdf" H 5950 6050 50  0001 C CNN
+	1    5950 6050
+	0    1    1    0
+$EndComp
+Wire Wire Line
+	6250 6400 6400 6400
+Wire Wire Line
+	6400 6400 6400 6350
+Wire Wire Line
+	6400 5750 6600 5750
+Text GLabel 5950 5750 1    50   Input ~ 0
 ROM1_EN
 Wire Wire Line
@@
 NoConn ~ 8300 6500
 Wire Wire Line
-	6050 5950 6050 6000
-Wire Wire Line
-	5950 5950 6050 5950
+	6050 6350 6050 6400
+Wire Wire Line
+	5950 6350 6050 6350
 Wire Wire Line
 	16050 5900 17200 5900
@@
 Wire Wire Line
 	2200 15450 2300 15450
-Text Notes 1900 14200 0    50   ~ 0
-Read-Only Memory\nROM Bank 2
+Text Notes 1900 14000 0    50   ~ 0
+Read-Only Memory\nBank 2 low
 $Comp
 L PC:28C64 ROM3
@@
 	5750 15450 5850 15450
 Text Notes 5450 14200 0    50   ~ 0
-Read-Only Memory\nBank 3 high
+Read-Only Memory\nBank 3 low
 $Comp
 L PC:28C64 ROM4
@@
 	9300 15450 9400 15450
 Text Notes 9000 14200 0    50   ~ 0
-Read-Only Memory\nROM bank 4 high
+Read-Only Memory\nbank 4 low
 Wire Wire Line
 	4150 14000 4150 14200
@@
 	11250 14000 11250 14200
 Wire Wire Line
-	6150 6600 6150 7050
-Wire Wire Line
-	6150 7050 7350 7050
+	6150 7000 6150 7050
 Wire Wire Line
 	2400 16100 2400 16550
@@
 $Comp
 L 74xx:74HCT04 ROM_NOR?
-U 6 1 635AA6FD
+U 3 1 635AA6FD
 P 3150 18250
 F 0 "ROM_NOR?" H 3150 17933 50  0000 C CNN
@@
 F 2 "Package_DIP:DIP-14_W7.62mm_Socket_LongPads" H 3150 18250 50  0001 C CNN
 F 3 "https://assets.nexperia.com/documents/data-sheet/74HC_HCT04.pdf" H 3150 18250 50  0001 C CNN
-	6    3150 18250
+	3    3150 18250
 	0    1    1    0
 $EndComp
@@
 $Comp
 L 74xx:74HCT04 ROM_NOR?
-U 5 1 635AA711
+U 2 1 635AA711
 P 2650 18250
 F 0 "ROM_NOR?" H 2650 17933 50  0000 C CNN
@@
 F 2 "Package_DIP:DIP-14_W7.62mm_Socket_LongPads" H 2650 18250 50  0001 C CNN
 F 3 "https://assets.nexperia.com/documents/data-sheet/74HC_HCT04.pdf" H 2650 18250 50  0001 C CNN
-	5    2650 18250
+	2    2650 18250
 	0    1    1    0
 $EndComp
 $Comp
 L 74xx:74HCT04 ROM_NOR?
-U 4 1 635AA717
+U 1 1 635AA717
 P 2200 18250
 F 0 "ROM_NOR?" H 2200 17933 50  0000 C CNN
@@
 F 2 "Package_DIP:DIP-14_W7.62mm_Socket_LongPads" H 2200 18250 50  0001 C CNN
 F 3 "https://assets.nexperia.com/documents/data-sheet/74HC_HCT04.pdf" H 2200 18250 50  0001 C CNN
-	4    2200 18250
+	1    2200 18250
 	0    1    1    0
 $EndComp
@@
 	2200 18550 2300 18550
 Text Notes 1900 17300 0    50   ~ 0
-Read-Only Memory\nROM Bank 2
+Read-Only Memory\nBank 1 high
 $Comp
 L PC:28C64 ROM?
@@
 	5750 18550 5850 18550
 Text Notes 5450 17300 0    50   ~ 0
-Read-Only Memory\nBank 3 high
+Read-Only Memory\nBank 2 high
 $Comp
 L PC:28C64 ROM?
@@
 $Comp
 L 74xx:74HCT04 ROM_NOR?
-U 6 1 635AA7AD
+U 3 1 635AA7AD
 P 10250 18250
 F 0 "ROM_NOR?" H 10250 17933 50  0000 C CNN
@@
 F 2 "Package_DIP:DIP-14_W7.62mm_Socket_LongPads" H 10250 18250 50  0001 C CNN
 F 3 "https://assets.nexperia.com/documents/data-sheet/74HC_HCT04.pdf" H 10250 18250 50  0001 C CNN
-	6    10250 18250
+	3    10250 18250
 	0    1    1    0
 $EndComp
@@
 $Comp
 L 74xx:74HCT04 ROM_NOR?
-U 5 1 635AA7C1
+U 2 1 635AA7C1
 P 9750 18250
 F 0 "ROM_NOR?" H 9750 17933 50  0000 C CNN
@@
 F 2 "Package_DIP:DIP-14_W7.62mm_Socket_LongPads" H 9750 18250 50  0001 C CNN
 F 3 "https://assets.nexperia.com/documents/data-sheet/74HC_HCT04.pdf" H 9750 18250 50  0001 C CNN
-	5    9750 18250
+	2    9750 18250
 	0    1    1    0
 $EndComp
 $Comp
 L 74xx:74HCT04 ROM_NOR?
-U 4 1 635AA7C7
+U 1 1 635AA7C7
 P 9300 18250
 F 0 "ROM_NOR?" H 9300 17933 50  0000 C CNN
@@
 F 2 "Package_DIP:DIP-14_W7.62mm_Socket_LongPads" H 9300 18250 50  0001 C CNN
 F 3 "https://assets.nexperia.com/documents/data-sheet/74HC_HCT04.pdf" H 9300 18250 50  0001 C CNN
-	4    9300 18250
+	1    9300 18250
 	0    1    1    0
 $EndComp
@@
 	9300 18550 9400 18550
 Text Notes 9000 17300 0    50   ~ 0
-Read-Only Memory\nROM bank 4 high
+Read-Only Memory\nBank 3 high
 Wire Wire Line
 	4150 17100 4150 17300
@@
 $Comp
 L 74xx:74HCT04 ROM_NOR?
-U 3 1 635AA7EC
+U 6 1 635AA7EC
 P 6700 18250
 F 0 "ROM_NOR?" H 6700 17933 50  0000 C CNN
@@
 F 2 "Package_DIP:DIP-14_W7.62mm_Socket_LongPads" H 6700 18250 50  0001 C CNN
 F 3 "https://assets.nexperia.com/documents/data-sheet/74HC_HCT04.pdf" H 6700 18250 50  0001 C CNN
-	3    6700 18250
+	6    6700 18250
 	0    1    1    0
 $EndComp
 $Comp
 L 74xx:74HCT04 ROM_NOR?
-U 2 1 635AA7F2
+U 5 1 635AA7F2
 P 6200 18250
 F 0 "ROM_NOR?" H 6200 17933 50  0000 C CNN
@@
 F 2 "Package_DIP:DIP-14_W7.62mm_Socket_LongPads" H 6200 18250 50  0001 C CNN
 F 3 "https://assets.nexperia.com/documents/data-sheet/74HC_HCT04.pdf" H 6200 18250 50  0001 C CNN
-	2    6200 18250
+	5    6200 18250
 	0    1    1    0
 $EndComp
 $Comp
 L 74xx:74HCT04 ROM_NOR?
-U 1 1 635AA7F8
+U 4 1 635AA7F8
 P 5750 18250
 F 0 "ROM_NOR?" H 5750 17933 50  0000 C CNN
@@
 F 2 "Package_DIP:DIP-14_W7.62mm_Socket_LongPads" H 5750 18250 50  0001 C CNN
 F 3 "https://assets.nexperia.com/documents/data-sheet/74HC_HCT04.pdf" H 5750 18250 50  0001 C CNN
-	1    5750 18250
+	4    5750 18250
 	0    1    1    0
 $EndComp
@@
 	12550 18550 12650 18550
 Text Notes 12250 17300 0    50   ~ 0
-Read-Only Memory\nROM bank 4 high
+Read-Only Memory\nBank 4 high
 Wire Wire Line
 	14500 17100 14500 17300
@@
 Wire Notes Line
 	1800 19950 15550 19950
+Wire Wire Line
+	6150 7050 7350 7050
+Wire Wire Line
+	7000 7000 6600 7000
+Wire Wire Line
+	6600 7000 6600 5750
 $EndSCHEMATC
