File: Motherboard/Motherboard.kicad_pcb (KiCad board)
At the start: 8 copper layers, 508 x 330.2 mm, 192 parts, among them J1 Jack-DC_18v, J2 65SIB_Connector, J3 DB9_Header, J4 GPIO_Connector, J5 Expansion_Connector, J6 Expansion_Connector, J7 Expansion_Connector, J8 Expansion_Connector, J9 Expansion_Connector, P1 POWER TERMINAL, Q1 2N3055, Q2 TIC106, SW1 SW_DPDT, SW2 FUSE RESET, SW3 PROCESSOR RESET, U1 LM7812_TO220, U13 LM386, U14 LM7912_TO220, U4 LM7805_TO220, X1 ACO-8MHz

Commit message: 488 traces to go...
Routing:
- net ~CS_DEV: track 509.1 -> 871.6 mm, vias 11 -> 15
- net MEM_D3: track 146.5 -> 250.9 mm
- net A9: track 144.9 -> 247.5 mm
- net A11: track 402.5 -> 505.1 mm
- net A5: track 162.3 -> 264.6 mm
- net A6: track 157.5 -> 259.8 mm
- net A4: track 168.6 -> 270.9 mm
- net A7: track 177.8 -> 280.1 mm
- net A3: track 163.8 -> 266.1 mm
- net ~RAM_OE: track 0.00 -> 102.1 mm
- net A8: track 177.8 -> 279.8 mm
- net A13: track 407.0 -> 509.0 mm

Commit message: 480 traces left to go...
Routing:
- net GND: track 2783.6 -> 2908.5 mm
- net VCC: track 3533.5 -> 3651.6 mm
Changed lines of the file:
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@@
     (thickness 4)
     (drawings 14)
-    (tracks 2928)
+    (tracks 2952)
     (zones 0)
     (modules 192)
@@
   (segment (start 383.54 87.376) (end 383.54 95.885) (width 0.25) (layer GND.Cu) (net 1))
   (segment (start 383.54 84.455) (end 383.54 87.376) (width 0.25) (layer GND.Cu) (net 1))
+  (segment (start 407.71 206.375) (end 407.035 206.375) (width 0.25) (layer GND.Cu) (net 1))
+  (segment (start 413.425 212.09) (end 413.425 208.367) (width 0.25) (layer GND.Cu) (net 1))
+  (segment (start 438.785 208.28) (end 445.008 208.28) (width 0.25) (layer GND.Cu) (net 1))
+  (segment (start 445.008 211.963) (end 445.135 212.09) (width 0.25) (layer GND.Cu) (net 1))
+  (segment (start 445.008 208.28) (end 445.008 211.963) (width 0.25) (layer GND.Cu) (net 1))
+  (segment (start 464.185 282.575) (end 457.835 282.575) (width 0.25) (layer GND.Cu) (net 1))
+  (segment (start 464.312 282.448) (end 464.185 282.575) (width 0.25) (layer GND.Cu) (net 1))
+  (segment (start 464.312 233.767) (end 464.225 233.68) (width 0.25) (layer GND.Cu) (net 1))
+  (segment (start 464.312 282.448) (end 464.312 233.767) (width 0.25) (layer GND.Cu) (net 1))
+  (segment (start 414.06 234.315) (end 414.06 282.408) (width 0.25) (layer GND.Cu) (net 1))
+  (segment (start 413.923 282.545) (end 407.155 282.545) (width 0.25) (layer GND.Cu) (net 1))
+  (segment (start 414.06 282.408) (end 413.923 282.545) (width 0.25) (layer GND.Cu) (net 1))
   (segment (start 247.0404 104.8004) (end 247.0404 118.7196) (width 1) (layer GND.Cu) (net 2) (status 10))
   (segment (start 247.015 118.745) (end 240.03 118.745) (width 1) (layer GND.Cu) (net 2) (status 20))
@@
   (segment (start 357.505 174.625) (end 357.505 173.355) (width 0.25) (layer VCC.Cu) (net 4) (status 20))
   (segment (start 390.525 174.625) (end 390.525 173.355) (width 0.25) (layer VCC.Cu) (net 4) (status 20))
-  (segment (start 390.525 174.625) (end 422.275 174.625) (width 0.25) (layer VCC.Cu) (net 4))
   (segment (start 422.275 174.625) (end 422.275 173.355) (width 0.25) (layer VCC.Cu) (net 4) (status 20))
-  (segment (start 422.275 174.625) (end 454.025 174.625) (width 0.25) (layer VCC.Cu) (net 4))
   (segment (start 454.025 174.625) (end 454.025 173.355) (width 0.25) (layer VCC.Cu) (net 4) (status 20))
   (segment (start 334.01 249.555) (end 334.01 252.095) (width 0.25) (layer VCC.Cu) (net 4) (status 20))
@@
   (segment (start 388.874 87.63) (end 389.128 87.884) (width 0.25) (layer VCC.Cu) (net 4))
   (segment (start 389.128 87.884) (end 389.128 91.44) (width 0.25) (layer VCC.Cu) (net 4))
+  (segment (start 415.925 174.879) (end 415.671 174.625) (width 0.25) (layer VCC.Cu) (net 4))
+  (segment (start 415.925 212.09) (end 415.925 174.879) (width 0.25) (layer VCC.Cu) (net 4))
+  (segment (start 415.671 174.625) (end 422.275 174.625) (width 0.25) (layer VCC.Cu) (net 4))
+  (segment (start 390.525 174.625) (end 415.671 174.625) (width 0.25) (layer VCC.Cu) (net 4))
+  (segment (start 447.635 174.665) (end 447.675 174.625) (width 0.25) (layer VCC.Cu) (net 4))
+  (segment (start 447.675 174.625) (end 454.025 174.625) (width 0.25) (layer VCC.Cu) (net 4))
+  (segment (start 447.635 212.09) (end 447.635 174.665) (width 0.25) (layer VCC.Cu) (net 4))
+  (segment (start 422.275 174.625) (end 447.675 174.625) (width 0.25) (layer VCC.Cu) (net 4))
+  (segment (start 466.725 233.68) (end 466.725 249.301) (width 0.25) (layer VCC.Cu) (net 4))
+  (segment (start 466.979 249.555) (end 473.075 249.555) (width 0.25) (layer VCC.Cu) (net 4))
+  (segment (start 466.725 249.301) (end 466.979 249.555) (width 0.25) (layer VCC.Cu) (net 4))
+  (segment (start 416.56 234.315) (end 416.56 249.428) (width 0.25) (layer VCC.Cu) (net 4))
+  (segment (start 422.298 249.428) (end 422.395 249.525) (width 0.25) (layer VCC.Cu) (net 4))
+  (segment (start 416.56 249.428) (end 422.298 249.428) (width 0.25) (layer VCC.Cu) (net 4))
   (via (at 155.575 160.655) (size 0.8) (drill 0.4) (layers SIGH.Cu SIGV.Cu) (net 5))
   (segment (start 155.5496 160.6804) (end 155.575 160.655) (width 0.25) (layer SIGH.Cu) (net 5))

Commit message: A lot closer now...
Routing:
- net 8MHz: track 169.5 -> 589.2 mm, vias 4 -> 11
- net VCC: track 3651.6 -> 3832.8 mm
- net GND: track 2908.5 -> 3041.8 mm
- net R\~W: track 968.2 -> 1078.7 mm, vias 11 -> 14
- net A10: track 108.6 -> 211.5 mm
- net A2: track 373.3 -> 475.6 mm
- net Net-(RAM_NAND2-Pad4): track 0.00 -> 59.6 mm, vias 0 -> 4
- net Net-(RAM_NAND2-Pad1): track 0.00 -> 59.6 mm, vias 0 -> 4
- net Net-(RAM_NAND1-Pad5): track 0.00 -> 22.6 mm, vias 0 -> 2
- net ~IRQ0: track 513.7 -> 504.1 mm, vias 6 -> 5
- net -12v: track 821.8 -> 819.0 mm
- net +12v: track 739.6 -> 738.8 mm

Commit message: Removed some old 2.2 files...
Routing:
- net Net-(IRQ_NOR1-Pad3): track 0.00 -> 442.5 mm, vias 0 -> 4
- net Net-(IRQ_NOR1-Pad2): track 0.00 -> 416.0 mm, vias 0 -> 4

Commit message: 420 traces to go...
420! 420!! 420!!!
Connections:
- CLK_DIV1 pad 14: (no net) -> VCC
- CLK_DIV1 pad 7: (no net) -> GND
Routing:
- net A1: track 108.5 -> 482.8 mm, vias 0 -> 5
- net A0: track 108.5 -> 379.6 mm, vias 0 -> 3
- net GND: track 3041.8 -> 3234.0 mm
- net A2: track 475.6 -> 582.2 mm, vias 7 -> 8
- net A3: track 266.1 -> 368.1 mm, vias 3 -> 4
- net CS_GPIO: track 0.00 -> 86.1 mm, vias 0 -> 4
- net A4: track 270.9 -> 354.2 mm, vias 1 -> 4
- net VCC: track 3832.8 -> 3914.6 mm
- net Net-(CS_UART_AND4-Pad2): track 0.00 -> 72.6 mm, vias 0 -> 4
- net MEM_D0: track 147.2 -> 203.7 mm, vias 0 -> 2
- net A5: track 264.6 -> 316.1 mm, vias 1 -> 4
- net A6: track 259.8 -> 309.9 mm, vias 2 -> 5
- net Net-(CS_UART_AND4-Pad1): track 0.00 -> 45.0 mm, vias 0 -> 4
- net CPU_D2: track 62.2 -> 105.1 mm, vias 2 -> 4
- net CPU_D4: track 41.9 -> 80.1 mm, vias 0 -> 2
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
Commit message: 202 traces until 2.3...
Parts:
- 12v1: value 12v INDICATOR -> +12v INDICATOR
- 5v1: value 5v INDICATOR -> +5v INDICATOR
Routing:
- net MEM_D0: track 203.7 -> 1006.0 mm, vias 2 -> 10
- net A3: track 368.1 -> 917.8 mm, vias 4 -> 7
- net A4: track 354.2 -> 897.9 mm, vias 4 -> 10
- net MEM_D1: track 146.5 -> 643.6 mm, vias 0 -> 4
- net MEM_D2: track 146.5 -> 642.4 mm, vias 0 -> 4
- net MEM_D4: track 146.9 -> 620.8 mm, vias 0 -> 4
- net MEM_D5: track 146.5 -> 616.1 mm, vias 0 -> 4
- net MEM_D6: track 146.6 -> 612.2 mm, vias 0 -> 4
- net MEM_D7: track 146.5 -> 606.4 mm, vias 0 -> 4
- net A10: track 241.3 -> 649.1 mm, vias 1 -> 4
- net MEM_D3: track 250.9 -> 628.9 mm, vias 0 -> 4
- net A9: track 280.4 -> 650.0 mm, vias 4 -> 8
- net RAM4_EN: track 0.00 -> 360.5 mm, vias 0 -> 2
- net RAM3_EN: track 0.00 -> 349.8 mm, vias 0 -> 2
- net RAM1_EN: track 0.00 -> 348.0 mm, vias 0 -> 2
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
Commit message: 168 traces to go...
Routing:
- net A5: track 524.9 -> 987.5 mm, vias 4 -> 9
- net A12: track 445.4 -> 816.3 mm, vias 1 -> 3
- net MEM_D1: track 643.6 -> 872.3 mm, vias 4 -> 8
- net A15: track 676.4 -> 891.0 mm, vias 20 -> 22
- net A13: track 783.4 -> 988.9 mm, vias 24 -> 26
- net A14: track 455.3 -> 656.2 mm, vias 6 -> 7
- net MEM_D0: track 1006.0 -> 1201.9 mm, vias 10 -> 13
- net A9: track 650.0 -> 808.9 mm
- net A8: track 594.9 -> 753.4 mm
- net A6: track 624.0 -> 782.4 mm
- net A11: track 831.8 -> 990.2 mm
- net A4: track 897.9 -> 1055.9 mm
- net A7: track 602.1 -> 759.5 mm

Commit message: 156 unrouted traces...
Routing:
- net A10: track 649.1 -> 807.5 mm
- net A2: track 791.0 -> 949.1 mm
- net A3: track 917.8 -> 1075.9 mm
- net A1: track 792.2 -> 949.7 mm
Changed lines of the file:
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@@
     (thickness 4)
     (drawings 14)
-    (tracks 4716)
+    (tracks 4763)
     (zones 0)
     (modules 192)
@@
   (segment (start 320.7004 334.6704) (end 320.7004 335.788) (width 0.25) (layer SIGV.Cu) (net 57))
   (segment (start 371.348 335.788) (end 320.548 335.788) (width 0.25) (layer SIGV.Cu) (net 57))
+  (segment (start 473.075 267.335) (end 473.075 268.605) (width 0.25) (layer SIGV.Cu) (net 57))
+  (segment (start 473.075 268.605) (end 472.948 268.732) (width 0.25) (layer SIGV.Cu) (net 57))
+  (segment (start 472.948 268.732) (end 422.148 268.732) (width 0.25) (layer SIGV.Cu) (net 57))
+  (segment (start 422.148 267.552) (end 422.395 267.305) (width 0.25) (layer SIGV.Cu) (net 57))
+  (segment (start 422.148 268.732) (end 422.148 267.552) (width 0.25) (layer SIGV.Cu) (net 57))
+  (segment (start 371.348 268.732) (end 422.148 268.732) (width 0.25) (layer SIGV.Cu) (net 57))
+  (segment (start 371.348 267.432) (end 371.348 268.732) (width 0.25) (layer SIGV.Cu) (net 57))
+  (segment (start 371.475 267.305) (end 371.348 267.432) (width 0.25) (layer SIGV.Cu) (net 57))
+  (segment (start 371.348 268.732) (end 320.548 268.732) (width 0.25) (layer SIGV.Cu) (net 57))
+  (segment (start 320.548 267.457) (end 320.7 267.305) (width 0.25) (layer SIGV.Cu) (net 57))
+  (segment (start 320.548 268.732) (end 320.548 267.457) (width 0.25) (layer SIGV.Cu) (net 57))
   (via (at 215.9 342.9) (size 0.8) (drill 0.4) (layers SIGH.Cu SIGV.Cu) (net 58))
   (segment (start 222.9104 342.9) (end 215.9 342.9) (width 0.25) (layer SIGH.Cu) (net 58) (status 10))
@@
   (segment (start 508.508 333.248) (end 508.508 332.2828) (width 0.25) (layer SIGH.Cu) (net 70))
   (segment (start 457.708 333.248) (end 508.508 333.248) (width 0.25) (layer SIGH.Cu) (net 70))
+  (segment (start 356.108 266.192) (end 356.108 264.892) (width 0.25) (layer SIGH.Cu) (net 70))
+  (segment (start 305.612 266.192) (end 356.108 266.192) (width 0.25) (layer SIGH.Cu) (net 70))
+  (segment (start 356.108 264.892) (end 356.235 264.765) (width 0.25) (layer SIGH.Cu) (net 70))
+  (segment (start 305.46 266.04) (end 305.612 266.192) (width 0.25) (layer SIGH.Cu) (net 70))
+  (segment (start 305.46 264.765) (end 305.46 266.04) (width 0.25) (layer SIGH.Cu) (net 70))
+  (segment (start 406.908 265.012) (end 407.155 264.765) (width 0.25) (layer SIGH.Cu) (net 70))
+  (segment (start 406.908 266.192) (end 406.908 265.012) (width 0.25) (layer SIGH.Cu) (net 70))
+  (segment (start 356.108 266.192) (end 406.908 266.192) (width 0.25) (layer SIGH.Cu) (net 70))
+  (segment (start 406.908 266.192) (end 457.708 266.192) (width 0.25) (layer SIGH.Cu) (net 70))
+  (segment (start 457.708 264.922) (end 457.835 264.795) (width 0.25) (layer SIGH.Cu) (net 70))
+  (segment (start 457.708 266.192) (end 457.708 264.922) (width 0.25) (layer SIGH.Cu) (net 70))
   (segment (start 522.6304 57.8104) (end 522.6304 59.0296) (width 0.25) (layer SIGV.Cu) (net 71) (status 10))
   (segment (start 522.6304 59.0296) (end 522.605 59.055) (width 0.25) (layer SIGV.Cu) (net 71))
@@
   (segment (start 508.508 334.8228) (end 508.6604 334.6704) (width 0.25) (layer SIGH.Cu) (net 72))
   (segment (start 508.508 335.788) (end 508.508 334.8228) (width 0.25) (layer SIGH.Cu) (net 72))
+  (segment (start 356.235 268.321) (end 356.235 267.305) (width 0.25) (layer SIGH.Cu) (net 72))
+  (segment (start 356.235 268.351) (end 356.235 268.321) (width 0.25) (layer SIGH.Cu) (net 72))
+  (segment (start 356.474 268.59) (end 356.235 268.351) (width 0.25) (layer SIGH.Cu) (net 72))
+  (segment (start 305.46 268.58) (end 305.47 268.59) (width 0.25) (layer SIGH.Cu) (net 72))
+  (segment (start 305.46 267.305) (end 305.46 268.58) (width 0.25) (layer SIGH.Cu) (net 72))
+  (segment (start 305.47 268.59) (end 356.25 268.59) (width 0.25) (layer SIGH.Cu) (net 72))
+  (segment (start 356.25 268.59) (end 356.474 268.59) (width 0.25) (layer SIGH.Cu) (net 72))
+  (segment (start 406.908 267.552) (end 407.155 267.305) (width 0.25) (layer SIGH.Cu) (net 72))
+  (segment (start 406.908 268.732) (end 406.908 267.552) (width 0.25) (layer SIGH.Cu) (net 72))
+  (segment (start 371.124 268.732) (end 406.908 268.732) (width 0.25) (layer SIGH.Cu) (net 72))
+  (segment (start 370.982 268.59) (end 371.124 268.732) (width 0.25) (layer SIGH.Cu) (net 72))
+  (segment (start 356.25 268.59) (end 370.982 268.59) (width 0.25) (layer SIGH.Cu) (net 72))
+  (segment (start 406.908 268.732) (end 457.708 268.732) (width 0.25) (layer SIGH.Cu) (net 72))
+  (segment (start 457.708 267.462) (end 457.835 267.335) (width 0.25) (layer SIGH.Cu) (net 72))
+  (segment (start 457.708 268.732) (end 457.708 267.462) (width 0.25) (layer SIGH.Cu) (net 72))
   (segment (start 497.205 56.515) (end 497.205 55.2958) (width 0.25) (layer SIGV.Cu) (net 73) (status 20))
   (segment (start 522.605 56.515) (end 497.205 56.515) (width 0.25) (layer SIGV.Cu) (net 73))
@@
   (segment (start 508.43541 338.25541) (end 508.43541 337.43539) (width 0.25) (layer SIGH.Cu) (net 74))
   (segment (start 457.63541 338.25541) (end 508.43541 338.25541) (width 0.25) (layer SIGH.Cu) (net 74))
+  (segment (start 305.46 269.845) (end 305.46 271.12) (width 0.25) (layer SIGH.Cu) (net 74))
+  (segment (start 305.46 271.12) (end 356.26 271.12) (width 0.25) (layer SIGH.Cu) (net 74))
+  (segment (start 356.235 271.095) (end 356.235 269.845) (width 0.25) (layer SIGH.Cu) (net 74))
+  (segment (start 356.26 271.12) (end 356.235 271.095) (width 0.25) (layer SIGH.Cu) (net 74))
+  (segment (start 356.26 271.12) (end 407.264 271.12) (width 0.25) (layer SIGH.Cu) (net 74))
+  (segment (start 407.155 271.011) (end 407.155 269.845) (width 0.25) (layer SIGH.Cu) (net 74))
+  (segment (start 407.264 271.12) (end 407.155 271.011) (width 0.25) (layer SIGH.Cu) (net 74))
+  (segment (start 407.264 271.12) (end 457.86 271.12) (width 0.25) (layer SIGH.Cu) (net 74))
+  (segment (start 457.835 271.095) (end 457.835 269.875) (width 0.25) (layer SIGH.Cu) (net 74))
+  (segment (start 457.86 271.12) (end 457.835 271.095) (width 0.25) (layer SIGH.Cu) (net 74))
   (segment (start 497.205 52.7558) (end 497.2304 52.7304) (width 0.25) (layer SIGV.Cu) (net 75) (status 30))
   (segment (start 497.205 53.975) (end 497.205 52.7558) (width 0.25) (layer SIGV.Cu) (net 75) (status 20))
