File: Motherboard/Motherboard.kicad_sch (KiCad schematic)
At the start: 140 parts, among them J2 65SIB_Connector, J3 DB9_Header, J4 GPIO_Connector, J5 Expansion_Connector, J6 Expansion_Connector, J7 Expansion_Connector, J8 Expansion_Connector, J9 Expansion_Connector, X1 ACO-8MHz

Commit message: 2.5 schematic complete...
Parts:
- removed C34, C35, C36, C37, C38, C39, C40, C41, C42, C43, C44, C45, C46, C47, C48, C49, C50, C51, C52, C53, C54, C55, C56, C57, C58: 100 nF, Capacitor_THT:C_Disc_D3.0mm_W1.6mm_P2.50mm, symbol Device:C
- removed CS_65SIB_AND1, CS_GPIO_AND1, CS_UART_AND1, IRQ_RW_AND1: 74HCT08, Package_DIP:DIP-14_W7.62mm_Socket_LongPads, symbol 74xx:74LS08
- removed CS_65SIB_AND4, CS_GPIO_AND4, CS_UART_AND4: 74HCT21, Package_DIP:DIP-14_W7.62mm_Socket_LongPads, symbol 74xx:74LS21
- removed CS_65SIB_NOR1, CS_GPIO_NOR1, CS_UART_NOR1, CS_VID_NOR1, RAM_NOR1, ~MAX235_EN1: 74HCT04, Package_DIP:DIP-14_W7.62mm_Socket_LongPads, symbol 74xx:74HCT04
- removed CS_VID_NAND1: 74HCT00, Package_DIP:DIP-14_W7.62mm_Socket_LongPads, symbol 74xx:74HCT00
- removed unit 1 of IRQ_NOR1
- added U10, U4, U5, U8: 74HCT138, Package_DIP:DIP-16_W7.62mm_Socket_LongPads, symbol 74xx:74LS138
- added unit 2 of U7
- PWR_OK1: renamed from PWR_OK; footprint (none) -> LED_THT:LED_D5.0mm
- R10: renamed from R?; value PWR220T-20-1R00J -> PWR220T-20-5R00J; footprint Resistor_THT:R_Axial_DIN0207_L6.3mm_D2.5mm_P7.62mm_Horizontal -> Package_TO_SOT_THT:TO-220-2_Horizontal_TabDown
- U1, U3, U9: renamed from U?; value 74LS138 -> 74HCT138; footprint (none) -> Package_DIP:DIP-16_W7.62mm_Socket_LongPads
- U6: renamed from U?; footprint (none) -> Socket:DIP_Socket-32_W11.9_W12.7_W15.24_W17.78_W18.5_3M_232-1285-00-0602J
- U7: renamed from U?; value 74LS08 -> 74HCT08; footprint (none) -> Package_DIP:DIP-14_W7.62mm_Socket_LongPads
- gave numbers to parts that had none: 6
- renumbered IRQ_NOR1 to NOR1, RESET_NOR1 to NOR1
Connections:
- net VID_OE is gone; now on net ~{RAM_OE}: VID_DECODER1.22 (~{OE})
- net +12v: now also J5.36 (Pin_36), J6.36 (Pin_36), J7.36 (Pin_36), J8.36 (Pin_36), J9.36 (Pin_36); no longer J5.42 (Pin_42), J6.42 (Pin_42), J7.42 (Pin_42), J8.42 (Pin_42), J9.42 (Pin_42)
- net -12v: now also J5.38 (Pin_38), J6.38 (Pin_38), J7.38 (Pin_38), J8.38 (Pin_38), J9.38 (Pin_38); no longer J5.40 (Pin_40), J6.40 (Pin_40), J7.40 (Pin_40), J8.40 (Pin_40), J9.40 (Pin_40)
- net A4: now also U10.1 (A0), U4.1 (A0), U8.1 (A0)
- net A5: now also U10.2 (A1), U4.2 (A1), U8.2 (A1)
- net A6: now also U10.3 (A2), U4.3 (A2), U8.3 (A2)
- net A7: now also U10.6 (E3), U4.6 (E3), U8.5 (E2)
- net BE: now also R11.2; no longer R11.1
- net CS_65SIB: no longer 65SIB_LATCH1.6 (E2)
- net CS_GPIO: now also U8.12 (O3)
- net GND: now also U10.4 (E1), U10.5 (E2), U10.8 (GND), U4.4 (E1), U4.5 (E2), U4.8 (GND), U5.2 (A1), U5.3 (A2), U5.4 (E1), U5.5 (E2), U5.8 (GND), U8.4 (E1), U8.8 (GND)
- net RDY: now also J5.30 (Pin_30), J6.30 (Pin_30), J7.30 (Pin_30), J8.30 (Pin_30), J9.30 (Pin_30); no longer J5.39 (Pin_39), J6.39 (Pin_39), J7.39 (Pin_39), J8.39 (Pin_39), J9.39 (Pin_39)
- net R\~{W}: now also U5.1 (A0)
- net SYNC: now also J5.32 (Pin_32), J6.32 (Pin_32), J7.32 (Pin_32), J8.32 (Pin_32), J9.32 (Pin_32); no longer J5.41 (Pin_41), J6.41 (Pin_41), J7.41 (Pin_41), J8.41 (Pin_41), J9.41 (Pin_41)
- net VCC: now also R11.1, U10.16 (VCC), U4.16 (VCC), U5.16 (VCC), U8.16 (VCC), U8.6 (E3)
- net ~{IRQ3}: now also J9.34 (Pin_34); no longer J5.30 (Pin_30), J6.30 (Pin_30), J7.30 (Pin_30), J8.30 (Pin_30), J9.30 (Pin_30)
- net ~{IRQ4}: now also J5.34 (Pin_34); no longer J5.32 (Pin_32), J6.32 (Pin_32), J7.32 (Pin_32), J8.32 (Pin_32), J9.32 (Pin_32)
- net ~{IRQ5}: no longer J5.34 (Pin_34), J7.34 (Pin_34), J8.34 (Pin_34), J9.34 (Pin_34)
- net ~{IRQ6}: now also J7.34 (Pin_34); no longer J5.36 (Pin_36), J6.36 (Pin_36), J7.36 (Pin_36), J8.36 (Pin_36), J9.36 (Pin_36)
- net ~{IRQ7}: now also J8.34 (Pin_34); no longer J5.38 (Pin_38), J6.38 (Pin_38), J7.38 (Pin_38), J8.38 (Pin_38), J9.38 (Pin_38)
- net ~{RAM_WE}: now also VID_BUFFER1.1 (G1), VID_BUFFER1.19 (G2)
- net at IRQ_MASK1.11 (Cp): now also U5.15 (O0)
- net at IRQ_PRIORITY1.1 (OE): now also U5.14 (O1)
- net ~{CS_UART}: now reaches UART-RS232.20 (~{En})
- net ~{CS_UART}: now also UART1.3 (~{CS1}), U4.14 (O1)
- net CS_UART renamed CS_DEV
- net CS_DEV: now also 65SIB/MM1.23 (~{CS2}), 65SIB_LATCH1.6 (E2), GPIO_CTRL1.23 (~{CS2}), J5.28 (Pin_28), J6.28 (Pin_28), J7.28 (Pin_28), J8.28 (Pin_28), J9.28 (Pin_28), U5.6 (E3), U7.6
- removed net ~{CS_DEV}: 65SIB/MM1.23 (~{CS2}), 65SIB_LATCH1.5 (~{E1}), GPIO_CTRL1.23 (~{CS2}), J5.28 (Pin_28), J6.28 (Pin_28), J7.28 (Pin_28), J8.28 (Pin_28), J9.28 (Pin_28), UART1.3 (~{CS1}), ~CS_DEV1.10 (O5), ~CS_DEV2.15 (O0)
- new net: U7.5, ~CS_DEV1.10 (O5)
- new net: U7.4, ~CS_DEV2.15 (O0)
- new net ~{CS_65SIB}: 65SIB_LATCH1.5 (~{E1}), U10.13 (O2)
- no-connect marks 53 -> 79
Other:
- moved on the sheet: H1, H2, H3, H4, H5, H6, J1, PWR_OK1, R10, R11, R9, SW1

Commit message: Road to 2.5 release...
Parts:
- added C1, C2: 100 nF, Capacitor_THT:C_Disc_D3.0mm_W1.6mm_P2.50mm, symbol Device:C
Connections:
- net GND: now also C1.2, C2.2
- net VCC: now also C1.1, C2.1
- net BE: no longer names the net of CPU1.36 (BE), R11.2
Other:
- moved on the sheet: CPU1, IRQ_EN1, NMI_EN1, R11, R18, R19, R20, VP_GND1

Commit message: Started on 2.5 PCB...
Parts:
- 65SIB/MM1, CPU1, GPIO_CTRL1: footprint Socket:DIP_Socket-40_W11.9_W12.7_W15.24_W17.78_W18.5_3M_240-1280-00-0602J -> Package_DIP:DIP-40_W15.24mm_Socket_LongPads
- J1: value ATX-24 -> ATX-20; footprint (none) -> Connector_Molex:Molex_Mini-Fit_Jr_5566-20A_2x10_P4.20mm_Vertical; symbol Connector:ATX-24 -> Connector:ATX-20
- UART1: footprint Socket:DIP_Socket-28_W11.9_W12.7_W15.24_W17.78_W18.5_3M_228-1277-00-0602J -> Package_DIP:DIP-28_W15.24mm_Socket_LongPads
Connections:
- net +12v: no longer J1.11 (+12V)
- net -12v: now also J1.12 (-12V); no longer J1.14 (-12V)
- net GND: now also J1.13 (GND), J1.16 (GND); no longer J1.18 (GND), J1.19 (GND), J1.24 (GND)
- net VCC: now also J1.19 (+5V), J1.20 (+5V); no longer J1.21 (+5V), J1.22 (+5V), J1.23 (+5V)
- net at SW1.2 (B): now also J1.14 (PS_ON#); no longer J1.16 (PS_ON#)
- net at J1.1 (+3.3V), J1.2 (+3.3V): now also J1.11 (+3.3V); no longer J1.12 (+3.3V), J1.13 (+3.3V)
- no-connect marks 79 -> 80
Changed lines of the file:
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@@
   (no_connect (at 257.81 157.48))
   (no_connect (at 257.81 160.02))
+  (no_connect (at 186.69 147.32))
   (no_connect (at 78.74 83.82))
   (no_connect (at 123.19 143.51))
@@
       (effects (font (size 1.524 1.524)))
     )
-    (property "Footprint" "Socket:DIP_Socket-40_W11.9_W12.7_W15.24_W17.78_W18.5_3M_240-1280-00-0602J" (id 2) (at 93.98 148.59 0)
+    (property "Footprint" "Package_DIP:DIP-40_W15.24mm_Socket_LongPads" (id 2) (at 93.98 148.59 0)
       (effects (font (size 1.524 1.524)) hide)
     )
@@
       (effects (font (size 1.524 1.524)))
     )
-    (property "Footprint" "Socket:DIP_Socket-40_W11.9_W12.7_W15.24_W17.78_W18.5_3M_240-1280-00-0602J" (id 2) (at 63.5 267.97 0)
+    (property "Footprint" "Package_DIP:DIP-40_W15.24mm_Socket_LongPads" (id 2) (at 63.5 267.97 0)
       (effects (font (size 1.524 1.524)) hide)
     )
@@
       (effects (font (size 1.524 1.524)))
     )
-    (property "Footprint" "Socket:DIP_Socket-40_W11.9_W12.7_W15.24_W17.78_W18.5_3M_240-1280-00-0602J" (id 2) (at 631.19 224.79 0)
+    (property "Footprint" "Package_DIP:DIP-40_W15.24mm_Socket_LongPads" (id 2) (at 631.19 224.79 0)
       (effects (font (size 1.524 1.524)) hide)
     )
@@
       (effects (font (size 1.524 1.524)))
     )
-    (property "Footprint" "Socket:DIP_Socket-28_W11.9_W12.7_W15.24_W17.78_W18.5_3M_228-1277-00-0602J" (id 2) (at 425.45 66.04 0)
+    (property "Footprint" "Package_DIP:DIP-28_W15.24mm_Socket_LongPads" (id 2) (at 425.45 66.04 0)
       (effects (font (size 1.524 1.524)) hide)
     )
@@
   (symbol (lib_id "WolfNet:LOGO") (at 411.48 320.04 0) (unit 1)
     (in_bom yes) (on_board yes)
-    (property "Reference" "#G?" (id 0) (at 411.48 325.2216 0)
+    (property "Reference" "#G1" (id 0) (at 411.48 325.2216 0)
       (effects (font (size 1.524 1.524)) hide)
     )
@@
     (pin "9")
   )
-  (symbol (lib_id "Connector:ATX-24") (at 173.99 139.7 0) (unit 1)
+  (symbol (lib_id "Connector:ATX-20") (at 173.99 139.7 0) (unit 1)
     (in_bom yes) (on_board yes) (fields_autoplaced)
     (property "Reference" "J1" (id 0) (at 173.99 123.3002 0))
-    (property "Value" "ATX-24" (id 1) (at 173.99 125.8371 0))
-    (property "Footprint" "" (id 2) (at 173.99 142.24 0)
+    (property "Value" "ATX-20" (id 1) (at 173.99 125.8371 0))
+    (property "Footprint" "Connector_Molex:Molex_Mini-Fit_Jr_5566-20A_2x10_P4.20mm_Vertical" (id 2) (at 173.99 142.24 0)
       (effects (font (size 1.27 1.27)) hide)
     )
-    (property "Datasheet" "https://www.intel.com/content/dam/www/public/us/en/documents/guides/power-supply-design-guide-june.pdf#page=33" (id 3) (at 234.95 153.67 0)
+    (property "Datasheet" "https://web.aub.edu.lb/pub/docs/atx_201.pdf#page=20" (id 3) (at 201.93 153.67 0)
       (effects (font (size 1.27 1.27)) hide)
     )
@@
     (pin "2")
     (pin "20")
-    (pin "21")
-    (pin "22")
-    (pin "23")
-    (pin "24")
     (pin "3")
     (pin "4")
@@
   (symbol_instances
     (path "/00000000-0000-0000-0000-000062809309"
-      (reference "#G?") (unit 1) (value "~") (footprint "WolfNet:WolfNet-Logo_silkscreen")
+      (reference "#G1") (unit 1) (value "~") (footprint "WolfNet:WolfNet-Logo_silkscreen")
     )
     (path "/00000000-0000-0000-0000-000061c12325"
@@
     )
     (path "/00000000-0000-0000-0000-000061c6031f"
-      (reference "65SIB/MM1") (unit 1) (value "WD65C22") (footprint "Socket:DIP_Socket-40_W11.9_W12.7_W15.24_W17.78_W18.5_3M_240-1280-00-0602J")
+      (reference "65SIB/MM1") (unit 1) (value "WD65C22") (footprint "Package_DIP:DIP-40_W15.24mm_Socket_LongPads")
     )
     (path "/00000000-0000-0000-0000-00006343fd00"
@@
     )
     (path "/00000000-0000-0000-0000-000061936e15"
-      (reference "CPU1") (unit 1) (value "WD65C02") (footprint "Socket:DIP_Socket-40_W11.9_W12.7_W15.24_W17.78_W18.5_3M_240-1280-00-0602J")
+      (reference "CPU1") (unit 1) (value "WD65C02") (footprint "Package_DIP:DIP-40_W15.24mm_Socket_LongPads")
     )
     (path "/00000000-0000-0000-0000-000061a772a1"
-      (reference "GPIO_CTRL1") (unit 1) (value "WD65C22") (footprint "Socket:DIP_Socket-40_W11.9_W12.7_W15.24_W17.78_W18.5_3M_240-1280-00-0602J")
+      (reference "GPIO_CTRL1") (unit 1) (value "WD65C22") (footprint "Package_DIP:DIP-40_W15.24mm_Socket_LongPads")
     )
     (path "/00000000-0000-0000-0000-00006483e48f"
@@
     )
     (path "/a8e3d340-f029-4539-9157-5cf54d8d3c01"
-      (reference "J1") (unit 1) (value "ATX-24") (footprint "")
+      (reference "J1") (unit 1) (value "ATX-20") (footprint "Connector_Molex:Molex_Mini-Fit_Jr_5566-20A_2x10_P4.20mm_Vertical")
     )
     (path "/00000000-0000-0000-0000-000061d1bdb7"
@@
     )
     (path "/00000000-0000-0000-0000-000061c6acb1"
-      (reference "UART1") (unit 1) (value "W65C51") (footprint "Socket:DIP_Socket-28_W11.9_W12.7_W15.24_W17.78_W18.5_3M_228-1277-00-0602J")
+      (reference "UART1") (unit 1) (value "W65C51") (footprint "Package_DIP:DIP-28_W15.24mm_Socket_LongPads")
     )
     (path "/00000000-0000-0000-0000-000061b94c4c"

Commit message: Almost finished 2.5 placements...
Parts:
- removed H3, H4: MountingHole, MountingHole:MountingHole_3.2mm_M3, symbol Mechanical:MountingHole
Changed lines of the file:
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@@
     (title "WolfNet 6502 WBC - Motherboard")
     (date "2022-05-06")
-    (rev "2.4")
+    (rev "2.5")
     (company "WolfNet Computing")
     (comment 1 "Motherboard for the WolfNet 65C02 based (NMOS Compatible) WorkBench Computer.")
@@
     )
   )
-  (symbol (lib_id "Mechanical:MountingHole") (at 459.74 337.82 0) (unit 1)
-    (in_bom yes) (on_board yes)
-    (property "Reference" "H4" (id 0) (at 462.28 336.6516 0)
-      (effects (font (size 1.27 1.27)) (justify left))
-    )
-    (property "Value" "MountingHole" (id 1) (at 462.28 338.963 0)
-      (effects (font (size 1.27 1.27)) (justify left))
-    )
-    (property "Footprint" "MountingHole:MountingHole_3.2mm_M3" (id 2) (at 459.74 337.82 0)
-      (effects (font (size 1.27 1.27)) hide)
-    )
-    (property "Datasheet" "~" (id 3) (at 459.74 337.82 0)
-      (effects (font (size 1.27 1.27)) hide)
-    )
-  )
-  (symbol (lib_id "Mechanical:MountingHole") (at 440.69 337.82 0) (unit 1)
-    (in_bom yes) (on_board yes)
-    (property "Reference" "H3" (id 0) (at 443.23 336.6516 0)
-      (effects (font (size 1.27 1.27)) (justify left))
-    )
-    (property "Value" "MountingHole" (id 1) (at 443.23 338.963 0)
-      (effects (font (size 1.27 1.27)) (justify left))
-    )
-    (property "Footprint" "MountingHole:MountingHole_3.2mm_M3" (id 2) (at 440.69 337.82 0)
-      (effects (font (size 1.27 1.27)) hide)
-    )
-    (property "Datasheet" "~" (id 3) (at 440.69 337.82 0)
-      (effects (font (size 1.27 1.27)) hide)
-    )
-  )
   (symbol (lib_id "Mechanical:MountingHole") (at 459.74 344.17 0) (unit 1)
     (in_bom yes) (on_board yes)
@@
       (reference "H2") (unit 1) (value "MountingHole") (footprint "MountingHole:MountingHole_3.2mm_M3")
     )
-    (path "/00000000-0000-0000-0000-00006483ec4b"
-      (reference "H3") (unit 1) (value "MountingHole") (footprint "MountingHole:MountingHole_3.2mm_M3")
-    )
-    (path "/00000000-0000-0000-0000-00006483ec45"
-      (reference "H4") (unit 1) (value "MountingHole") (footprint "MountingHole:MountingHole_3.2mm_M3")
-    )
     (path "/00000000-0000-0000-0000-000064893671"

Commit message: Finished 2.5 placement...
Parts:
- removed C32: 100 nF, Capacitor_THT:C_Disc_D3.0mm_W1.6mm_P2.50mm, symbol Device:C
- removed VP_GND1: VP_GND, Connector_PinHeader_2.54mm:PinHeader_1x02_P2.54mm_Vertical, symbol Jumper:Jumper_2_Open
- added unit 7 of NOR1
- added unit 5 of U7
Connections:
- net CS_DEV: now also GPIO_CTRL1.24 (CS1); no longer GPIO_CTRL1.23 (~{CS2})
- net GND: now also CPU1.1 (~{VP}), NOR1.7 (GND), U7.7 (GND)
- net VCC: now also NOR1.14 (VCC), U7.14 (VCC)
- net CS_GPIO renamed ~{CS_GPIO}
- net ~{CS_GPIO}: now also GPIO_CTRL1.23 (~{CS2}); no longer GPIO_CTRL1.24 (CS1)
Other:
- moved on the sheet: C1, C2, C33

Commit message: Bug fixes...
Parts:
- removed unit 2 of U7
- added U?: 74HCT02, symbol 74xx:74HCT02
- renumbered NOR1 to NOT1
Connections:
- net CS_DEV: now also U?.1
- net ~{CS_65SIB}: now also U10.11 (O4); no longer U10.13 (O2)
- net at ~CS_DEV1.10 (O5): now also U?.3
- net at ~CS_DEV2.15 (O0): now also U?.2
Other:
- note added: "RS-232 (Serial/UART) ports IRQ0 Address space: 0xD010 - 0xD013"
- note removed: "RS-232 (Serial/UART) ports IRQ0 Address space: 0xD014 - 0xD017"
Changed lines of the file:
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@@
   (no_connect (at 539.75 298.45))
   (no_connect (at 539.75 303.53))
-  (no_connect (at 539.75 306.07))
+  (no_connect (at 539.75 300.99))
   (no_connect (at 539.75 308.61))
   (no_connect (at 539.75 311.15))
@@
     (effects (font (size 1.27 1.27)) (justify right bottom))
   )
-  (text "RS-232 (Serial/UART) ports\nIRQ0\nAddress space: 0xD014 - 0xD017"
+  (text "RS-232 (Serial/UART) ports\nIRQ0\nAddress space: 0xD010 - 0xD013"
     (at 627.38 40.64 0)
     (effects (font (size 1.27 1.27)) (justify right bottom))
@@
     )
   )
-  (global_label "~{CS_65SIB}" (shape output) (at 539.75 300.99 0) (fields_autoplaced)
+  (global_label "~{CS_65SIB}" (shape output) (at 539.75 306.07 0) (fields_autoplaced)
     (effects (font (size 1.27 1.27)) (justify left))
-    (property "Intersheet References" "${INTERSHEET_REFS}" (id 0) (at 551.0247 300.9106 0)
+    (property "Intersheet References" "${INTERSHEET_REFS}" (id 0) (at 551.0247 305.9906 0)
       (effects (font (size 1.27 1.27)) (justify left) hide)
     )
@@
   (symbol (lib_id "74xx:74HCT04") (at 365.76 83.82 0) (unit 2)
     (in_bom yes) (on_board yes)
-    (property "Reference" "NOR1" (id 0) (at 365.76 75.7682 0))
+    (property "Reference" "NOT1" (id 0) (at 365.76 75.7682 0))
     (property "Value" "74HCT04" (id 1) (at 365.76 78.0796 0))
     (property "Footprint" "Package_DIP:DIP-14_W7.62mm_Socket_LongPads" (id 2) (at 365.76 83.82 0)
@@
   (symbol (lib_id "74xx:74HCT04") (at 119.38 193.04 0) (unit 1)
     (in_bom yes) (on_board yes)
-    (property "Reference" "NOR1" (id 0) (at 119.38 184.9882 0))
+    (property "Reference" "NOT1" (id 0) (at 119.38 184.9882 0))
     (property "Value" "74HCT04" (id 1) (at 119.38 187.2996 0))
     (property "Footprint" "Package_DIP:DIP-14_W7.62mm_Socket_LongPads" (id 2) (at 119.38 193.04 0)
@@
   (symbol (lib_id "74xx:74HCT04") (at 360.68 288.29 0) (unit 7)
     (in_bom yes) (on_board yes)
-    (property "Reference" "NOR1" (id 0) (at 369.57 287.02 0))
+    (property "Reference" "NOT1" (id 0) (at 369.57 287.02 0))
     (property "Value" "74HCT04" (id 1) (at 370.84 289.56 0))
     (property "Footprint" "Package_DIP:DIP-14_W7.62mm_Socket_LongPads" (id 2) (at 360.68 288.29 0)
@@
     (pin "7")
   )
-  (symbol (lib_id "74xx:74LS08") (at 548.64 265.43 270) (unit 2)
+  (symbol (lib_id "74xx:74HCT02") (at 548.64 265.43 270) (unit 1)
     (in_bom yes) (on_board yes) (fields_autoplaced)
-    (property "Reference" "U7" (id 0) (at 553.212 264.5953 90)
+    (property "Reference" "U?" (id 0) (at 553.212 264.5953 90)
       (effects (font (size 1.27 1.27)) (justify left))
     )
-    (property "Value" "74HCT08" (id 1) (at 553.212 267.1322 90)
+    (property "Value" "74HCT02" (id 1) (at 553.212 267.1322 90)
       (effects (font (size 1.27 1.27)) (justify left))
     )
-    (property "Footprint" "Package_DIP:DIP-14_W7.62mm_Socket_LongPads" (id 2) (at 548.64 265.43 0)
+    (property "Footprint" "" (id 2) (at 548.64 265.43 0)
       (effects (font (size 1.27 1.27)) hide)
     )
-    (property "Datasheet" "http://www.ti.com/lit/gpn/sn74LS08" (id 3) (at 548.64 265.43 0)
+    (property "Datasheet" "http://www.ti.com/lit/gpn/sn74hct02" (id 3) (at 548.64 265.43 0)
       (effects (font (size 1.27 1.27)) hide)
     )
@@
     )
     (path "/00000000-0000-0000-0000-000061a0ca4d"
-      (reference "NOR1") (unit 1) (value "74HCT04") (footprint "Package_DIP:DIP-14_W7.62mm_Socket_LongPads")
+      (reference "NOT1") (unit 1) (value "74HCT04") (footprint "Package_DIP:DIP-14_W7.62mm_Socket_LongPads")
     )
     (path "/00000000-0000-0000-0000-000061a0241a"
-      (reference "NOR1") (unit 2) (value "74HCT04") (footprint "Package_DIP:DIP-14_W7.62mm_Socket_LongPads")
+      (reference "NOT1") (unit 2) (value "74HCT04") (footprint "Package_DIP:DIP-14_W7.62mm_Socket_LongPads")
     )
     (path "/4fb7f8d4-9f5a-4a16-bef7-b6dda8fca016"
-      (reference "NOR1") (unit 7) (value "74HCT04") (footprint "Package_DIP:DIP-14_W7.62mm_Socket_LongPads")
+      (reference "NOT1") (unit 7) (value "74HCT04") (footprint "Package_DIP:DIP-14_W7.62mm_Socket_LongPads")
     )
     (path "/74c4812c-6e06-4d26-a5a5-c7b65c0620a4"
@@
       (reference "U7") (unit 1) (value "74HCT08") (footprint "Package_DIP:DIP-14_W7.62mm_Socket_LongPads")
     )
-    (path "/58f6de8c-87fc-41e9-9236-faf56ec59b02"
-      (reference "U7") (unit 2) (value "74HCT08") (footprint "Package_DIP:DIP-14_W7.62mm_Socket_LongPads")
-    )
     (path "/ef159bbf-04b6-41d8-9ab2-4cc02c43ed30"
       (reference "U7") (unit 5) (value "74HCT08") (footprint "Package_DIP:DIP-14_W7.62mm_Socket_LongPads")
@@
       (reference "U10") (unit 1) (value "74HCT138") (footprint "Package_DIP:DIP-16_W7.62mm_Socket_LongPads")
     )
+    (path "/611b0589-bb94-4bca-94da-5581b461c9a7"
+      (reference "U?") (unit 1) (value "74HCT02") (footprint "")
+    )
     (path "/00000000-0000-0000-0000-000061d2c69c"
