File: Motherboard/Motherboard.kicad_sch (KiCad schematic)
At the start: 103 parts, among them J1 ATX-20, J2 65SIB_Connector, J3 DB9_Header, J4 GPIO_Connector, J5 Expansion_Connector, J6 Expansion_Connector, J7 Expansion_Connector, J8 Expansion_Connector, J9 Expansion_Connector, SW1 SW_SPST, U1 74HCT138, U10 74HCT138, U2 AS6C4008-55PCN, U3 74HCT138, U4 74HCT138, U5 74HCT138, U6 28C010, U7 74HCT08, U8 74HCT138, U9 74HCT138, X1 ACO-8MHz

Commit message: 406 traces left to route...
Parts:
- added C3: 100 nF, Capacitor_THT:C_Disc_D3.0mm_W1.6mm_P2.50mm, symbol Device:C
- added unit 5 of U11
- J4: footprint Connector_PinSocket_2.54mm:PinSocket_2x11_P2.54mm_Vertical -> Connector_PinHeader_2.54mm:PinHeader_2x11_P2.54mm_Vertical
- U11: renamed from U?; footprint (none) -> Package_DIP:DIP-14_W7.62mm_Socket_LongPads
Connections:
- net A7: now also U4.5 (E2); no longer U4.6 (E3)
- net GND: now also C3.2, U11.7 (GND); no longer U4.5 (E2)
- net RAM1_EN: now also U2.31 (A15)
- net RAM2_EN: now also U2.2 (A16)
- net RAM3_EN: now also U2.30 (A17)
- net RAM4_EN: now also U2.1 (A18)
- net ROM1_EN: no longer U2.31 (A15)
- net ROM2_EN: no longer U2.2 (A16)
- net ROM3_EN: no longer U2.30 (A17)
- net ROM4_EN: no longer U2.1 (A18)
- net VCC: now also U4.6 (E3), C3.1, U11.14 (VCC)
- no-connect marks 80 -> 87
Changed lines of the file:
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@@
   (junction (at 173.99 154.94) (diameter 0) (color 0 0 0 0)
   )
-  (junction (at 419.1 138.43) (diameter 0) (color 0 0 0 0)
-  )
   (junction (at 257.81 53.34) (diameter 0) (color 0 0 0 0)
   )
@@
   (no_connect (at 260.35 292.1))
   (no_connect (at 299.72 134.62))
+  (no_connect (at 565.15 237.49))
+  (no_connect (at 565.15 234.95))
+  (no_connect (at 565.15 240.03))
+  (no_connect (at 565.15 224.79))
+  (no_connect (at 565.15 227.33))
+  (no_connect (at 565.15 229.87))
+  (no_connect (at 565.15 232.41))
   (no_connect (at 524.51 226.06))
   (no_connect (at 358.14 71.12))
@@
     (stroke (width 0) (type default) (color 0 0 0 0))
   )
-  (wire (pts (xy 419.1 135.89) (xy 419.1 138.43))
-    (stroke (width 0) (type default) (color 0 0 0 0))
-  )
   (wire (pts (xy 92.71 228.6) (xy 116.84 228.6))
     (stroke (width 0) (type default) (color 0 0 0 0))
@@
     )
   )
-  (global_label "ROM2_EN" (shape input) (at 177.8 87.63 180) (fields_autoplaced)
+  (global_label "RAM2_EN" (shape input) (at 177.8 87.63 180) (fields_autoplaced)
     (effects (font (size 1.27 1.27)) (justify right))
-    (property "Intersheet References" "${INTERSHEET_REFS}" (id 0) (at 0 0 0)
-      (effects (font (size 1.27 1.27)) hide)
+    (property "Intersheet References" "${INTERSHEET_REFS}" (id 0) (at 167.0091 87.5506 0)
+      (effects (font (size 1.27 1.27)) (justify right) hide)
     )
   )
@@
     )
   )
-  (global_label "ROM3_EN" (shape input) (at 177.8 90.17 180) (fields_autoplaced)
+  (global_label "RAM3_EN" (shape input) (at 177.8 90.17 180) (fields_autoplaced)
     (effects (font (size 1.27 1.27)) (justify right))
-    (property "Intersheet References" "${INTERSHEET_REFS}" (id 0) (at 0 0 0)
-      (effects (font (size 1.27 1.27)) hide)
+    (property "Intersheet References" "${INTERSHEET_REFS}" (id 0) (at 167.0091 90.0906 0)
+      (effects (font (size 1.27 1.27)) (justify right) hide)
     )
   )
@@
     )
   )
+  (global_label "GND" (shape output) (at 381 300.99 270) (fields_autoplaced)
+    (effects (font (size 1.27 1.27)) (justify right))
+    (property "Intersheet References" "${INTERSHEET_REFS}" (id 0) (at -238.76 -115.57 0)
+      (effects (font (size 1.27 1.27)) hide)
+    )
+  )
   (global_label "A8" (shape input) (at 631.19 316.23 180) (fields_autoplaced)
     (effects (font (size 1.27 1.27)) (justify right))
@@
     )
   )
+  (global_label "GND" (shape output) (at 441.96 254 270) (fields_autoplaced)
+    (effects (font (size 1.27 1.27)) (justify right))
+    (property "Intersheet References" "${INTERSHEET_REFS}" (id 0) (at -254 -162.56 0)
+      (effects (font (size 1.27 1.27)) hide)
+    )
+  )
   (global_label "PHI2" (shape input) (at 334.01 142.24 180) (fields_autoplaced)
     (effects (font (size 1.27 1.27)) (justify right))
@@
     )
   )
+  (global_label "VCC" (shape input) (at 419.1 133.35 180) (fields_autoplaced)
+    (effects (font (size 1.27 1.27)) (justify right))
+    (property "Intersheet References" "${INTERSHEET_REFS}" (id 0) (at 413.1472 133.2706 0)
+      (effects (font (size 1.27 1.27)) (justify right) hide)
+    )
+  )
   (global_label "MEM_D5" (shape output) (at 116.84 60.96 0) (fields_autoplaced)
     (effects (font (size 1.27 1.27)) (justify left))
@@
     )
   )
-  (global_label "ROM1_EN" (shape input) (at 177.8 85.09 180) (fields_autoplaced)
+  (global_label "RAM1_EN" (shape input) (at 177.8 85.09 180) (fields_autoplaced)
     (effects (font (size 1.27 1.27)) (justify right))
-    (property "Intersheet References" "${INTERSHEET_REFS}" (id 0) (at 0 0 0)
-      (effects (font (size 1.27 1.27)) hide)
+    (property "Intersheet References" "${INTERSHEET_REFS}" (id 0) (at 167.0091 85.0106 0)
+      (effects (font (size 1.27 1.27)) (justify right) hide)
     )
   )
@@
     )
   )
-  (global_label "A7" (shape input) (at 419.1 133.35 180) (fields_autoplaced)
+  (global_label "A7" (shape input) (at 419.1 135.89 180) (fields_autoplaced)
     (effects (font (size 1.27 1.27)) (justify right))
-    (property "Intersheet References" "${INTERSHEET_REFS}" (id 0) (at 414.4777 133.2706 0)
+    (property "Intersheet References" "${INTERSHEET_REFS}" (id 0) (at 414.4777 135.8106 0)
       (effects (font (size 1.27 1.27)) (justify right) hide)
     )
@@
     )
   )
+  (global_label "VCC" (shape input) (at 381 275.59 90) (fields_autoplaced)
+    (effects (font (size 1.27 1.27)) (justify left))
+    (property "Intersheet References" "${INTERSHEET_REFS}" (id 0) (at -238.76 -133.35 0)
+      (effects (font (size 1.27 1.27)) hide)
+    )
+  )
   (global_label "GND" (shape output) (at 416.56 254 270) (fields_autoplaced)
     (effects (font (size 1.27 1.27)) (justify right))
@@
     )
   )
+  (global_label "VCC" (shape input) (at 441.96 246.38 90) (fields_autoplaced)
+    (effects (font (size 1.27 1.27)) (justify left))
+    (property "Intersheet References" "${INTERSHEET_REFS}" (id 0) (at -254 -162.56 0)
+      (effects (font (size 1.27 1.27)) hide)
+    )
+  )
   (global_label "GND" (shape output) (at 247.65 312.42 270) (fields_autoplaced)
     (effects (font (size 1.27 1.27)) (justify right))
@@
     )
   )
-  (global_label "ROM4_EN" (shape input) (at 177.8 92.71 180) (fields_autoplaced)
+  (global_label "RAM4_EN" (shape input) (at 177.8 92.71 180) (fields_autoplaced)
     (effects (font (size 1.27 1.27)) (justify right))
-    (property "Intersheet References" "${INTERSHEET_REFS}" (id 0) (at 0 0 0)
-      (effects (font (size 1.27 1.27)) hide)
+    (property "Intersheet References" "${INTERSHEET_REFS}" (id 0) (at 167.0091 92.6306 0)
+      (effects (font (size 1.27 1.27)) (justify right) hide)
     )
   )
@@
     (property "Reference" "J4" (id 0) (at 121.92 246.38 0))
     (property "Value" "GPIO_Connector" (id 1) (at 121.92 248.92 0))
-    (property "Footprint" "Connector_PinSocket_2.54mm:PinSocket_2x11_P2.54mm_Vertical" (id 2) (at 120.65 264.16 0)
+    (property "Footprint" "Connector_PinHeader_2.54mm:PinHeader_2x11_P2.54mm_Vertical" (id 2) (at 120.65 264.16 0)
       (effects (font (size 1.27 1.27)) hide)
     )
@@
     (pin "9")
   )
+  (symbol (lib_id "74xx:74HCT02") (at 381 288.29 0) (unit 5)
+    (in_bom yes) (on_board yes) (fields_autoplaced)
+    (property "Reference" "U11" (id 0) (at 386.842 287.4553 0)
+      (effects (font (size 1.27 1.27)) (justify left))
+    )
+    (property "Value" "74HCT02" (id 1) (at 386.842 289.9922 0)
+      (effects (font (size 1.27 1.27)) (justify left))
+    )
+    (property "Footprint" "Package_DIP:DIP-14_W7.62mm_Socket_LongPads" (id 2) (at 381 288.29 0)
+      (effects (font (size 1.27 1.27)) hide)
+    )
+    (property "Datasheet" "http://www.ti.com/lit/gpn/sn74hct02" (id 3) (at 381 288.29 0)
+      (effects (font (size 1.27 1.27)) hide)
+    )
+    (pin "1")
+    (pin "2")
+    (pin "3")
+    (pin "4")
+    (pin "5")
+    (pin "6")
+    (pin "10")
+    (pin "8")
+    (pin "9")
+    (pin "11")
+    (pin "12")
+    (pin "13")
+    (pin "14")
+    (pin "7")
+  )
   (symbol (lib_name "Expansion_Connector_4") (lib_id "PC:Expansion_Connector") (at 637.54 313.69 0) (unit 1)
     (in_bom yes) (on_board yes)
@@
   (symbol (lib_id "74xx:74HCT02") (at 548.64 265.43 270) (unit 1)
     (in_bom yes) (on_board yes) (fields_autoplaced)
-    (property "Reference" "U?" (id 0) (at 553.212 264.5953 90)
+    (property "Reference" "U11" (id 0) (at 553.212 264.5953 90)
       (effects (font (size 1.27 1.27)) (justify left))
     )
@@
       (effects (font (size 1.27 1.27)) (justify left))
     )
-    (property "Footprint" "" (id 2) (at 548.64 265.43 0)
+    (property "Footprint" "Package_DIP:DIP-14_W7.62mm_Socket_LongPads" (id 2) (at 548.64 265.43 0)
       (effects (font (size 1.27 1.27)) hide)
     )
@@
     (pin "7")
   )
+  (symbol (lib_id "Device:C") (at 441.96 250.19 0) (unit 1)
+    (in_bom yes) (on_board yes)
+    (property "Reference" "C3" (id 0) (at 444.881 249.0216 0)
+      (effects (font (size 1.27 1.27)) (justify left))
+    )
+    (property "Value" "100 nF" (id 1) (at 444.881 251.333 0)
+      (effects (font (size 1.27 1.27)) (justify left))
+    )
+    (property "Footprint" "Capacitor_THT:C_Disc_D3.0mm_W1.6mm_P2.50mm" (id 2) (at 442.9252 254 0)
+      (effects (font (size 1.27 1.27)) hide)
+    )
+    (property "Datasheet" "~" (id 3) (at 441.96 250.19 0)
+      (effects (font (size 1.27 1.27)) hide)
+    )
+    (pin "1")
+    (pin "2")
+  )
   (sheet_instances
     (path "/" (page "1"))
@@
       (reference "C2") (unit 1) (value "100 nF") (footprint "Capacitor_THT:C_Disc_D3.0mm_W1.6mm_P2.50mm")
     )
+    (path "/f6206360-21d5-44bd-9a6b-f3c2817e3915"
+      (reference "C3") (unit 1) (value "100 nF") (footprint "Capacitor_THT:C_Disc_D3.0mm_W1.6mm_P2.50mm")
+    )
     (path "/00000000-0000-0000-0000-00006197f873"
       (reference "C5") (unit 1) (value "0.1uF") (footprint "Capacitor_THT:C_Disc_D3.0mm_W1.6mm_P2.50mm")
@@
     )
     (path "/00000000-0000-0000-0000-000061a7b6be"
-      (reference "J4") (unit 1) (value "GPIO_Connector") (footprint "Connector_PinSocket_2.54mm:PinSocket_2x11_P2.54mm_Vertical")
+      (reference "J4") (unit 1) (value "GPIO_Connector") (footprint "Connector_PinHeader_2.54mm:PinHeader_2x11_P2.54mm_Vertical")
     )
     (path "/22f31cf2-4767-4dec-b717-a3e71968aeb4"
@@
     )
     (path "/611b0589-bb94-4bca-94da-5581b461c9a7"
-      (reference "U?") (unit 1) (value "74HCT02") (footprint "")
+      (reference "U11") (unit 1) (value "74HCT02") (footprint "Package_DIP:DIP-14_W7.62mm_Socket_LongPads")
+    )
+    (path "/102c3cdb-36ec-4b35-9db1-5864af8de5cc"
+      (reference "U11") (unit 5) (value "74HCT02") (footprint "Package_DIP:DIP-14_W7.62mm_Socket_LongPads")
     )
     (path "/00000000-0000-0000-0000-000061d2c69c"
