File: Motherboard/Motherboard.kicad_sch (KiCad schematic)
At the start: 63 parts, among them J1 ATX-20, J2 65SIB_Connector, J3 DB9_Header, J4 GPIO_Connector, J5 Expansion_Connector, J6 Expansion_Connector, J7 Expansion_Connector, J8 Expansion_Connector, J9 Expansion_Connector, SW1 SW_SPST, U2 AS6C4008-55PCN, U3 ATF22V10C, U4 DS1813, U6 28C010, X1 ACO-8MHz

Commit message: Version 2.6 completed...
Parts:
- JP1, JP2: renamed from JP?; footprint (none) -> Connector_PinHeader_2.54mm:PinHeader_1x03_P2.54mm_Vertical
- R1: footprint (none) -> Resistor_THT:R_Axial_DIN0207_L6.3mm_D2.5mm_P7.62mm_Horizontal
- gave numbers to parts that had none: 1
Changed lines of the file:
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@@
   (symbol (lib_id "Jumper:Jumper_3_Bridged12") (at 259.08 246.38 90) (unit 1)
     (in_bom yes) (on_board yes) (fields_autoplaced)
-    (property "Reference" "JP?" (id 0) (at 257.4539 245.5453 90)
+    (property "Reference" "JP2" (id 0) (at 257.4539 245.5453 90)
       (effects (font (size 1.27 1.27)) (justify left))
     )
@@
       (effects (font (size 1.27 1.27)) (justify left))
     )
-    (property "Footprint" "" (id 2) (at 259.08 246.38 0)
+    (property "Footprint" "Connector_PinHeader_2.54mm:PinHeader_1x03_P2.54mm_Vertical" (id 2) (at 259.08 246.38 0)
       (effects (font (size 1.27 1.27)) hide)
     )
@@
   (symbol (lib_id "Jumper:Jumper_3_Bridged12") (at 76.2 88.9 90) (unit 1)
     (in_bom yes) (on_board yes) (fields_autoplaced)
-    (property "Reference" "JP?" (id 0) (at 74.5739 88.0653 90)
+    (property "Reference" "JP1" (id 0) (at 74.5739 88.0653 90)
       (effects (font (size 1.27 1.27)) (justify left))
     )
@@
       (effects (font (size 1.27 1.27)) (justify left))
     )
-    (property "Footprint" "" (id 2) (at 76.2 88.9 0)
+    (property "Footprint" "Connector_PinHeader_2.54mm:PinHeader_1x03_P2.54mm_Vertical" (id 2) (at 76.2 88.9 0)
       (effects (font (size 1.27 1.27)) hide)
     )
@@
       (effects (font (size 1.27 1.27)) (justify left))
     )
-    (property "Footprint" "" (id 2) (at 102.362 208.28 90)
+    (property "Footprint" "Resistor_THT:R_Axial_DIN0207_L6.3mm_D2.5mm_P7.62mm_Horizontal" (id 2) (at 102.362 208.28 90)
       (effects (font (size 1.27 1.27)) hide)
     )
@@
   (symbol (lib_id "Device:R") (at 76.2 78.74 0) (unit 1)
     (in_bom yes) (on_board yes)
-    (property "Reference" "R?" (id 0) (at 70.9422 78.74 90))
+    (property "Reference" "R2" (id 0) (at 70.9422 78.74 90))
     (property "Value" "3.3k Ω" (id 1) (at 73.2536 78.74 90))
     (property "Footprint" "Resistor_THT:R_Axial_DIN0207_L6.3mm_D2.5mm_P7.62mm_Horizontal" (id 2) (at 74.422 78.74 90)
@@
       (reference "J9") (unit 1) (value "Expansion_Connector") (footprint "PC:Expansion_Connector_Motherboard")
     )
+    (path "/add8bc41-e3d3-481e-b128-ae08b0cb09f3"
+      (reference "JP1") (unit 1) (value "Jumper_3_Bridged12") (footprint "Connector_PinHeader_2.54mm:PinHeader_1x03_P2.54mm_Vertical")
+    )
+    (path "/6f4b6105-224e-42bf-b7e2-d653e1d8735d"
+      (reference "JP2") (unit 1) (value "Jumper_3_Bridged12") (footprint "Connector_PinHeader_2.54mm:PinHeader_1x03_P2.54mm_Vertical")
+    )
     (path "/00000000-0000-0000-0000-000061a41acc"
       (reference "JP4") (unit 1) (value "CLK/1") (footprint "Connector_PinHeader_2.54mm:PinHeader_1x02_P2.54mm_Vertical")
@@
       (reference "JP6") (unit 1) (value "CLK/4") (footprint "Connector_PinHeader_2.54mm:PinHeader_1x02_P2.54mm_Vertical")
     )
-    (path "/6f4b6105-224e-42bf-b7e2-d653e1d8735d"
-      (reference "JP?") (unit 1) (value "Jumper_3_Bridged12") (footprint "")
-    )
-    (path "/add8bc41-e3d3-481e-b128-ae08b0cb09f3"
-      (reference "JP?") (unit 1) (value "Jumper_3_Bridged12") (footprint "")
-    )
     (path "/00000000-0000-0000-0000-000061a75d9b"
       (reference "NMI/IRQ1") (unit 1) (value "SW") (footprint "Connector_PinHeader_2.54mm:PinHeader_1x03_P2.54mm_Vertical")
@@
     )
     (path "/dde2964d-78c7-464b-aee8-feca4368665c"
-      (reference "R1") (unit 1) (value "3.3k") (footprint "")
+      (reference "R1") (unit 1) (value "3.3k") (footprint "Resistor_THT:R_Axial_DIN0207_L6.3mm_D2.5mm_P7.62mm_Horizontal")
+    )
+    (path "/dff96944-e331-4220-a56d-d8c923ac86a8"
+      (reference "R2") (unit 1) (value "3.3k Ω") (footprint "Resistor_THT:R_Axial_DIN0207_L6.3mm_D2.5mm_P7.62mm_Horizontal")
     )
     (path "/dcd42140-1abc-4c79-b38e-d454cf8ccfb6"
@@
       (reference "R21") (unit 1) (value "3.3k Ω") (footprint "Resistor_THT:R_Axial_DIN0207_L6.3mm_D2.5mm_P7.62mm_Horizontal")
     )
-    (path "/dff96944-e331-4220-a56d-d8c923ac86a8"
-      (reference "R?") (unit 1) (value "3.3k Ω") (footprint "Resistor_THT:R_Axial_DIN0207_L6.3mm_D2.5mm_P7.62mm_Horizontal")
-    )
     (path "/00000000-0000-0000-0000-00006196bac3"

Commit message: Completed 2.7...
Parts:
- removed SW1: SW_SPST, Button_Switch_THT:SW_DIP_SPSTx01_Slide_9.78x4.72mm_W7.62mm_P2.54mm, symbol Switch:SW_SPST
- added C1: C_Polarized, Capacitor_THT:CP_Radial_D5.0mm_P2.50mm, symbol Device:C_Polarized
- added C2: C, Capacitor_THT:C_Disc_D3.0mm_W1.6mm_P2.50mm, symbol Device:C
- added D1, D2: LED, LED_THT:LED_D5.0mm, symbol Device:LED
- added J10: USB_B_Mini, Connector_USB:USB_Mini-B_Tensility_54-00023_Vertical, symbol Connector:USB_B_Mini
- added R3, R4: 220, Resistor_THT:R_Axial_DIN0207_L6.3mm_D2.5mm_P7.62mm_Horizontal, symbol Device:R
- added SW1: SW_Push, Button_Switch_THT:SW_PUSH_6mm, symbol Switch:SW_Push
- added U1: MCP2200-I-SO, Package_SO:SOIC-20W_7.5x12.8mm_P1.27mm, symbol Interface_USB:MCP2200-I-SO
- added USB_CLK1: ACO-12MHz, Oscillator:Oscillator_DIP-14, symbol Oscillator:ACO-xxxMHz
Connections:
- net DCD_COM: no longer UART1.16 (~{DCD})
- net DSR_COM: no longer UART1.17 (~{DSR})
- net DTR_COM: no longer UART1.11 (~{DTR})
- net GND: now also C1.2, C2.2, D1.1 (K), D2.1 (K), J10.5 (GND), J10.6 (Shield), SW1.1, U1.20 (VSS), USB_CLK1.7 (GND)
- net Rx_COM: now also U1.12 (RX)
- net Tx_COM: now also U1.10 (TX)
- net VCC: now also USB_CLK1.14 (Vcc)
- net ~{RESET}: now also U1.4 (RST)
- net at J1.14 (PS_ON#): now also SW1.2
- net CTS_COM renamed ~{CTS_COM}
- net ~{CTS_COM}: now also U1.11 (RTS)
- net CTS_COM_PORT renamed ~{CTS_COM_PORT}
- net RTS_COM renamed ~{RTS_COM}
- net ~{RTS_COM}: now also U1.13 (CTS)
- net RTS_COM_PORT renamed ~{RTS_COM_PORT}
- new net: C1.1, J10.1 (VBUS), U1.1 (VDD)
- new net: R3.1, U1.6 (GP6/RxLED)
- new net: D1.2 (A), R3.2
- new net: J10.2 (D-), U1.18 (D-)
- new net: J10.3 (D+), U1.19 (D+)
- new net: C2.1, U1.17 (V_USB)
- new net: D2.2 (A), R4.2
- new net: U1.2 (OSC1), USB_CLK1.8 (OUT)
- new net: R4.1, U1.5 (GP7/TxLED)
- no-connect marks 23 -> 33
Other:
- moved on the sheet: J3, UART-RS232

Commit message: Updated motherboard...
Connections:
- net RAM_OE is gone; now on net ~{RAM_OE}: SHARED_ROM1.22 (~{OE})
- net R/~{W} is gone; now on net R\~{W}: U3.23 (I/O)
- net A4: now also U3.14 (I/O)
- net ~{CS_65SIB}: now also U3.17 (I/O); no longer U3.16 (I/O)
- net ~{CS_GPIO}: now also U3.16 (I/O); no longer U3.15 (I/O)
- net ~{CS_UART}: now also U3.15 (I/O); no longer U3.14 (I/O)
- net 5vSB: no longer names the net of J1.9 (+5VSB)
- net DCD_COM: no longer names the net of UART-RS232.17 (R4OUT)
- net DCD_COM_PORT: no longer names the net of UART-RS232.18 (R4IN)
- net DCD_COM_PORT: no longer J3.1
- net DSR_COM: no longer names the net of UART-RS232.23 (R3OUT)
- net DSR_COM_PORT: no longer names the net of UART-RS232.24 (R3IN)
- net DSR_COM_PORT: no longer J3.2 (6)
- net DTR_COM: no longer names the net of UART-RS232.15 (T3IN)
- net DTR_COM_PORT: no longer names the net of UART-RS232.2 (T3OUT)
- net DTR_COM_PORT: no longer J3.7 (4)
- no-connect marks 33 -> 42
Changed lines of the file:
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@@
   )
   (no_connect (at 549.91 123.19))
-  (no_connect (at 186.69 142.24))
-  (no_connect (at 474.98 149.86))
   (no_connect (at 709.93 154.94))
   (no_connect (at 394.97 101.6))
@@
   (no_connect (at 186.69 147.32))
   (no_connect (at 549.91 128.27))
+  (no_connect (at 610.87 69.85))
+  (no_connect (at 608.33 69.85))
+  (no_connect (at 623.57 69.85))
   (no_connect (at 764.54 322.58))
   (no_connect (at 622.3 322.58))
@@
   (no_connect (at 664.21 149.86))
   (no_connect (at 509.27 128.27))
+  (no_connect (at 549.91 118.11))
+  (no_connect (at 549.91 148.59))
+  (no_connect (at 549.91 143.51))
+  (no_connect (at 509.27 143.51))
+  (no_connect (at 509.27 148.59))
+  (no_connect (at 509.27 118.11))
+  (no_connect (at 186.69 142.24))
   (no_connect (at 549.91 158.75))
   (no_connect (at 549.91 153.67))
   (no_connect (at 90.17 140.97))
+  (no_connect (at 186.69 139.7))
   (no_connect (at 509.27 123.19))
   (no_connect (at 513.08 57.15))
@@
     )
   )
-  (global_label "DSR_COM_PORT" (shape output) (at 610.87 69.85 90) (fields_autoplaced)
-    (effects (font (size 1.27 1.27)) (justify left))
-    (property "Intersheet References" "${INTERSHEET_REFS}" (id 0) (at 93.98 -5.08 0)
-      (effects (font (size 1.27 1.27)) hide)
-    )
-  )
   (global_label "~{CS_RAM}" (shape input) (at 203.2 72.39 0) (fields_autoplaced)
     (effects (font (size 1.27 1.27)) (justify left))
@@
     )
   )
-  (global_label "RAM_OE" (shape input) (at 96.52 91.44 180) (fields_autoplaced)
+  (global_label "~{RAM_OE}" (shape input) (at 96.52 91.44 180) (fields_autoplaced)
     (effects (font (size 1.27 1.27)) (justify right))
     (property "Intersheet References" "${INTERSHEET_REFS}" (id 0) (at 86.9387 91.3606 0)
@@
     )
   )
-  (global_label "DTR_COM_PORT" (shape output) (at 549.91 118.11 0) (fields_autoplaced)
-    (effects (font (size 1.27 1.27)) (justify left))
-    (property "Intersheet References" "${INTERSHEET_REFS}" (id 0) (at -40.64 7.62 0)
-      (effects (font (size 1.27 1.27)) hide)
-    )
-  )
   (global_label "~{RESET}" (shape input) (at 664.21 124.46 180) (fields_autoplaced)
     (effects (font (size 1.27 1.27)) (justify right))
@@
     )
   )
-  (global_label "DTR_COM" (shape input) (at 509.27 118.11 180) (fields_autoplaced)
-    (effects (font (size 1.27 1.27)) (justify right))
-    (property "Intersheet References" "${INTERSHEET_REFS}" (id 0) (at -40.64 7.62 0)
-      (effects (font (size 1.27 1.27)) hide)
-    )
-  )
   (global_label "8MHz" (shape output) (at 205.74 205.74 180) (fields_autoplaced)
     (effects (font (size 1.27 1.27)) (justify right))
@@
     )
   )
-  (global_label "DCD_COM_PORT" (shape input) (at 549.91 148.59 0) (fields_autoplaced)
-    (effects (font (size 1.27 1.27)) (justify left))
-    (property "Intersheet References" "${INTERSHEET_REFS}" (id 0) (at -40.64 7.62 0)
-      (effects (font (size 1.27 1.27)) hide)
-    )
-  )
   (global_label "MEM_D5" (shape bidirectional) (at 655.32 302.26 0) (fields_autoplaced)
     (effects (font (size 1.27 1.27)) (justify left))
@@
     )
   )
-  (global_label "~{CS_RAM}" (shape input) (at 474.98 142.24 0) (fields_autoplaced)
+  (global_label "~{CS_RAM}" (shape output) (at 474.98 142.24 0) (fields_autoplaced)
     (effects (font (size 1.27 1.27)) (justify left))
     (property "Intersheet References" "${INTERSHEET_REFS}" (id 0) (at 484.5613 142.1606 0)
@@
     )
   )
-  (global_label "~{CS_UART}" (shape output) (at 474.98 157.48 0) (fields_autoplaced)
+  (global_label "~{CS_UART}" (shape output) (at 474.98 154.94 0) (fields_autoplaced)
     (effects (font (size 1.27 1.27)) (justify left))
-    (property "Intersheet References" "${INTERSHEET_REFS}" (id 0) (at 485.408 157.4006 0)
+    (property "Intersheet References" "${INTERSHEET_REFS}" (id 0) (at 485.408 154.8606 0)
       (effects (font (size 1.27 1.27)) (justify left) hide)
     )
@@
     )
   )
+  (global_label "A4" (shape input) (at 474.98 157.48 0) (fields_autoplaced)
+    (effects (font (size 1.27 1.27)) (justify left))
+    (property "Intersheet References" "${INTERSHEET_REFS}" (id 0) (at 479.6023 157.4006 0)
+      (effects (font (size 1.27 1.27)) (justify left) hide)
+    )
+  )
   (global_label "A5" (shape input) (at 713.74 307.34 180) (fields_autoplaced)
     (effects (font (size 1.27 1.27)) (justify right))
@@
     )
   )
-  (global_label "5vSB" (shape output) (at 186.69 139.7 0) (fields_autoplaced)
-    (effects (font (size 1.27 1.27)) (justify left))
-    (property "Intersheet References" "${INTERSHEET_REFS}" (id 0) (at 193.6709 139.6206 0)
-      (effects (font (size 1.27 1.27)) (justify left) hide)
-    )
-  )
   (global_label "GND" (shape output) (at 106.68 99.06 270) (fields_autoplaced)
     (effects (font (size 1.27 1.27)) (justify right))
@@
     )
   )
-  (global_label "~{CS_ROM}" (shape input) (at 474.98 144.78 0) (fields_autoplaced)
+  (global_label "~{CS_ROM}" (shape output) (at 474.98 144.78 0) (fields_autoplaced)
     (effects (font (size 1.27 1.27)) (justify left))
     (property "Intersheet References" "${INTERSHEET_REFS}" (id 0) (at 484.8032 144.7006 0)
@@
     )
   )
-  (global_label "~{CS_65SIB}" (shape output) (at 474.98 152.4 0) (fields_autoplaced)
+  (global_label "~{CS_65SIB}" (shape output) (at 474.98 149.86 0) (fields_autoplaced)
     (effects (font (size 1.27 1.27)) (justify left))
-    (property "Intersheet References" "${INTERSHEET_REFS}" (id 0) (at 486.2547 152.3206 0)
+    (property "Intersheet References" "${INTERSHEET_REFS}" (id 0) (at 486.2547 149.7806 0)
       (effects (font (size 1.27 1.27)) (justify left) hide)
     )
@@
     )
   )
-  (global_label "DTR_COM_PORT" (shape input) (at 623.57 69.85 90) (fields_autoplaced)
-    (effects (font (size 1.27 1.27)) (justify left))
-    (property "Intersheet References" "${INTERSHEET_REFS}" (id 0) (at 93.98 -5.08 0)
-      (effects (font (size 1.27 1.27)) hide)
-    )
-  )
   (global_label "4MHz" (shape input) (at 193.04 226.06 180) (fields_autoplaced)
     (effects (font (size 1.27 1.27)) (justify right))
@@
     )
   )
-  (global_label "R{slash}~{W}" (shape input) (at 474.98 134.62 0) (fields_autoplaced)
+  (global_label "R\\~{W}" (shape input) (at 474.98 134.62 0) (fields_autoplaced)
     (effects (font (size 1.27 1.27)) (justify left))
-    (property "Intersheet References" "${INTERSHEET_REFS}" (id 0) (at 481.3561 134.5406 0)
+    (property "Intersheet References" "${INTERSHEET_REFS}" (id 0) (at 480.8723 134.5406 0)
       (effects (font (size 1.27 1.27)) (justify left) hide)
     )
@@
     )
   )
-  (global_label "DCD_COM" (shape output) (at 509.27 148.59 180) (fields_autoplaced)
-    (effects (font (size 1.27 1.27)) (justify right))
-    (property "Intersheet References" "${INTERSHEET_REFS}" (id 0) (at -40.64 7.62 0)
-      (effects (font (size 1.27 1.27)) hide)
-    )
-  )
   (global_label "CPU_D7" (shape bidirectional) (at 123.19 166.37 0) (fields_autoplaced)
     (effects (font (size 1.27 1.27)) (justify left))
@@
     )
   )
-  (global_label "DSR_COM_PORT" (shape input) (at 549.91 143.51 0) (fields_autoplaced)
+  (global_label "~{CS_GPIO}" (shape output) (at 474.98 152.4 0) (fields_autoplaced)
     (effects (font (size 1.27 1.27)) (justify left))
-    (property "Intersheet References" "${INTERSHEET_REFS}" (id 0) (at -40.64 7.62 0)
-      (effects (font (size 1.27 1.27)) hide)
-    )
-  )
-  (global_label "~{CS_GPIO}" (shape output) (at 474.98 154.94 0) (fields_autoplaced)
-    (effects (font (size 1.27 1.27)) (justify left))
-    (property "Intersheet References" "${INTERSHEET_REFS}" (id 0) (at 485.2266 154.8606 0)
+    (property "Intersheet References" "${INTERSHEET_REFS}" (id 0) (at 485.2266 152.3206 0)
       (effects (font (size 1.27 1.27)) (justify left) hide)
     )
@@
     )
   )
-  (global_label "DCD_COM_PORT" (shape output) (at 608.33 69.85 90) (fields_autoplaced)
-    (effects (font (size 1.27 1.27)) (justify left))
-    (property "Intersheet References" "${INTERSHEET_REFS}" (id 0) (at 93.98 -5.08 0)
-      (effects (font (size 1.27 1.27)) hide)
-    )
-  )
   (global_label "~{65SIB_IRQ}" (shape input) (at 394.97 104.14 180) (fields_autoplaced)
     (effects (font (size 1.27 1.27)) (justify right))
@@
       (effects (font (size 1.27 1.27)) hide)
     )
-  )
-  (global_label "DSR_COM" (shape output) (at 509.27 143.51 180) (fields_autoplaced)
-    (effects (font (size 1.27 1.27)) (justify right))
-    (property "Intersheet References" "${INTERSHEET_REFS}" (id 0) (at -40.64 7.62 0)
-      (effects (font (size 1.27 1.27)) hide)
-    )
