File: Debug/Debug.sch (KiCad schematic (older format))
At the start: 53 parts, among them SW1 Step, SW2 PHI1/Step, SW3 Run, SW4 SI/SC, U1 74LS04, U10 MC14495P1, U11 HDSP-7803, U12 MC14495P1, U13 HDSP-7803, U14 MC14495P1, U15 HDSP-7803, U2 74LS74, U3 MC14495P1, U4 HDSP-7803, U5 74LS374, U6 MC14495P1, U7 HDSP-7803, U8 MC14495P1, U9 HDSP-7803

Commit message: Debug card added...
Parts:
- added J?: Expansion_Connector, symbol PC:Expansion_Connector
Connections:
- net RW renamed R~W
Changed lines of the file:
@@
 Sync
 Text GLabel 2700 5400 0    50   Input ~ 0
-RW
+R~W
 Text GLabel 2700 5500 0    50   Input ~ 0
 Reset
@@
 Text GLabel 2700 7950 0    50   Input ~ 0
 IRQ7
+$Comp
+L PC:Expansion_Connector J?
+U 1 1 627369F2
+P 6400 5850
+F 0 "J?" H 6450 7067 50  0000 C CNN
+F 1 "Expansion_Connector" H 6450 6976 50  0000 C CNN
+F 2 "" H 6400 5850 50  0001 C CNN
+F 3 "~" H 6400 5850 50  0001 C CNN
+	1    6400 5850
+	1    0    0    -1
+$EndComp
 $EndSCHEMATC
