File: Debug/Debug.kicad_pcb (KiCad board)
At the start: 4 copper layers, 127 x 88.9 mm, 38 parts, among them J1 Expansion_Connector, SW1 Step, SW2 PHI1/Step, SW3 Run, SW4 SI/SC, U1 74HCT04, U10 MC14495P1, U11 HDSP-7803, U12 MC14495P1, U13 HDSP-7803, U14 MC14495P1, U15 HDSP-7803, U2 74HCT74, U3 MC14495P1, U4 HDSP-7803, U5 74HCT374, U6 MC14495P1, U7 HDSP-7803, U8 MC14495P1, U9 HDSP-7803

Commit message: Update to latest KiCad version and other edits.
Updated the files formatting to conform to KiCad 10 standards, updated dates and corrected company name, also first signed commit to this repository.
Parts:
- renumbered R2 to R1, R3 to R2, R4 to R3, R5 to R4, R6 to R5, R7 to R6, R8 to R7, R9 to R8, R1 to R9, SW4 to SW2, SW2 to SW4, U3 to U1, U4 to U2, U5 to U3, U6 to U4, U7 to U5, U1 to U6, U8 to U7, U9 to U8, U2 to U9
Connections:
- SW2 pad 1: unconnected-(SW4-Pad1) -> +5V
- SW3 pad 1: unconnected-(SW3-Pad1) -> +5V
- U9 pad 2: unconnected-(U2-Pad2) -> GND
