File: Sound/Sound.sch (KiCad schematic (older format))
At the start: 9 parts, among them U10 74HCT04, U15 74HCT04, U18 74LS08, U2 74HCT04, U21 74HCT04, U22 74LS21, U27 74HCT04

Commit message: 2.3 has arrived...
2.3! 2.3!! 2.3!!!
Parts:
- added J1: Expansion_Connector, PC:Expansion_Connector_Board, symbol PC:Expansion_Connector
- added U1: 74HCT74, Package_DIP:DIP-14_W7.62mm_Socket_LongPads, symbol 74xx:74LS74
- added U? (x3): LM386, symbol Amplifier_Audio:LM386
- U2: renamed from U18; value 74LS08 -> 74HCT08
- U3: renamed from U22; value 74LS21 -> 74HCT21
- renumbered U27 to U4, U21 to U4, U15 to U4, U10 to U4, U2 to U4, SaMM_CTRL1 to YamahaSound1
Connections:
- net 2MHz: now also U1.9 (Q)
- net A0: now also J1.5 (Pin_5)
- net A1: now also J1.7 (Pin_7)
- net A10: now also J1.25 (Pin_25)
- net A11: now also J1.27 (Pin_27)
- net A2: now also J1.9 (Pin_9)
- net A3: now also J1.11 (Pin_11)
- net A4: now also J1.13 (Pin_13)
- net A5: now also J1.15 (Pin_15)
- net A6: now also J1.17 (Pin_17)
- net A7: now also J1.19 (Pin_19)
- net A8: now also J1.21 (Pin_21)
- net A9: now also J1.23 (Pin_23)
- net GND: now also J1.3 (Pin_3), U?.2 (-), U?.2 (-), U?.2 (-), U?.4 (GND), U?.4 (GND), U?.4 (GND)
- net PHI2: now also J1.24 (Pin_24)
- net R\~W: now also J1.37 (Pin_37)
- net VCC: now also J1.1, U1.1 (~R), U1.10 (~S), U1.13 (~R), U1.4 (~S), U?.6 (V+), U?.6 (V+), U?.6 (V+)
- net ~CS_DEV: now also J1.28 (Pin_28)
- net ~RESET: now also J1.18 (Pin_18)
- net CLK_SND: no longer names the net of YamahaSound1.17 (PB7)
- net IRQ3 renamed ~IRQ3
- net ~IRQ3: now also J1.30 (Pin_30)
- net MEM_D0 renamed D0
- net D0: now also J1.2 (Pin_2)
- net MEM_D1 renamed D1
- net D1: now also J1.4 (Pin_4)
- net MEM_D2 renamed D2
- net D2: now also J1.6 (Pin_6)
- net MEM_D3 renamed D3
- net D3: now also J1.8 (Pin_8)
- net MEM_D4 renamed D4
- net D4: now also J1.10 (Pin_10)
- net MEM_D5 renamed D5
- net D5: now also J1.12 (Pin_12)
- net MEM_D6 renamed D6
- net D6: now also J1.14 (Pin_14)
- net MEM_D7 renamed D7
- net D7: now also J1.16 (Pin_16)
- net RAM1_EN: no longer names the net of YamahaSound1.40 (CA1)
- net RAM2_EN: no longer names the net of YamahaSound1.39 (CA2)
- net RAM3_EN: no longer names the net of YamahaSound1.18 (CB1)
- net RAM4_EN: no longer names the net of YamahaSound1.19 (CB2)
- net ROM1_EN: no longer names the net of YamahaSound1.13 (PB3)
- net ROM2_EN: no longer names the net of YamahaSound1.14 (PB4)
- net ROM3_EN: no longer names the net of YamahaSound1.15 (PB5)
- net ROM4_EN: no longer names the net of YamahaSound1.16 (PB6)
- new net: U1.11 (C), U1.2 (D), U1.6 (~Q)
- new net: U1.12 (D), U1.8 (~Q)
- new net 8MHz: J1.26 (Pin_26), U1.3 (C)
- no-connect marks 0 -> 24
Other:
- moved on the sheet: SOUND_GEN1, U2C, U3A, U3B, U4A, U4B, U4C, U4D, U4E, U4F, YamahaSound1

Commit message: Bug fixes...
Parts:
- added C1, C3, C5: CP, symbol Device:CP
- added C2, C4, C6: C, symbol Device:C
- added J2: LINE OUT, Connector_Audio:Jack_3.5mm_CUI_SJ1-3533NG_Horizontal, symbol Connector:AudioJack3_Ground
- added J3: SUB OUT, Connector_Audio:Jack_3.5mm_CUI_SJ1-3533NG_Horizontal, symbol Connector:AudioJack2_Ground
- added RV1: R_POT_Dual_Separate, Potentiometer_THT:Potentiometer_Piher_T-16H_Double_Horizontal, symbol Device:R_POT_Dual_Separate
- added RV3: R_POT, Potentiometer_THT:Potentiometer_Piher_T-16H_Single_Horizontal, symbol Device:R_POT
- U5, U6, U7: renamed from U?; footprint (none) -> Package_DIP:DIP-8_W7.62mm_Socket_LongPads
Connections:
- net GND: now also C2.2, C4.2, C6.2, J2.G, J2.S, J3.G, J3.S, RV1.3, RV1.6, RV3.3
- net at U6.3 (+): now also RV1.5
- net at U6.5: now also C3.1, C4.1
- net at U7.3 (+): now also RV3.2
- net at U7.5: now also C5.1, C6.1
- net at U5.3 (+): now also RV1.2
- net at U5.5: now also C1.1, C2.1
- net OUT_A: no longer names the net of SOUND_GEN1.17 (A)
- net OUT_A: now also RV1.1
- net OUT_B: no longer names the net of SOUND_GEN1.15 (B)
- net OUT_B: now also RV1.4
- net OUT_C: no longer names the net of SOUND_GEN1.18 (C)
- net OUT_C: now also RV3.1
- new net SND_L: C3.2, J2.T
- new net SND_R: C1.2, J2.R
- new net SND_SUB: C5.2, J3.T
- no-connect marks 24 -> 33
Other:
- note added: "Sound controller\nIRQ3\nAddress space: 0xD120 - 0xD12F"
- note removed: "Sound and Memory Mapping controller (SaMM)\nIRQ3\nAddress space: 0xD120 - 0xD12F"

Commit message: Updated documentation location...
Parts:
- C1, C3, C5: footprint (none) -> Capacitor_THT:CP_Radial_D5.0mm_P2.50mm
- C2, C4, C6: footprint (none) -> Capacitor_THT:C_Disc_D3.0mm_W2.0mm_P2.50mm
- renumbered YamahaSound1 to SOUND_CTRL1
Connections:
- net ~IRQ3: no longer names the net of J1.30 (Pin_30)
- net ~IRQ3: no longer SOUND_CTRL1.21 (~IRQ)
- no-connect marks 33 -> 35
Changed lines of the file:
@@
 DA7
 $Comp
-L 65xx:WD65C22 YamahaSound1
+L 65xx:WD65C22 SOUND_CTRL1
 U 1 1 65829668
 P 5050 5750
-F 0 "YamahaSound1" H 5050 4513 60  0000 C CNN
+F 0 "SOUND_CTRL1" H 5050 4513 60  0000 C CNN
 F 1 "WD65C22" H 5050 4619 60  0000 C CNN
 F 2 "Socket:DIP_Socket-40_W11.9_W12.7_W15.24_W17.78_W18.5_3M_240-1280-00-0602J" H 4550 5950 60  0001 C CNN
@@
 Wire Wire Line
 	4000 4950 4400 4950
-Text GLabel 4200 4750 0    50   Output ~ 0
-~IRQ3
-Wire Wire Line
-	4400 4750 4200 4750
 Wire Wire Line
 	2550 5150 2550 5300
@@
 Text Notes 1150 1300 0    50   ~ 0
 Sound controller\nIRQ3\nAddress space: 0xD120 - 0xD12F
-$Comp
-L PC:Expansion_Connector J1
-U 1 1 62713709
-P 2000 3150
-F 0 "J1" H 2050 4367 50  0000 C CNN
-F 1 "Expansion_Connector" H 2050 4276 50  0000 C CNN
-F 2 "PC:Expansion_Connector_Board" H 2000 3150 50  0001 C CNN
-F 3 "~" H 2000 3150 50  0001 C CNN
-	1    2000 3150
-	1    0    0    -1
-$EndComp
 Text GLabel 1800 2150 0    50   Output ~ 0
 VCC
@@
 NoConn ~ 2300 3050
 NoConn ~ 2300 3150
-Text GLabel 2300 3550 2    50   Input ~ 0
-~IRQ3
-NoConn ~ 2300 3650
-NoConn ~ 2300 3750
-NoConn ~ 2300 3850
-NoConn ~ 2300 3950
 NoConn ~ 2300 4050
 NoConn ~ 2300 4150
@@
 F 0 "C4" H 9465 3846 50  0000 L CNN
 F 1 "C" H 9465 3755 50  0000 L CNN
-F 2 "" H 9388 3650 50  0001 C CNN
+F 2 "Capacitor_THT:C_Disc_D3.0mm_W2.0mm_P2.50mm" H 9388 3650 50  0001 C CNN
 F 3 "~" H 9350 3800 50  0001 C CNN
 	1    9350 3800
@@
 F 0 "C2" H 9465 2446 50  0000 L CNN
 F 1 "C" H 9465 2355 50  0000 L CNN
-F 2 "" H 9388 2250 50  0001 C CNN
+F 2 "Capacitor_THT:C_Disc_D3.0mm_W2.0mm_P2.50mm" H 9388 2250 50  0001 C CNN
 F 3 "~" H 9350 2400 50  0001 C CNN
 	1    9350 2400
@@
 F 0 "C6" H 9465 5146 50  0000 L CNN
 F 1 "C" H 9465 5055 50  0000 L CNN
-F 2 "" H 9388 4950 50  0001 C CNN
+F 2 "Capacitor_THT:C_Disc_D3.0mm_W2.0mm_P2.50mm" H 9388 4950 50  0001 C CNN
 F 3 "~" H 9350 5100 50  0001 C CNN
 	1    9350 5100
@@
 F 0 "C1" V 9955 2100 50  0000 C CNN
 F 1 "CP" V 9864 2100 50  0000 C CNN
-F 2 "" H 9738 1950 50  0001 C CNN
+F 2 "Capacitor_THT:CP_Radial_D5.0mm_P2.50mm" H 9738 1950 50  0001 C CNN
 F 3 "~" H 9700 2100 50  0001 C CNN
 	1    9700 2100
@@
 F 0 "C3" V 9955 3500 50  0000 C CNN
 F 1 "CP" V 9864 3500 50  0000 C CNN
-F 2 "" H 9738 3350 50  0001 C CNN
+F 2 "Capacitor_THT:CP_Radial_D5.0mm_P2.50mm" H 9738 3350 50  0001 C CNN
 F 3 "~" H 9700 3500 50  0001 C CNN
 	1    9700 3500
@@
 F 0 "C5" V 9955 4800 50  0000 C CNN
 F 1 "CP" V 9864 4800 50  0000 C CNN
-F 2 "" H 9738 4650 50  0001 C CNN
+F 2 "Capacitor_THT:CP_Radial_D5.0mm_P2.50mm" H 9738 4650 50  0001 C CNN
 F 3 "~" H 9700 4800 50  0001 C CNN
 	1    9700 4800
@@
 Text GLabel 7050 5850 2    50   Output ~ 0
 SND_SUB
+$Comp
+L PC:Expansion_Connector J1
+U 1 1 62713709
+P 2000 3150
+F 0 "J1" H 2050 4367 50  0000 C CNN
+F 1 "Expansion_Connector" H 2050 4276 50  0000 C CNN
+F 2 "PC:Expansion_Connector_Board" H 2000 3150 50  0001 C CNN
+F 3 "~" H 2000 3150 50  0001 C CNN
+	1    2000 3150
+	1    0    0    -1
+$EndComp
+NoConn ~ 4400 4750
+NoConn ~ 2300 3550
+NoConn ~ 2300 3650
+NoConn ~ 2300 3750
+NoConn ~ 2300 3850
+NoConn ~ 2300 3950
 $EndSCHEMATC

Commit message: Renamed some components...
Parts:
- added unit 3 of U1
- added unit 5 of U2
- added unit 3 of U3
- added unit 7 of U4
- J2: symbol Connector:AudioJack3_Ground -> Connector:AudioJack3
- J3: symbol Connector:AudioJack2_Ground -> Connector:AudioJack2
- LINE_OUT_VOLUME1: renamed from RV1; value R_POT_Dual_Separate -> LINE OUT VOLUME
- renumbered RV3 to SUB_VOLUME1
Connections:
- net GND: now also U1.7 (GND), U2.7 (GND), U3.7 (GND), U4.7 (GND); no longer J2.G, J3.G
- net VCC: now also U1.14 (VCC), U2.14 (VCC), U3.14 (VCC), U4.14 (VCC)
Other:
- moved on the sheet: U1A, U1B
Changed lines of the file:
@@
 L 74xx:74LS74 U1
 U 1 1 6271DA31
-P 3750 2700
-F 0 "U1" H 3750 3181 50  0000 C CNN
-F 1 "74HCT74" H 3750 3090 50  0000 C CNN
-F 2 "Package_DIP:DIP-14_W7.62mm_Socket_LongPads" H 3750 2700 50  0001 C CNN
-F 3 "74xx/74hc_hct74.pdf" H 3750 2700 50  0001 C CNN
-	1    3750 2700
+P 3700 3750
+F 0 "U1" H 3700 4231 50  0000 C CNN
+F 1 "74HCT74" H 3700 4140 50  0000 C CNN
+F 2 "Package_DIP:DIP-14_W7.62mm_Socket_LongPads" H 3700 3750 50  0001 C CNN
+F 3 "74xx/74hc_hct74.pdf" H 3700 3750 50  0001 C CNN
+	1    3700 3750
 	1    0    0    -1
 $EndComp
@@
 L 74xx:74LS74 U1
 U 2 1 6271E60A
-P 4750 2750
-F 0 "U1" H 4750 3231 50  0000 C CNN
-F 1 "74HCT74" H 4750 3140 50  0000 C CNN
-F 2 "Package_DIP:DIP-14_W7.62mm_Socket_LongPads" H 4750 2750 50  0001 C CNN
-F 3 "74xx/74hc_hct74.pdf" H 4750 2750 50  0001 C CNN
-	2    4750 2750
-	1    0    0    -1
-$EndComp
-NoConn ~ 4050 2600
-Text GLabel 3450 2700 0    50   Input ~ 0
+P 4700 3800
+F 0 "U1" H 4700 4281 50  0000 C CNN
+F 1 "74HCT74" H 4700 4190 50  0000 C CNN
+F 2 "Package_DIP:DIP-14_W7.62mm_Socket_LongPads" H 4700 3800 50  0001 C CNN
+F 3 "74xx/74hc_hct74.pdf" H 4700 3800 50  0001 C CNN
+	2    4700 3800
+	1    0    0    -1
+$EndComp
+NoConn ~ 4000 3650
+Text GLabel 3400 3750 0    50   Input ~ 0
 8MHz
 Wire Wire Line
-	4200 2800 4200 3100
-Wire Wire Line
-	3100 3100 3100 2600
-Wire Wire Line
-	3100 2600 3450 2600
-Wire Wire Line
-	4200 2750 4200 2800
-Wire Wire Line
-	3750 3000 3750 3050
-Wire Wire Line
-	5050 2850 5050 3100
-Wire Wire Line
-	5050 3100 4400 3100
-Wire Wire Line
-	4400 3100 4400 2650
-Wire Wire Line
-	4400 2650 4450 2650
-Wire Wire Line
-	3750 2400 3750 2150
-Wire Wire Line
-	3750 2150 4250 2150
-Wire Wire Line
-	4750 2150 4750 2450
-Wire Wire Line
-	4250 2150 4250 2050
-Connection ~ 4250 2150
-Wire Wire Line
-	4250 2150 4300 2150
-Wire Wire Line
-	3750 3050 4300 3050
-Wire Wire Line
-	4300 3050 4300 2150
-Connection ~ 4300 2150
-Connection ~ 4300 3050
-Wire Wire Line
-	4300 3050 4750 3050
-Wire Wire Line
-	4300 2150 4750 2150
-Wire Wire Line
-	4200 2750 4450 2750
-Connection ~ 4200 2800
-Wire Wire Line
-	4050 2800 4200 2800
-Wire Wire Line
-	3100 3100 4200 3100
-Text GLabel 4250 2050 1    50   Input ~ 0
-VCC
-Text GLabel 5050 2650 2    50   Output ~ 0
+	4150 3850 4150 4150
+Wire Wire Line
+	3050 4150 3050 3650
+Wire Wire Line
+	3050 3650 3400 3650
+Wire Wire Line
+	4150 3800 4150 3850
+Wire Wire Line
+	3700 4050 3700 4100
+Wire Wire Line
+	5000 3900 5000 4150
+Wire Wire Line
+	5000 4150 4350 4150
+Wire Wire Line
+	4350 4150 4350 3700
+Wire Wire Line
+	4350 3700 4400 3700
+Wire Wire Line
+	3700 3450 3700 3200
+Wire Wire Line
+	3700 3200 4200 3200
+Wire Wire Line
+	4700 3200 4700 3500
+Wire Wire Line
+	4200 3200 4200 3100
+Connection ~ 4200 3200
+Wire Wire Line
+	4200 3200 4250 3200
+Wire Wire Line
+	3700 4100 4250 4100
+Wire Wire Line
+	4250 4100 4250 3200
+Connection ~ 4250 3200
+Connection ~ 4250 4100
+Wire Wire Line
+	4250 4100 4700 4100
+Wire Wire Line
+	4250 3200 4700 3200
+Wire Wire Line
+	4150 3800 4400 3800
+Connection ~ 4150 3850
+Wire Wire Line
+	4000 3850 4150 3850
+Wire Wire Line
+	3050 4150 4150 4150
+Text GLabel 4200 3100 1    50   Input ~ 0
+VCC
+Text GLabel 5000 3700 2    50   Output ~ 0
 2MHz
 NoConn ~ 5700 5050
@@
 	8050 1450 8050 1850
 $Comp
-L Device:R_POT RV3
+L Device:R_POT SUB_VOLUME1
 U 1 1 6271DAF0
 P 8050 4700
-F 0 "RV3" H 7981 4746 50  0000 R CNN
+F 0 "SUB_VOLUME1" H 7981 4746 50  0000 R CNN
 F 1 "R_POT" H 7981 4655 50  0000 R CNN
 F 2 "Potentiometer_THT:Potentiometer_Piher_T-16H_Single_Horizontal" H 8050 4700 50  0001 C CNN
@@
 NoConn ~ 8900 4500
 $Comp
-L Device:R_POT_Dual_Separate RV1
+L Device:R_POT_Dual_Separate LINE_OUT_VOLUME1
 U 1 1 62732FE3
 P 8050 2000
-F 0 "RV1" H 7980 2046 50  0000 R CNN
-F 1 "R_POT_Dual_Separate" H 7980 1955 50  0000 R CNN
+F 0 "LINE_OUT_VOLUME1" H 7980 2046 50  0000 R CNN
+F 1 "LINE OUT VOLUME" H 7980 1955 50  0000 R CNN
 F 2 "Potentiometer_THT:Potentiometer_Piher_T-16H_Double_Horizontal" H 8050 2000 50  0001 C CNN
 F 3 "~" H 8050 2000 50  0001 C CNN
@@
 $EndComp
 $Comp
-L Device:R_POT_Dual_Separate RV1
+L Device:R_POT_Dual_Separate LINE_OUT_VOLUME1
 U 2 1 62733622
 P 7950 3400
-F 0 "RV1" H 7880 3446 50  0000 R CNN
-F 1 "R_POT_Dual_Separate" H 7880 3355 50  0000 R CNN
+F 0 "LINE_OUT_VOLUME1" H 7880 3446 50  0000 R CNN
+F 1 "LINE OUT VOLUME" H 7880 3355 50  0000 R CNN
 F 2 "Potentiometer_THT:Potentiometer_Piher_T-16H_Double_Horizontal" H 7950 3400 50  0001 C CNN
 F 3 "~" H 7950 3400 50  0001 C CNN
@@
 SND_SUB
 $Comp
-L Connector:AudioJack3_Ground J2
+L Connector:AudioJack3 J2
 U 1 1 62762067
 P 6900 4900
@@
 	1    0    0    -1
 $EndComp
-Text GLabel 6900 5200 3    50   Output ~ 0
-GND
 Text GLabel 7100 5000 2    50   Input ~ 0
 SND_L
@@
 GND
 $Comp
-L Connector:AudioJack2_Ground J3
+L Connector:AudioJack2 J3
 U 1 1 62765D72
 P 6850 5850
@@
 	1    0    0    -1
 $EndComp
-Text GLabel 6850 6050 3    50   Output ~ 0
-GND
 Text GLabel 7050 5750 2    50   Output ~ 0
 GND
@@
 NoConn ~ 2300 3850
 NoConn ~ 2300 3950
+$Comp
+L 74xx:74HCT04 U4
+U 7 1 6273984F
+P 2850 1700
+F 0 "U4" H 3080 1746 50  0000 L CNN
+F 1 "74HCT04" H 3080 1655 50  0000 L CNN
+F 2 "Package_DIP:DIP-14_W7.62mm_Socket_LongPads" H 2850 1700 50  0001 C CNN
+F 3 "https://assets.nexperia.com/documents/data-sheet/74HC_HCT04.pdf" H 2850 1700 50  0001 C CNN
+	7    2850 1700
+	1    0    0    -1
+$EndComp
+$Comp
+L 74xx:74LS21 U3
+U 3 1 6273C74D
+P 3650 1700
+F 0 "U3" H 3880 1746 50  0000 L CNN
+F 1 "74HCT21" H 3880 1655 50  0000 L CNN
+F 2 "Package_DIP:DIP-14_W7.62mm_Socket_LongPads" H 3650 1700 50  0001 C CNN
+F 3 "http://www.ti.com/lit/gpn/sn74LS21" H 3650 1700 50  0001 C CNN
+	3    3650 1700
+	1    0    0    -1
+$EndComp
+$Comp
+L 74xx:74LS08 U2
+U 5 1 6273E4DC
+P 4400 1700
+F 0 "U2" H 4630 1746 50  0000 L CNN
+F 1 "74HCT08" H 4630 1655 50  0000 L CNN
+F 2 "Package_DIP:DIP-14_W7.62mm_Socket_LongPads" H 4400 1700 50  0001 C CNN
+F 3 "http://www.ti.com/lit/gpn/sn74LS08" H 4400 1700 50  0001 C CNN
+	5    4400 1700
+	1    0    0    -1
+$EndComp
+$Comp
+L 74xx:74LS74 U1
+U 3 1 62740A05
+P 5150 1700
+F 0 "U1" H 5380 1746 50  0000 L CNN
+F 1 "74HCT74" H 5380 1655 50  0000 L CNN
+F 2 "Package_DIP:DIP-14_W7.62mm_Socket_LongPads" H 5150 1700 50  0001 C CNN
+F 3 "74xx/74hc_hct74.pdf" H 5150 1700 50  0001 C CNN
+	3    5150 1700
+	1    0    0    -1
+$EndComp
+Text GLabel 2850 1200 1    50   Input ~ 0
+VCC
+Text GLabel 3650 1200 1    50   Input ~ 0
+VCC
+Text GLabel 4400 1200 1    50   Input ~ 0
+VCC
+Text GLabel 5150 1300 1    50   Input ~ 0
+VCC
+Text GLabel 2850 2200 3    50   Output ~ 0
+GND
+Text GLabel 3650 2200 3    50   Output ~ 0
+GND
+Text GLabel 4400 2200 3    50   Output ~ 0
+GND
+Text GLabel 5150 2100 3    50   Output ~ 0
+GND
 $EndSCHEMATC
