File: Sound/Sound.sch (KiCad schematic (older format))
At the start: 20 parts, among them J1 Expansion_Connector, J2 LINE OUT, J3 SUB OUT, U1 74HCT74, U2 74HCT08, U3 74HCT21, U4 74HCT04, U5 LM386, U6 LM386, U7 LM386

Commit message: Sound card schematic completed...
Parts:
- added C10, C8: 10 µF, Capacitor_THT:CP_Radial_D5.0mm_P2.50mm, symbol Device:CP
- added C11, C7, C9: 0.1 µF, Capacitor_THT:C_Disc_D3.0mm_W2.0mm_P2.50mm, symbol Device:C
- added C12: 0.033 µF, Capacitor_THT:C_Disc_D3.0mm_W2.0mm_P2.50mm, symbol Device:C
- added R1, R2, R3, R5: 10 Ω, Resistor_THT:R_Axial_DIN0204_L3.6mm_D1.6mm_P5.08mm_Horizontal, symbol Device:R
- added R4: ? Ω, Resistor_THT:R_Axial_DIN0204_L3.6mm_D1.6mm_P5.08mm_Horizontal, symbol Device:R
- C1, C3, C5: value CP -> 250 µF
- C2, C4, C6: value C -> 0.05 µF
- LINE_OUT_VOLUME1: value LINE OUT VOLUME -> 10k Ω
- SUB_VOLUME1: value R_POT -> 10k Ω
Connections:
- net GND: now also C11.1, C7.1, C9.1, R1.2, R2.2, R3.2, R4.2; no longer C2.2, C4.2, C6.2
- net at U6.1 (GAIN): now also C10.1
- net at U6.7 (BYPASS): now also C9.2
- net at U6.8 (GAIN): now also C10.2
- net at U7.1 (GAIN): now also R5.2
- net at C5.1, C6.1, U7.5: now also C12.2
- net at U7.7 (BYPASS): now also C11.2
- net at U5.1 (GAIN): now also C8.1
- net at U5.7 (BYPASS): now also C7.2
- net at U5.8 (GAIN): now also C8.2
- new net: C2.2, R1.1
- new net: C4.2, R2.1
- new net: C6.2, R3.1
- new net: C12.1, R5.1
- no-connect marks 35 -> 27
Other:
- moved on the sheet: C5, C6
Changed lines of the file:
@@
-	1    0    0    -1
-$EndComp
-$Comp
-L Amplifier_Audio:LM386 U5
-U 1 1 6273E396
-P 8900 2100
-F 0 "U5" H 9244 2146 50  0000 L CNN
-F 1 "LM386" H 9244 2055 50  0000 L CNN
-F 2 "Package_DIP:DIP-8_W7.62mm_Socket_LongPads" H 9000 2200 50  0001 C CNN
-F 3 "http://www.ti.com/lit/ds/symlink/lm386.pdf" H 9100 2300 50  0001 C CNN
-	1    8900 2100
 	1    0    0    -1
 $EndComp
@@
 P 8050 4700
 F 0 "SUB_VOLUME1" H 7981 4746 50  0000 R CNN
-F 1 "R_POT" H 7981 4655 50  0000 R CNN
+F 1 "10k Ω" H 7981 4655 50  0000 R CNN
 F 2 "Potentiometer_THT:Potentiometer_Piher_T-16H_Single_Horizontal" H 8050 4700 50  0001 C CNN
 F 3 "~" H 8050 4700 50  0001 C CNN
@@
 Wire Wire Line
 	8050 4050 8050 4550
-NoConn ~ 8900 1800
-NoConn ~ 8900 3200
-NoConn ~ 8900 4500
 $Comp
 L Device:R_POT_Dual_Separate LINE_OUT_VOLUME1
@@
 P 8050 2000
 F 0 "LINE_OUT_VOLUME1" H 7980 2046 50  0000 R CNN
-F 1 "LINE OUT VOLUME" H 7980 1955 50  0000 R CNN
+F 1 "10k Ω" H 7980 1955 50  0000 R CNN
 F 2 "Potentiometer_THT:Potentiometer_Piher_T-16H_Double_Horizontal" H 8050 2000 50  0001 C CNN
 F 3 "~" H 8050 2000 50  0001 C CNN
@@
 P 7950 3400
 F 0 "LINE_OUT_VOLUME1" H 7880 3446 50  0000 R CNN
-F 1 "LINE OUT VOLUME" H 7880 3355 50  0000 R CNN
+F 1 "10k Ω" H 7880 3355 50  0000 R CNN
 F 2 "Potentiometer_THT:Potentiometer_Piher_T-16H_Double_Horizontal" H 7950 3400 50  0001 C CNN
 F 3 "~" H 7950 3400 50  0001 C CNN
@@
 	9200 3500 9350 3500
 Wire Wire Line
-	9550 4800 9350 4800
-NoConn ~ 8900 2400
-NoConn ~ 9000 2400
-NoConn ~ 8900 3800
-NoConn ~ 9000 3800
-NoConn ~ 8900 5100
-NoConn ~ 9000 5100
+	9850 4800 9650 4800
 $Comp
 L Device:C C4
@@
 P 9350 3800
 F 0 "C4" H 9465 3846 50  0000 L CNN
-F 1 "C" H 9465 3755 50  0000 L CNN
+F 1 "0.05 µF" H 9465 3755 50  0000 L CNN
 F 2 "Capacitor_THT:C_Disc_D3.0mm_W2.0mm_P2.50mm" H 9388 3650 50  0001 C CNN
 F 3 "~" H 9350 3800 50  0001 C CNN
@@
 $EndComp
 $Comp
-L Device:C C2
-U 1 1 6274EADA
-P 9350 2400
-F 0 "C2" H 9465 2446 50  0000 L CNN
-F 1 "C" H 9465 2355 50  0000 L CNN
-F 2 "Capacitor_THT:C_Disc_D3.0mm_W2.0mm_P2.50mm" H 9388 2250 50  0001 C CNN
-F 3 "~" H 9350 2400 50  0001 C CNN
-	1    9350 2400
-	1    0    0    -1
-$EndComp
-$Comp
 L Device:C C6
 U 1 1 6274F92D
-P 9350 5100
-F 0 "C6" H 9465 5146 50  0000 L CNN
-F 1 "C" H 9465 5055 50  0000 L CNN
-F 2 "Capacitor_THT:C_Disc_D3.0mm_W2.0mm_P2.50mm" H 9388 4950 50  0001 C CNN
-F 3 "~" H 9350 5100 50  0001 C CNN
-	1    9350 5100
-	1    0    0    -1
-$EndComp
-Wire Wire Line
-	9350 2100 9350 2250
+P 9650 5100
+F 0 "C6" H 9765 5146 50  0000 L CNN
+F 1 "0.05 µF" H 9765 5055 50  0000 L CNN
+F 2 "Capacitor_THT:C_Disc_D3.0mm_W2.0mm_P2.50mm" H 9688 4950 50  0001 C CNN
+F 3 "~" H 9650 5100 50  0001 C CNN
+	1    9650 5100
+	1    0    0    -1
+$EndComp
 Connection ~ 9350 2100
 Wire Wire Line
@@
 	9350 3500 9550 3500
 Wire Wire Line
-	9350 4950 9350 4800
-Connection ~ 9350 4800
-Wire Wire Line
-	9350 4800 9200 4800
-Text GLabel 9350 5250 3    50   Output ~ 0
-GND
-Text GLabel 9350 3950 3    50   Output ~ 0
-GND
-Text GLabel 9350 2550 3    50   Output ~ 0
+	9650 4950 9650 4800
+Connection ~ 9650 4800
+Text GLabel 9650 5550 3    50   Output ~ 0
+GND
+Text GLabel 9350 4250 3    50   Output ~ 0
+GND
+Text GLabel 9350 2850 3    50   Output ~ 0
 GND
 $Comp
@@
 P 9700 2100
 F 0 "C1" V 9955 2100 50  0000 C CNN
-F 1 "CP" V 9864 2100 50  0000 C CNN
+F 1 "250 µF" V 9864 2100 50  0000 C CNN
 F 2 "Capacitor_THT:CP_Radial_D5.0mm_P2.50mm" H 9738 1950 50  0001 C CNN
 F 3 "~" H 9700 2100 50  0001 C CNN
@@
 P 9700 3500
 F 0 "C3" V 9955 3500 50  0000 C CNN
-F 1 "CP" V 9864 3500 50  0000 C CNN
+F 1 "250 µF" V 9864 3500 50  0000 C CNN
 F 2 "Capacitor_THT:CP_Radial_D5.0mm_P2.50mm" H 9738 3350 50  0001 C CNN
 F 3 "~" H 9700 3500 50  0001 C CNN
@@
 L Device:CP C5
 U 1 1 6275E993
-P 9700 4800
-F 0 "C5" V 9955 4800 50  0000 C CNN
-F 1 "CP" V 9864 4800 50  0000 C CNN
-F 2 "Capacitor_THT:CP_Radial_D5.0mm_P2.50mm" H 9738 4650 50  0001 C CNN
-F 3 "~" H 9700 4800 50  0001 C CNN
-	1    9700 4800
+P 10000 4800
+F 0 "C5" V 10255 4800 50  0000 C CNN
+F 1 "250 µF" V 10164 4800 50  0000 C CNN
+F 2 "Capacitor_THT:CP_Radial_D5.0mm_P2.50mm" H 10038 4650 50  0001 C CNN
+F 3 "~" H 10000 4800 50  0001 C CNN
+	1    10000 4800
 	0    -1   -1   0
 $EndComp
@@
 Text GLabel 9850 3500 2    50   Output ~ 0
 SND_L
-Text GLabel 9850 4800 2    50   Output ~ 0
+Text GLabel 10500 4800 2    50   Output ~ 0
 SND_SUB
 $Comp
@@
 Text GLabel 5150 2100 3    50   Output ~ 0
 GND
+Wire Wire Line
+	9350 2100 9350 2250
+$Comp
+L Device:C C2
+U 1 1 6274EADA
+P 9350 2400
+F 0 "C2" H 9465 2446 50  0000 L CNN
+F 1 "0.05 µF" H 9465 2355 50  0000 L CNN
+F 2 "Capacitor_THT:C_Disc_D3.0mm_W2.0mm_P2.50mm" H 9388 2250 50  0001 C CNN
+F 3 "~" H 9350 2400 50  0001 C CNN
+	1    9350 2400
+	1    0    0    -1
+$EndComp
+$Comp
+L Device:R R1
+U 1 1 62731CE4
+P 9350 2700
+F 0 "R1" H 9420 2746 50  0000 L CNN
+F 1 "10 Ω" H 9420 2655 50  0000 L CNN
+F 2 "Resistor_THT:R_Axial_DIN0204_L3.6mm_D1.6mm_P5.08mm_Horizontal" V 9280 2700 50  0001 C CNN
+F 3 "~" H 9350 2700 50  0001 C CNN
+	1    9350 2700
+	1    0    0    -1
+$EndComp
+$Comp
+L Device:R R2
+U 1 1 627320F2
+P 9350 4100
+F 0 "R2" H 9420 4146 50  0000 L CNN
+F 1 "10 Ω" H 9420 4055 50  0000 L CNN
+F 2 "Resistor_THT:R_Axial_DIN0204_L3.6mm_D1.6mm_P5.08mm_Horizontal" V 9280 4100 50  0001 C CNN
+F 3 "~" H 9350 4100 50  0001 C CNN
+	1    9350 4100
+	1    0    0    -1
+$EndComp
+$Comp
+L Device:R R3
+U 1 1 627325BE
+P 9650 5400
+F 0 "R3" H 9720 5446 50  0000 L CNN
+F 1 "10 Ω" H 9720 5355 50  0000 L CNN
+F 2 "Resistor_THT:R_Axial_DIN0204_L3.6mm_D1.6mm_P5.08mm_Horizontal" V 9580 5400 50  0001 C CNN
+F 3 "~" H 9650 5400 50  0001 C CNN
+	1    9650 5400
+	1    0    0    -1
+$EndComp
+$Comp
+L Device:CP C10
+U 1 1 62745B6D
+P 8900 3950
+F 0 "C10" H 9018 3996 50  0000 L CNN
+F 1 "10 µF" H 9018 3905 50  0000 L CNN
+F 2 "Capacitor_THT:CP_Radial_D5.0mm_P2.50mm" H 8938 3800 50  0001 C CNN
+F 3 "~" H 8900 3950 50  0001 C CNN
+	1    8900 3950
+	1    0    0    -1
+$EndComp
+$Comp
+L Device:CP C8
+U 1 1 6274648A
+P 8900 2550
+F 0 "C8" H 9018 2596 50  0000 L CNN
+F 1 "10 µF" H 9018 2505 50  0000 L CNN
+F 2 "Capacitor_THT:CP_Radial_D5.0mm_P2.50mm" H 8938 2400 50  0001 C CNN
+F 3 "~" H 8900 2550 50  0001 C CNN
+	1    8900 2550
+	1    0    0    -1
+$EndComp
+Wire Wire Line
+	9000 2400 9000 2700
+Wire Wire Line
+	9000 2700 8900 2700
+Wire Wire Line
+	9000 3800 9000 4100
+Wire Wire Line
+	9000 4100 8900 4100
+$Comp
+L Device:R R5
+U 1 1 62753AA3
+P 9050 5500
+F 0 "R5" V 8843 5500 50  0000 C CNN
+F 1 "10 Ω" V 8934 5500 50  0000 C CNN
+F 2 "Resistor_THT:R_Axial_DIN0204_L3.6mm_D1.6mm_P5.08mm_Horizontal" V 8980 5500 50  0001 C CNN
+F 3 "~" H 9050 5500 50  0001 C CNN
+	1    9050 5500
+	0    1    1    0
+$EndComp
+$Comp
+L Device:C C12
+U 1 1 62753E9A
+P 9350 5200
+F 0 "C12" H 9465 5246 50  0000 L CNN
+F 1 "0.033 µF" H 9465 5155 50  0000 L CNN
+F 2 "Capacitor_THT:C_Disc_D3.0mm_W2.0mm_P2.50mm" H 9388 5050 50  0001 C CNN
+F 3 "~" H 9350 5200 50  0001 C CNN
+	1    9350 5200
+	-1   0    0    1
+$EndComp
+Wire Wire Line
+	9200 4800 9350 4800
+Wire Wire Line
+	9350 5050 9350 4800
+Connection ~ 9350 4800
+Wire Wire Line
+	9350 4800 9650 4800
+Wire Wire Line
+	8900 5500 8900 5100
+Wire Wire Line
+	9200 5500 9350 5500
+Wire Wire Line
+	9350 5500 9350 5350
+Wire Wire Line
+	10150 4800 10500 4800
+Text GLabel 10300 5100 3    50   Output ~ 0
+GND
+$Comp
+L Device:R R4
+U 1 1 62766EED
+P 10300 4950
+F 0 "R4" H 10370 4996 50  0000 L CNN
+F 1 "? Ω" H 10370 4905 50  0000 L CNN
+F 2 "Resistor_THT:R_Axial_DIN0204_L3.6mm_D1.6mm_P5.08mm_Horizontal" V 10230 4950 50  0001 C CNN
+F 3 "~" H 10300 4950 50  0001 C CNN
+	1    10300 4950
+	1    0    0    -1
+$EndComp
+NoConn ~ 9000 5100
+$Comp
+L Amplifier_Audio:LM386 U5
+U 1 1 6273E396
+P 8900 2100
+F 0 "U5" H 9244 2146 50  0000 L CNN
+F 1 "LM386" H 9244 2055 50  0000 L CNN
+F 2 "Package_DIP:DIP-8_W7.62mm_Socket_LongPads" H 9000 2200 50  0001 C CNN
+F 3 "http://www.ti.com/lit/ds/symlink/lm386.pdf" H 9100 2300 50  0001 C CNN
+	1    8900 2100
+	1    0    0    -1
+$EndComp
+$Comp
+L Device:C C7
+U 1 1 62770B43
+P 9050 1800
+F 0 "C7" V 8798 1800 50  0000 C CNN
+F 1 "0.1 µF" V 8889 1800 50  0000 C CNN
+F 2 "Capacitor_THT:C_Disc_D3.0mm_W2.0mm_P2.50mm" H 9088 1650 50  0001 C CNN
+F 3 "~" H 9050 1800 50  0001 C CNN
+	1    9050 1800
+	0    1    1    0
+$EndComp
+Text GLabel 9200 1800 2    50   Output ~ 0
+GND
+$Comp
+L Device:C C9
+U 1 1 62777C6E
+P 9050 3200
+F 0 "C9" V 8798 3200 50  0000 C CNN
+F 1 "0.1 µF" V 8889 3200 50  0000 C CNN
+F 2 "Capacitor_THT:C_Disc_D3.0mm_W2.0mm_P2.50mm" H 9088 3050 50  0001 C CNN
+F 3 "~" H 9050 3200 50  0001 C CNN
+	1    9050 3200
+	0    1    1    0
+$EndComp
+$Comp
+L Device:C C11
+U 1 1 62778328
+P 9050 4500
+F 0 "C11" V 8798 4500 50  0000 C CNN
+F 1 "0.1 µF" V 8889 4500 50  0000 C CNN
+F 2 "Capacitor_THT:C_Disc_D3.0mm_W2.0mm_P2.50mm" H 9088 4350 50  0001 C CNN
+F 3 "~" H 9050 4500 50  0001 C CNN
+	1    9050 4500
+	0    1    1    0
+$EndComp
+Text GLabel 9200 3200 2    50   Output ~ 0
+GND
+Text GLabel 9200 4500 2    50   Output ~ 0
+GND
 $EndSCHEMATC

Commit message: Completed Sound Card...
Parts:
- LINE_OUT1: renamed from J2; value LINE OUT -> 3.5mm stereo
- SUB_OUT1: renamed from J3; value SUB OUT -> 3.5mm mono
Connections:
- net SND_SUB: now also R4.1
Changed lines of the file:
@@
 SND_SUB
 $Comp
-L Connector:AudioJack3 J2
+L Connector:AudioJack3 LINE_OUT1
 U 1 1 62762067
 P 6900 4900
-F 0 "J2" H 6882 5225 50  0000 C CNN
-F 1 "LINE OUT" H 6882 5134 50  0000 C CNN
+F 0 "LINE_OUT1" H 6882 5225 50  0000 C CNN
+F 1 "3.5mm stereo" H 6882 5134 50  0000 C CNN
 F 2 "Connector_Audio:Jack_3.5mm_CUI_SJ1-3533NG_Horizontal" H 6900 4900 50  0001 C CNN
 F 3 "~" H 6900 4900 50  0001 C CNN
@@
 GND
 $Comp
-L Connector:AudioJack2 J3
+L Connector:AudioJack2 SUB_OUT1
 U 1 1 62765D72
 P 6850 5850
-F 0 "J3" H 6882 6175 50  0000 C CNN
-F 1 "SUB OUT" H 6882 6084 50  0000 C CNN
+F 0 "SUB_OUT1" H 6882 6175 50  0000 C CNN
+F 1 "3.5mm mono" H 6882 6084 50  0000 C CNN
 F 2 "Connector_Audio:Jack_3.5mm_CUI_SJ1-3533NG_Horizontal" H 6850 5850 50  0001 C CNN
 F 3 "~" H 6850 5850 50  0001 C CNN
@@
 Wire Wire Line
 	9350 5500 9350 5350
-Wire Wire Line
-	10150 4800 10500 4800
 Text GLabel 10300 5100 3    50   Output ~ 0
 GND
@@
 Text GLabel 9200 4500 2    50   Output ~ 0
 GND
+Wire Wire Line
+	10150 4800 10300 4800
+Connection ~ 10300 4800
+Wire Wire Line
+	10300 4800 10500 4800
 $EndSCHEMATC
