File: Sound/Sound.kicad_sch (KiCad schematic)
At the start: 31 parts, among them J1 Expansion_Connector, U1 74HCT74, U2 74HCT02, U3 74HCT138, U4 74HCT138, U5 LM386, U6 LM386, U7 LM386

Commit message: 405 unrouted traces...
Parts:
- J1: value Expansion_Connector -> 2x19 2.54mm Right-angled Header
Changed lines of the file:
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@@
     (in_bom yes) (on_board yes)
     (property "Reference" "J1" (id 0) (at 53.34 46.5582 0))
-    (property "Value" "Expansion_Connector" (id 1) (at 53.34 48.8696 0))
+    (property "Value" "2x19 2.54mm Right-angled Header" (id 1) (at 53.34 48.8696 0))
     (property "Footprint" "PC:Expansion_Connector_Board" (id 2) (at 52.07 77.47 0)
       (effects (font (size 1.27 1.27)) hide)
@@
     )
     (path "/00000000-0000-0000-0000-000062713709"
-      (reference "J1") (unit 1) (value "Expansion_Connector") (footprint "PC:Expansion_Connector_Board")
+      (reference "J1") (unit 1) (value "2x19 2.54mm Right-angled Header") (footprint "PC:Expansion_Connector_Board")
     )
     (path "/00000000-0000-0000-0000-000062762067"

Commit message: Finished sound card 1.2...
Parts:
- removed U2: 74HCT02, Package_DIP:DIP-14_W7.62mm_Socket_LongPads, symbol 74xx:74HCT02
- removed U3, U4: 74HCT138, Package_DIP:DIP-16_W7.62mm_Socket_LongPads, symbol 74xx:74LS138
- added U3: ATF22V10C, Package_DIP:DIP-24_W7.62mm_Socket_LongPads, symbol PC:ATF22V10C
Connections:
- net A10: now also U3.7 (IN)
- net A11: now also U3.6 (IN)
- net A5: now also U3.13 (IN)
- net A6: now also U3.11 (IN)
- net A7: now also U3.10 (IN)
- net A8: now also U3.9 (IN)
- net A9: now also U3.8 (IN)
- net GND: now also U3.12 (GND)
- net PHI2: now also U3.1 (CLK/IN)
- net VCC: now also SOUND_CTRL1.24 (CS1), U3.24 (VCC)
- net ~{CS_SND}: now also SOUND_CTRL1.23 (~{CS2}), U3.14 (I/O); no longer SOUND_CTRL1.12 (PB2)
- net A12: now reaches J1.29 (Pin_29)
- net A12: now also U3.5 (IN)
- net A13: now reaches J1.31 (Pin_31)
- net A13: now also U3.4 (IN/PD)
- net A14: now reaches J1.33 (Pin_33)
- net A14: now also U3.3 (IN)
- net A15: now reaches J1.35 (Pin_35)
- net A15: now also U3.2 (IN)
- net CS_DEV: no longer names the net of J1.28 (Pin_28)
- net CS_DEV: no longer SOUND_CTRL1.24 (CS1)
- no-connect marks 37 -> 30
