File: Sound/Sound.kicad_sch (KiCad schematic)
At the start: 29 parts, among them J1 2x19 2.54mm Right-angled Head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, U1 74HCT74, U3 ATF22V10C, U5 LM386, U6 LM386, U7 LM386

Commit message: Update to latest KiCad version and other edits.
Updated the files formatting to conform to KiCad 10 standards, updated dates and corrected company name, also first signed commit to this repository.
Other:
- company: WolfNet Computing -> WolfNet Computing C.I.C.
