File: Sound/Sound.kicad_pcb (KiCad board)
At the start: 4 copper layers, 133.6 x 74.7 mm, 32 parts, among them J1 Expansion_Connector, U1 74HCT74, U2 74HCT02, U3 74HCT138, U4 74HCT138, U5 LM386, U6 LM386, U7 LM386

Commit message: 405 unrouted traces...
Parts:
- removed G***: LOGO, WolfNet:WolfNet-Logo_silkscreen
- J1: value Expansion_Connector -> 2x19 2.54mm Right-angled Header

Commit message: Finished sound card...
Parts:
- moved R2 39.2 mm to (54.6, 110.5)
- moved R1 17.6 mm to (104.4, 58.4)
- moved R4 17.6 mm to (91.4, 58.4)
- moved U1 11.3 mm to (115.6, 90.2)
- moved C10 9.08 mm to (83.8, 99.1), turned to -90 degrees
- moved R3 8.98 mm to (100.3, 85.1)
- moved C8 8.76 mm to (87.6, 85.1), turned to -90 degrees
- moved R5 8.09 mm to (88.9, 77.5)
- moved C4 5.07 mm to (57.1, 108.0), turned to 180 degrees
- moved C6 3.33 mm to (100.3, 78.7), turned to -90 degrees
- moved C3 2.99 mm to (63.5, 108.0)
- moved C5 2.68 mm to (83.8, 82.5)
- moved C12 0.84 mm to (97.8, 71.1)
- moved U6 0.40 mm to (70.0, 101.6)
- moved U5 0.37 mm to (70.0, 87.6)
Routing:
- net GND: track 0.00 -> 379.9 mm, vias 0 -> 1
- net VCC: track 0.00 -> 256.8 mm
- net A5: track 0.00 -> 130.2 mm, vias 0 -> 4
- net A9: track 0.00 -> 126.1 mm, vias 0 -> 2
- net A8: track 0.00 -> 119.3 mm, vias 0 -> 6
- net Net-(LINE_OUT_VOLUME1-Pad1): track 0.00 -> 108.9 mm, vias 0 -> 3
- net A6: track 0.00 -> 108.6 mm, vias 0 -> 2
- net A10: track 0.00 -> 105.0 mm, vias 0 -> 4
- net A11: track 0.00 -> 104.1 mm, vias 0 -> 4
- net A4: track 0.00 -> 102.7 mm, vias 0 -> 3
- net A7: track 0.00 -> 100.8 mm, vias 0 -> 2
- net Net-(LINE_OUT_VOLUME1-Pad4): track 0.00 -> 88.8 mm, vias 0 -> 2
- net Net-(SOUND_GEN1-Pad18): track 0.00 -> 69.7 mm
- net ~{RESET}: track 0.00 -> 69.7 mm
- net 8MHz: track 0.00 -> 67.3 mm
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
Commit message: Updated worksheet...
Parts:
- moved R5 37.6 mm to (67.6, 46.5)
- moved C1 37.6 mm to (66.4, 37.5)
- moved C11 37.6 mm to (63.7, 26.0)
- moved C12 37.6 mm to (76.5, 40.2)
- moved C2 37.6 mm to (77.1, 33.3)
- moved C3 37.6 mm to (42.2, 77.0)
- moved C4 37.6 mm to (35.8, 77.0)
- moved C6 37.6 mm to (79.0, 47.7)
- moved C8 37.6 mm to (66.3, 54.1)
- moved LINE_OUT1 37.6 mm to (43.7, 25.2)
- moved R1 37.6 mm to (83.1, 27.5)
- moved R3 37.6 mm to (79.0, 54.1)
- moved R4 37.6 mm to (70.1, 27.5)
- moved SOUND_CTRL1 37.6 mm to (126.1, 23.7)
- moved SOUND_GEN1 37.6 mm to (117.1, 51.6)
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
Commit message: Finished sound card 1.2...
Parts:
- removed U2: 74HCT02, Package_DIP:DIP-14_W7.62mm_Socket_LongPads
- removed U4: 74HCT138, Package_DIP:DIP-16_W7.62mm_Socket_LongPads
- U3: value 74HCT138 -> ATF22V10C; footprint Package_DIP:DIP-16_W7.62mm_Socket_LongPads -> Package_DIP:DIP-24_W7.62mm_Socket_LongPads
- moved U3 13.2 mm to (89.1, 81.5), turned to 90 degrees
Connections:
- J1 pad 28: CS_DEV -> unconnected-(J1-Pad28)
- J1 pad 29: unconnected-(J1-Pad29) -> A12
- J1 pad 31: unconnected-(J1-Pad31) -> A13
- J1 pad 33: unconnected-(J1-Pad33) -> A14
- J1 pad 35: unconnected-(J1-Pad35) -> A15
- SOUND_CTRL1 pad 12: ~{CS_SND} -> unconnected-(SOUND_CTRL1-Pad12)
- SOUND_CTRL1 pad 23: Net-(SOUND_CTRL1-Pad23) -> ~{CS_SND}
- SOUND_CTRL1 pad 24: CS_DEV -> VCC
- U3 pad 1: A4 -> PHI2
- U3 pad 10: unconnected-(U3-Pad10) -> A7
- U3 pad 11: unconnected-(U3-Pad11) -> A6
- U3 pad 12: unconnected-(U3-Pad12) -> GND
- U3 pad 13: unconnected-(U3-Pad13) -> A5
- U3 pad 14: unconnected-(U3-Pad14) -> ~{CS_SND}
- U3 pad 15: Net-(U2-Pad2) -> unconnected-(U3-Pad15)
- U3 pad 16: VCC -> unconnected-(U3-Pad16)
- U3 pad 2: A6 -> A15
- U3 pad 3: A7 -> A14
- U3 pad 4: GND -> A13
- U3 pad 5: GND -> A12
- U3 pad 6: A5 -> A11
- U3 pad 7: unconnected-(U3-Pad7) -> A10
- U3 pad 8: GND -> A9
- U3 pad 9: unconnected-(U3-Pad9) -> A8
Routing:
- net A4: track 102.7 -> 0.00 mm, vias 3 -> 0
- net A12: track 0.00 -> 86.9 mm, vias 0 -> 3
- net A15: track 0.00 -> 79.7 mm, vias 0 -> 1
- net A13: track 0.00 -> 79.2 mm, vias 0 -> 1
- net A14: track 0.00 -> 78.5 mm, vias 0 -> 1
- net PHI2: track 25.3 -> 97.0 mm, vias 0 -> 1
- net A5: track 130.2 -> 76.1 mm, vias 4 -> 2
- net Net-(SOUND_CTRL1-Pad23): track 47.1 -> 0.00 mm
- net A8: track 119.3 -> 78.7 mm, vias 6 -> 1
- net ~{CS_SND}: track 25.2 -> 64.6 mm, vias 0 -> 2
- net A9: track 126.1 -> 90.3 mm, vias 2 -> 3
- net Net-(U2-Pad3): track 31.1 -> 0.00 mm
- net A6: track 108.6 -> 83.2 mm, vias 2 -> 3
- net CS_DEV: track 25.3 -> 0.00 mm
- net Net-(U2-Pad2): track 22.1 -> 0.00 mm, vias 2 -> 0
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
Commit message: Logo added...
Parts:
- added G***: LOGO, WolfNet:WolfNet-Logo_silkscreen, F.Cu at (71.1, 81.3)
