File: Video/Video.sch (KiCad schematic (older format))
At the start: 0 parts

Commit message: Added video card project files...
Parts:
- added J?: WolfNet_Bus_ISA_8bit, symbol PC:WolfNet_Bus_ISA_8bit
Changed lines of the file:
@@
 Comment4 ""
 $EndDescr
+$Comp
+L PC:WolfNet_Bus_ISA_8bit J?
+U 1 1 6274B212
+P 5800 3750
+F 0 "J?" H 5800 5517 50  0000 C CNN
+F 1 "WolfNet_Bus_ISA_8bit" H 5800 5426 50  0000 C CNN
+F 2 "" H 5800 3750 50  0001 C CNN
+F 3 "https://en.wikipedia.org/wiki/Industry_Standard_Architecture" H 5800 3750 50  0001 C CNN
+	1    5800 3750
+	1    0    0    -1
+$EndComp
 $EndSCHEMATC

Commit message: Updated libraries and started video card...
Parts:
- removed J?: WolfNet_Bus_ISA_8bit, symbol PC:WolfNet_Bus_ISA_8bit
- added J?: Bus_ISA_8bit, symbol Connector:Bus_ISA_8bit
Changed lines of the file:
@@
 $EndDescr
 $Comp
-L PC:WolfNet_Bus_ISA_8bit J?
-U 1 1 6274B212
-P 5800 3750
-F 0 "J?" H 5800 5517 50  0000 C CNN
-F 1 "WolfNet_Bus_ISA_8bit" H 5800 5426 50  0000 C CNN
-F 2 "" H 5800 3750 50  0001 C CNN
-F 3 "https://en.wikipedia.org/wiki/Industry_Standard_Architecture" H 5800 3750 50  0001 C CNN
-	1    5800 3750
+L Connector:Bus_ISA_8bit J?
+U 1 1 6273BFD6
+P 5600 3800
+F 0 "J?" H 5600 5567 50  0000 C CNN
+F 1 "Bus_ISA_8bit" H 5600 5476 50  0000 C CNN
+F 2 "" H 5600 3800 50  0001 C CNN
+F 3 "https://en.wikipedia.org/wiki/Industry_Standard_Architecture" H 5600 3800 50  0001 C CNN
+	1    5600 3800
 	1    0    0    -1
 $EndComp

Commit message: Updated video card...
Parts:
- removed J?: Bus_ISA_8bit, symbol Connector:Bus_ISA_8bit
Changed lines of the file:
@@
 Comment4 ""
 $EndDescr
-$Comp
-L Connector:Bus_ISA_8bit J?
-U 1 1 6273BFD6
-P 5600 3800
-F 0 "J?" H 5600 5567 50  0000 C CNN
-F 1 "Bus_ISA_8bit" H 5600 5476 50  0000 C CNN
-F 2 "" H 5600 3800 50  0001 C CNN
-F 3 "https://en.wikipedia.org/wiki/Industry_Standard_Architecture" H 5600 3800 50  0001 C CNN
-	1    5600 3800
-	1    0    0    -1
-$EndComp
 $EndSCHEMATC
