File: Video/Video.kicad_sch (KiCad schematic)
At the start: 6 parts

Commit message: Update to latest KiCad version and other edits.
Updated the files formatting to conform to KiCad 10 standards, updated dates and corrected company name, also first signed commit to this repository.
Parts:
- gave numbers to parts that had none: 5
- renumbered SYNC_GENERATOR to SYNC_GENERATOR1
Other:
- company: WolfNet Computing -> WolfNet Computing C.I.C.
